Commit message: some control testing

File: src/freefloating_gazebo_demo/urdf/barcoLeme_tmp.xacro (robot description, xacro)
@@ -90,10 +90,10 @@
 			<mass value="0.05" />
 			<inertia
-			  ixx="0.2708000"
+			  ixx="0.4708000"
 			  ixy="0.0"
-			  iyy="0.0508"
+			  iyy="0.5208"
 			  ixz="0.0"
 			  iyz="0.0"
-			  izz="0.5208"/>
+			  izz="0.0508"/>
 		</inertial>
 	      <collision name="collision">
@@ -116,5 +116,5 @@
             <dynamics damping="1.0"/>
             <axis xyz="0 0 1"/>
-            <limit effort="50" velocity="5" lower="-${PI/3}" upper="${PI/3}" />
+            <limit effort="50" velocity="5" lower="-${PI/2}" upper="${PI/2}" />
         </joint>
 <!-- Plugin list -->
