Commit message: update

File: src/freefloating_gazebo_demo/urdf/outroTeste.urdf (robot description, URDF)
Before this commit: robot barco_auv, 3 links, 2 joints
Links:
- added link camera_link, mass 1e-5; collision box size=${camera_link} ${camera_link} ${camera_link}; visual box size=${camera_link} ${camera_link} ${camera_link}
- added link camera_link_optical
Joints:
- added joint camera_joint: type fixed, parent link3, child camera_link, origin xyz=${camera_link} 0 ${height3 - axel_offset*2} rpy=0 0 0, axis 0 1 0
- added joint camera_optical_joint: type fixed, parent camera_link, child camera_link_optical, origin xyz=0 0 0 rpy=${-pi/2} 0 ${-pi/2}
