Commit message: Fixing barcoLeme.xacro to not sink

File: src/freefloating_gazebo_demo/urdf/barcoLeme.xacro (robot description, xacro)
@@ -4,5 +4,5 @@
     <xacro:property name="PI" value="3.1415926535897931"/>
     <!-- Body properties -->
-    <xacro:property name="body_mass" value="5"/>
+    <xacro:property name="body_mass" value="10"/>
     <xacro:property name="body_radius" value="0.13"/>
     <xacro:property name="body_length" value="1.5" />
@@ -44,12 +44,12 @@
             </visual>
             <inertial>
-                <mass value=".1"/>
+                <mass value="0.1"/>
                 <inertia
-                    ixx=".1"
+                    ixx="0.01"
                     ixy="0.0"
                     ixz="0.0"
-                    iyy=".1"
+                    iyy="0.01"
                     iyz="0.0"
-                    izz=".1"/>
+                    izz="0.01"/>
                 </inertial>
             </link>
@@ -80,13 +80,13 @@
                 </inertial>
                 <buoyancy>
-                    <compensation>1.05</compensation>
+                    <compensation>1.2</compensation>
                     <origin xyz= "0 0 0"/>
                     <limit radius="${body_radius}"/>
-                    <damping xyz="40 100 100" rpy="20 50 50"/>
+                    <damping xyz="20 50 50" rpy="20 50 50"/>
                 </buoyancy>
             </link>
 	<link name="rudder">
 		<inertial>
-			<mass value="0.1" />
+			<mass value="0.05" />
 			<inertia
 			  ixx="0.4708"
@@ -146,5 +146,5 @@
                 <thruster>
                     <effort>30</effort>
-                    <name>fwd_left</name>
+                    <name>fwd</name>
                 </thruster>
                 <!-- these thrusters are fixed and the map can be hard-coded
@@ -153,5 +153,5 @@
         </gazebo>
     <!-- Define two steering thrusters, with assumed force control in Z-direction -->
-    <xacro:thruster_link name="fwd_left" xyz="-0.52 0 0" rpy="0 ${-PI/2} 0"/>
+    <xacro:thruster_link name="fwd" xyz="-0.52 0 -0.03" rpy="0 ${-PI/2} 0"/>
     <xacro:macro name="thruster_dummy_link" params="name xyz rpy">
         <joint name="${name}" type="fixed">
@@ -166,3 +166,3 @@
     <xacro:thruster_dummy_link name="thr3" xyz="-0.45 0.0 0.0" rpy="0.0 -0.0 0.0"/>
     <xacro:thruster_dummy_link name="thr4" xyz="0.45 0.0 0.0" rpy="0.0 -0.0 0.0"/>-->
-        </robot>
+</robot>

File: src/freefloating_gazebo_demo/urdf/barcoLeme_dummy.urdf (robot description, URDF)
Before this commit: robot thrusters, 0 links, 1 joints
Joints:
- removed joint fwd_left
- added joint fwd: type None, limit lower=-30 upper=30

Commit message: Changing CMakeLists from packages. Testing topic /vehicle/Surface

File: src/freefloating_gazebo_demo/urdf/barcoLeme.xacro (robot description, xacro)
@@ -90,10 +90,10 @@
 			<mass value="0.05" />
 			<inertia
-			  ixx="0.4708"
+			  ixx="0.05"
 			  ixy="0.0"
-			  iyy="0.5208"
+			  iyy="0.05"
 			  ixz="0.0"
 			  iyz="0.0"
-			  izz="0.0508"/>
+			  izz="0.005"/>
 		</inertial>
 	      <collision name="collision">
@@ -124,11 +124,13 @@
 		<!--<plugin name="LiftDrag" filename="libliftdragww.so">-->
 			<a0>0</a0>
-			<cla>4.752798721</cla>
-			<cda>0.6417112299</cda>
-			<cma>-1.8</cma>
+			<cla>0.752798721</cla>
+			<cda>0.3417112299</cda>
+			<!--
+			<cma>-1.8</cma> momentum
+			<cma_stall>0</cma_stall>
+			-->
 			<alpha_stall>0.785</alpha_stall>
-			<cla_stall>-3.85</cla_stall>
-			<cda_stall>-0.9233984055</cda_stall>
-			<cma_stall>0</cma_stall>
+			<cla_stall>-0.85</cla_stall>
+			<cda_stall>-0.3233984055</cda_stall>
 			<cp>-0.5 0 0</cp>
 			<area>0.03</area>

File: src/freefloating_gazebo_demo/urdf/bbox.xacro (robot description, xacro)
@@ -6,5 +6,5 @@
       <origin rpy="0 0 0" xyz="0 0 0"/>
       <geometry>
-          <mesh filename="package://freefloating_gazebo_demo/objects/blackbox_uib_trimesh.dae"/>
+          <mesh filename="/objects/blackbox_uib_trimesh.dae"/>
       </geometry>
     </visual>
@@ -17,5 +17,5 @@
       <origin xyz="0 0 0" rpy="0 0 0"/>
      <geometry>
-          <mesh filename="package://freefloating_gazebo_demo/objects/blackbox_uib_trimesh.dae"/>
+          <mesh filename="/objects/blackbox_uib_trimesh.dae"/>
       </geometry>
     </collision>

File: src/freefloating_gazebo_demo/urdf/bbox_uwsim.urdf (robot description, URDF)
Before this commit: robot blackbox, 1 links, 0 joints
Links:
- link link: geometry visual mesh filename=/objects/blackbox_uib_trimesh.osg
