Commit message: barcoDiferential model updated and velocity control (cmd_vel) added

File: src/freefloating_gazebo_demo/urdf/barcoDiferencial.xacro (robot description, xacro)
@@ -57,50 +57,41 @@
                 <material>Gazebo/Black</material>
             </gazebo>
-        </xacro:macro>
-        <link name="base_link">
-            <visual>
-                <origin rpy="0 0 0"/>
-                <geometry>
-<!--		    <mesh filename="file://$(env HOME)/.uwsim/data/robot/barco/pt90.stl"/>-->
-	 		<box size="1.0 0.4 0.2" />
-                </geometry>
-		  <material name="blue">
-		    <color rgba="0 0 .8 1"/>
-		  </material>
-            </visual>
-            <inertial>
-                <origin xyz="0 0 ${X_cog}" rpy="0 0 0"/>
-                <mass value="${body_mass}"/>
-                <inertia
-                    ixx="${body_mass*(body_radius*body_radius/4+body_length*body_length/12)}"
-                    ixy="0.0"
-                    ixz="0.0"
-                    iyy="${body_mass*(body_radius*body_radius/4+body_length*body_length/12)}"
-                    iyz="0.0"
-                    izz="${body_mass*body_radius*body_radius/2}"/>
-                </inertial>
-                <buoyancy>
-                    <compensation>1.05</compensation>
-                    <origin xyz= "0 0 0"/>
-                    <limit radius="${body_radius}"/>
-                    <damping xyz="40 100 100" rpy="20 50 50"/>
-                </buoyancy>
-            </link>
+    </xacro:macro>
+    <link name="base_link">
+        <visual>
+          <origin rpy="1.57079632679 0 1.57079632679"/>
+          <geometry>
+            <mesh filename="file:///home/lsa/.uwsim/data/robot/barco/pt90.stl"/>
+          </geometry>
+          <material name="blue"/>
+        </visual>
+        <inertial>
+            <origin rpy="0 0 0" xyz="0 0 -0.05"/>
+          <mass value="10"/>
+          <inertia ixx="0.1" ixy="0.0" ixz="0.0" iyy="1.4" iyz="0.0" izz="1.4"/>
+        </inertial>
+        <buoyancy>
+          <compensation>1.2</compensation>
+          <origin xyz="-0.0005 0 0.05"/>
+          <limit radius="0.1"/>
+          <damping rpy="20 50 50" xyz="20 50 50"/>
+        </buoyancy>
+    </link>
 	<!-- Plugin list -->
-        <gazebo>
-            <plugin name="freefloating_gazebo_control" filename="libfreefloating_gazebo_control.so">
-                <switchService>switch</switchService>
-                <updateRate>100</updateRate>
-                <link>base_link</link>
-                <thruster>
-                    <effort>30</effort>
-                    <name>fwd_left</name>
-                </thruster>
-		<thruster>
-                    <effort>30</effort>
-                    <name>fwd_right</name>
-                </thruster>
-            </plugin>
-        </gazebo>
+    <gazebo>
+        <plugin name="freefloating_gazebo_control" filename="libfreefloating_gazebo_control.so">
+            <switchService>switch</switchService>
+            <updateRate>100</updateRate>
+            <link>base_link</link>
+            <thruster>
+                <effort>30</effort>
+                <name>fwd_left</name>
+            </thruster>
+    <thruster>
+                <effort>30</effort>
+                <name>fwd_right</name>
+            </thruster>
+        </plugin>
+    </gazebo>
     <!-- Define two steering thrusters, with assumed force control in Z-direction -->
     <xacro:thruster_link name="fwd_left" xyz="-0.52 0.1 0" rpy="0 ${-PI/2} 0"/>
@@ -118,3 +109,3 @@
     <xacro:thruster_dummy_link name="thr3" xyz="-0.45 0.0 0.0" rpy="0.0 -0.0 0.0"/>
     <xacro:thruster_dummy_link name="thr4" xyz="0.45 0.0 0.0" rpy="0.0 -0.0 0.0"/>-->
-        </robot>
+</robot>

Commit message: horizontal laser added to barcoDiferential model

File: src/freefloating_gazebo_demo/urdf/barcoDiferencial.xacro (robot description, xacro)
@@ -78,4 +78,65 @@
         </buoyancy>
     </link>
+    <joint name="hokuyo_joint" type="fixed">
+    <axis xyz="0 1 0" />
+    <origin xyz="0.6 0 0.1" rpy="0 0 0"/>
+    <parent link="base_link"/>
+    <child link="hokuyo_link"/>
+    </joint>
+    <!-- Hokuyo Laser -->
+    <link name="hokuyo_link">
+    <collision>
+    <origin xyz="0 0 0" rpy="0 0 0"/>
+    <geometry>
+    <box size="0.1 0.1 0.1"/>
+    </geometry>
+    </collision>
+    <visual>
+    <origin xyz="0 0 0" rpy="0 0 0"/>
+    <geometry>
+    <mesh filename="package://rrbot_description/meshes/hokuyo.dae"/>
+    </geometry>
+    </visual>
+    <inertial>
+    <mass value="1e-5" />
+    <origin xyz="0 0 0" rpy="0 0 0"/>
+    <inertia ixx="1e-6" ixy="0" ixz="0" iyy="1e-6" iyz="0" izz="1e-6" />
+    </inertial>
+</link>
+    <gazebo reference="hokuyo_link">
+    <sensor type="gpu_ray" name="head_hokuyo_sensor">
+    <pose>0 0 0 0 0 0</pose>
+    <visualize>true</visualize>
+    <update_rate>40</update_rate>
+    <ray>
+    <scan>
+    <horizontal>
+    <samples>720</samples>
+    <resolution>1</resolution>
+    <min_angle>-1.570796</min_angle>
+    <max_angle>1.570796</max_angle>
+    </horizontal>
+    </scan>
+    <range>
+    <min>0.10</min>
+    <max>30.0</max>
+    <resolution>0.01</resolution>
+    </range>
+    <noise>
+    <type>gaussian</type>
+    <!-- Noise parameters based on published spec for Hokuyo laser
+    achieving "+-30mm" accuracy at range < 10m.  A mean of 0.0m and
+    stddev of 0.01m will put 99.7% of samples within 0.03m of the true
+    reading. -->
+    <mean>0.0</mean>
+    <stddev>0.01</stddev>
+    </noise>
+    </ray>
+    <plugin name="gazebo_ros_head_hokuyo_controller" filename="libgazebo_ros_gpu_laser.so">
+    <topicName>/rrbot/laser/scan</topicName>
+    <frameName>hokuyo_link</frameName>
+    </plugin>
+    </sensor>
+    </gazebo>
 	<!-- Plugin list -->
     <gazebo>

Commit message: added navigation with navigation_stack

File: src/freefloating_gazebo_demo/urdf/barcoDiferencial.xacro (robot description, xacro)
@@ -134,5 +134,5 @@
     </ray>
     <plugin name="gazebo_ros_head_hokuyo_controller" filename="libgazebo_ros_gpu_laser.so">
-    <topicName>/rrbot/laser/scan</topicName>
+    <topicName>/scan</topicName>
     <frameName>hokuyo_link</frameName>
     </plugin>

File: src/freefloating_gazebo_demo/urdf/barco_obs.xacro (robot description, xacro)
@@ -29,10 +29,5 @@
           <inertia ixx="0.5" ixy="0.0" ixz="0.0" iyy="0.5" iyz="0.0" izz="0.5"/>
         </inertial>
-        <buoyancy>
-            <compensation>1.2</compensation>
-            <origin xyz= "0 0 0"/>
-            <limit radius="0.1"/>
-            <damping xyz="20 50 50" rpy="20 50 50"/>
-        </buoyancy>
+        <static>true</static>
     </link>
 </robot>

File: src/freefloating_gazebo_demo/urdf/barco_obs1.xacro (robot description, xacro)
@@ -29,10 +29,5 @@
           <inertia ixx="0.5" ixy="0.0" ixz="0.0" iyy="0.5" iyz="0.0" izz="0.5"/>
         </inertial>
-        <buoyancy>
-            <compensation>1.2</compensation>
-            <origin xyz= "0 0 0"/>
-            <limit radius="0.1"/>
-            <damping xyz="20 50 50" rpy="20 50 50"/>
-        </buoyancy>
+        <static>true</static>
     </link>
 </robot>

File: src/freefloating_gazebo_demo/urdf/barco_obs2.xacro (robot description, xacro)
@@ -29,10 +29,10 @@
           <inertia ixx="0.5" ixy="0.0" ixz="0.0" iyy="0.5" iyz="0.0" izz="0.5"/>
         </inertial>
-        <buoyancy>
-            <compensation>1.2</compensation>
-            <origin xyz= "0 0 0"/>
-            <limit radius="0.1"/>
-            <damping xyz="20 50 50" rpy="20 50 50"/>
-        </buoyancy>
+        <static>true</static>
     </link>
+    <joint name="obs2_joint" type="fixed">
+        <origin xyz="0 0 0" rpy="0 0 0" />
+        <parent link="underwater"/>
+        <child link="side_link2"/>
+    </joint>
 </robot>

Commit message: Fixing some stuff

File: src/freefloating_gazebo_demo/urdf/barcoDiferencial.xacro (robot description, xacro)
@@ -62,6 +62,5 @@
                 <origin rpy="0 0 0"/>
                 <geometry>
-<!--		    <mesh filename="file://$(env HOME)/.uwsim/data/robot/barco/pt90.stl"/>-->
-	 		<box size="1.0 0.4 0.2" />
+		    <mesh filename="file://$(env HOME)/.uwsim/data/robot/barco/pt90.stl"/>
                 </geometry>
 		  <material name="blue">

Commit message: Testing Water surface update

File: src/freefloating_gazebo_demo/urdf/barcoDiferencial.xacro (robot description, xacro)
@@ -60,5 +60,5 @@
         <link name="base_link">
             <visual>
-                <origin rpy="0 0 0"/>
+		<origin rpy="${pi/2} 0 ${pi/2}" xyz="0 0 0"/>
                 <geometry>
 		    <mesh filename="file://$(env HOME)/.uwsim/data/robot/barco/pt90.stl"/>
@@ -69,5 +69,5 @@
             </visual>
             <inertial>
-                <origin xyz="0 0 ${X_cog}" rpy="0 0 0"/>
+                <origin xyz="0 0 -0.05" rpy="0 0 0"/>
                 <mass value="${body_mass}"/>
                 <inertia
@@ -80,7 +80,7 @@
                 </inertial>
                 <buoyancy>
-                    <compensation>1.05</compensation>
-                    <origin xyz= "0 0 0"/>
-                    <limit radius="${body_radius}"/>
+                    <compensation>1.5</compensation>
+                    <origin xyz= "0 0 0.05"/>
+                    <limit radius="${2*body_radius}"/>
                     <damping xyz="40 100 100" rpy="20 50 50"/>
                 </buoyancy>

Commit message: Fixing buoyancy

File: src/freefloating_gazebo_demo/urdf/barcoDiferencial.xacro (robot description, xacro)
@@ -80,7 +80,7 @@
                 </inertial>
                 <buoyancy>
-                    <compensation>1.5</compensation>
+                    <compensation>5</compensation>
                     <origin xyz= "0 0 0.05"/>
-                    <limit radius="${2*body_radius}"/>
+                    <limit radius="${body_radius*0.4}"/>
                     <damping xyz="40 100 100" rpy="20 50 50"/>
                 </buoyancy>
@@ -103,6 +103,6 @@
         </gazebo>
     <!-- Define two steering thrusters, with assumed force control in Z-direction -->
-    <xacro:thruster_link name="fwd_left" xyz="-0.52 0.1 0" rpy="0 ${-PI/2} 0"/>
-    <xacro:thruster_link name="fwd_right" xyz="-0.52 -0.1 0" rpy="0 ${-PI/2} 0"/>
+    <!--<xacro:thruster_link name="fwd_left" xyz="-0.52 0.1 0" rpy="0 ${-PI/2} 0"/>-->
+    <!--<xacro:thruster_link name="fwd_right" xyz="-0.52 -0.1 0" rpy="0 ${-PI/2} 0"/>-->
     <xacro:macro name="thruster_dummy_link" params="name xyz rpy">
         <joint name="${name}" type="fixed">
