Commit message: Fixing boat_rudder configuration

File: src/usv_sim/urdf/barcoLeme_master.xacro (robot description, xacro)
@@ -1,5 +1,5 @@
 <?xml version="1.0"?>
 <!-- STL-version of the URDF, used with gazebo for dynamic simulation  -->
-<robot name="barco_auv" xmlns:xacro="http://www.ros.org/wiki/xacro">
+<robot name="boat_rudder_usv" xmlns:xacro="http://www.ros.org/wiki/xacro">
     <xacro:property name="PI" value="3.1415926535897931"/>
     <!-- Body properties -->

File: src/usv_sim/urdf/boat_rudder.xacro (robot description, xacro)
@@ -67,6 +67,13 @@
                     <mesh filename="file://$(env HOME)/.uwsim/data/robot/barco/pt90.stl"/>
                 </geometry>
-                <material name="blue"/>
+                      <material name="blue"/>
             </visual>
+            <collision>
+                <origin rpy="${PI/2} 0 ${PI/2}"/>
+                <geometry>
+                    <mesh filename="file://$(env HOME)/.uwsim/data/robot/barco/pt90.stl"/>
+                </geometry>
+                      <material name="blue"/>
+            </collision>
             <inertial>
                 <origin xyz="0 0 ${X_cog}" rpy="0 ${-PI/2} 0"/>
@@ -91,10 +98,10 @@
 			<mass value="0.05" />
 			<inertia
-			  ixx="0.2708000"
+			  ixx="0.05"
 			  ixy="0.0"
-			  iyy="0.0508"
+			  iyy="0.05"
 			  ixz="0.0"
 			  iyz="0.0"
-			  izz="0.5208"/>
+			  izz="0.005"/>
 		</inertial>
 	      <collision name="collision">
@@ -125,11 +132,13 @@
 		<!--<plugin name="LiftDrag" filename="libliftdragww.so">-->
 			<a0>0</a0>
-			<cla>4.752798721</cla>
-			<cda>0.6417112299</cda>
-			<cma>-1.8</cma>
+			<cla>0.752798721</cla>
+			<cda>0.3417112299</cda>
+			<!--
+			<cma>-1.8</cma> momentum
+			<cma_stall>0</cma_stall>
+			-->
 			<alpha_stall>0.785</alpha_stall>
-			<cla_stall>-3.85</cla_stall>
-			<cda_stall>-0.9233984055</cda_stall>
-			<cma_stall>0</cma_stall>
+			<cla_stall>-0.85</cla_stall>
+			<cda_stall>-0.3233984055</cda_stall>
 			<cp>-0.5 0 0</cp>
 			<area>0.03</area>
@@ -137,5 +146,5 @@
 			<forward>1 0 0</forward>
 			<upward>0 1 0</upward>
-			<link_name>rudder</link_name>
+<link_name>rudder</link_name>
 	      </plugin>
 <plugin name="freefloating_gazebo_control" filename="libfreefloating_gazebo_control.so">
