Commit message: removing rrbot package

File: src/usv_sim/urdf/boat_diff.xacro (robot description, xacro)
@@ -95,5 +95,5 @@
     <origin xyz="0 0 0" rpy="0 0 0"/>
     <geometry>
-    <mesh filename="package://rrbot_description/meshes/hokuyo.dae"/>
+    <mesh filename="package://usv_sim/meshes/hokuyo.dae"/>
     </geometry>
     </visual>

Commit message: boat xacro segregation

File: src/usv_sim/urdf/boat_diff.xacro (robot description, xacro)
@@ -2,142 +2,6 @@
 <!-- STL-version of the URDF, used with gazebo for dynamic simulation  -->
 <robot name="boat_diff" xmlns:xacro="http://www.ros.org/wiki/xacro">
-    <xacro:property name="PI" value="3.1415926535897931"/>
-    <!-- Body properties -->
-    <xacro:property name="body_mass" value="5"/>
-    <xacro:property name="body_radius" value="0.13"/>
-    <xacro:property name="body_length" value="1.0" />
-    <xacro:property name="X_cog" value="${-0.5*body_radius}" />
-    <!-- thrusters -->
-    <xacro:property name="tr1" value=".02" />
-    <xacro:property name="tl1" value=".1" />
-    <xacro:property name="tr2" value=".05" />
-    <xacro:property name="tl2" value=".03" />
-    <xacro:property name="eps" value="0.00000001"/>
-    <!-- Thruster link -->
-    <xacro:macro name="thruster_link" params="name xyz rpy">
-        <joint name="${name}_link" type="revolute">
-            <parent link="base_link"/>
-            <child link="${name}"/>
-            <origin rpy="${rpy}" xyz="${xyz}"/>
-            <dynamics damping="10.0"/>
-            <axis xyz="0 1 0"/>
-            <limit effort="30" velocity="5.0" lower="-${PI/2}" upper="${PI/2}" />
-        </joint>
-        <link name="${name}">
-            <buoyancy><compensation>1.0</compensation></buoyancy>
-            <visual name="${name}_1">
-                <geometry>
-                    <cylinder length="${tl1}" radius="${tr1}"/>
-                </geometry>
-                <material name="black">
-                    <color rgba="0 0 0 1"/>
-                </material>
-            </visual>
-            <visual name="${name}_2">
-                <origin xyz="0 0 ${(tl1+tl2)/2}"/>
-                <geometry>
-                    <cylinder length="${tl2}" radius="${tr2}"/>
-                </geometry>
-                <material name="black">
-                    <color rgba="0 0 0 1"/>
-                </material>
-            </visual>
-            <inertial>
-                <mass value=".1"/>
-                <inertia
-                    ixx=".1"
-                    ixy="0.0"
-                    ixz="0.0"
-                    iyy=".1"
-                    iyz="0.0"
-                    izz=".1"/>
-                </inertial>
-            </link>
-            <gazebo reference="${name}">
-                <material>Gazebo/Black</material>
-            </gazebo>
-    </xacro:macro>
-    <link name="base_link">
-        <visual>
-          <origin rpy="1.57079632679 0 1.57079632679"/>
-          <geometry>
-            <mesh filename="file:///home/lsa/.uwsim/data/robot/barco/pt90.stl"/>
-          </geometry>
-          <material name="blue"/>
-        </visual>
-        <inertial>
-            <origin rpy="0 0 0" xyz="0 0 -0.05"/>
-          <mass value="10"/>
-          <inertia ixx="0.1" ixy="0.0" ixz="0.0" iyy="1.4" iyz="0.0" izz="1.4"/>
-        </inertial>
-        <buoyancy>
-          <compensation>1.2</compensation>
-          <origin xyz="-0.0005 0 0.05"/>
-          <limit radius="0.1"/>
-          <damping rpy="20 50 50" xyz="20 50 50"/>
-        </buoyancy>
-    </link>
-    <joint name="hokuyo_joint" type="fixed">
-    <axis xyz="0 1 0" />
-    <origin xyz="0.6 0 0.1" rpy="0 0 0"/>
-    <parent link="base_link"/>
-    <child link="hokuyo_link"/>
-    </joint>
-    <!-- Hokuyo Laser -->
-    <link name="hokuyo_link">
-    <collision>
-    <origin xyz="0 0 0" rpy="0 0 0"/>
-    <geometry>
-    <box size="0.1 0.1 0.1"/>
-    </geometry>
-    </collision>
-    <visual>
-    <origin xyz="0 0 0" rpy="0 0 0"/>
-    <geometry>
-    <mesh filename="package://usv_sim/meshes/hokuyo.dae"/>
-    </geometry>
-    </visual>
-    <inertial>
-    <mass value="1e-5" />
-    <origin xyz="0 0 0" rpy="0 0 0"/>
-    <inertia ixx="1e-6" ixy="0" ixz="0" iyy="1e-6" iyz="0" izz="1e-6" />
-    </inertial>
-</link>
-    <gazebo reference="hokuyo_link">
-    <sensor type="gpu_ray" name="head_hokuyo_sensor">
-    <pose>0 0 0 0 0 0</pose>
-    <visualize>true</visualize>
-    <update_rate>40</update_rate>
-    <ray>
-    <scan>
-    <horizontal>
-    <samples>720</samples>
-    <resolution>1</resolution>
-    <min_angle>-1.570796</min_angle>
-    <max_angle>1.570796</max_angle>
-    </horizontal>
-    </scan>
-    <range>
-    <min>0.10</min>
-    <max>30.0</max>
-    <resolution>0.01</resolution>
-    </range>
-    <noise>
-    <type>gaussian</type>
-    <!-- Noise parameters based on published spec for Hokuyo laser
-    achieving "+-30mm" accuracy at range < 10m.  A mean of 0.0m and
-    stddev of 0.01m will put 99.7% of samples within 0.03m of the true
-    reading. -->
-    <mean>0.0</mean>
-    <stddev>0.01</stddev>
-    </noise>
-    </ray>
-    <plugin name="gazebo_ros_head_hokuyo_controller" filename="libgazebo_ros_gpu_laser.so">
-    <topicName>/scan</topicName>
-    <frameName>base_laser</frameName>
-    </plugin>
-    </sensor>
-    </gazebo>
-	<!-- Plugin list -->
+    <xacro:include filename="$(find usv_sim)/urdf/boat_common.xacro" />
+    <!-- Plugin list -->
     <gazebo>
         <plugin name="freefloating_gazebo_control" filename="libfreefloating_gazebo_control.so">
@@ -149,8 +13,8 @@
                 <name>fwd_left</name>
             </thruster>
-    <thruster>
-                <effort>30</effort>
-                <name>fwd_right</name>
-            </thruster>
+        <thruster>
+            <effort>30</effort>
+            <name>fwd_right</name>
+        </thruster>
         </plugin>
     </gazebo>
@@ -158,11 +22,3 @@
     <xacro:thruster_link name="fwd_left" xyz="-0.52 0.1 0" rpy="0 ${-PI/2} 0"/>
     <xacro:thruster_link name="fwd_right" xyz="-0.52 -0.1 0" rpy="0 ${-PI/2} 0"/>
-    <xacro:macro name="thruster_dummy_link" params="name xyz rpy">
-        <joint name="${name}" type="fixed">
-            <parent link="base_link"/>
-            <child link="${name}"/>
-            <origin rpy="${rpy}" xyz="${xyz}"/>
-        </joint>
-        <link name="${name}"/>
-    </xacro:macro>
 </robot>
