Commit message: removing useless launch and xacro from usv_sim

File: src/usv_sim/urdf/boat_rudder.xacro (robot description, xacro)
@@ -1,5 +1,5 @@
 <?xml version="1.0"?>
 <!-- STL-version of the URDF, used with gazebo for dynamic simulation  -->
-<robot name="barco_auv" xmlns:xacro="http://www.ros.org/wiki/xacro">
+<robot name="rudder_boat_usv" xmlns:xacro="http://www.ros.org/wiki/xacro">
       <material name="blue">
         <color rgba="0 0 .8 1"/>

File: src/usv_sim/urdf/sailboat.xacro (robot description, xacro)
@@ -1,5 +1,5 @@
 <?xml version="1.0"?>
 <!-- STL-version of the URDF, used with gazebo for dynamic simulation  -->
-<robot name="barco_auv" xmlns:xacro="http://www.ros.org/wiki/xacro">
+<robot name="sailboat" xmlns:xacro="http://www.ros.org/wiki/xacro">
     <xacro:property name="PI" value="3.1415926535897931"/>
     <!-- Body properties -->
@@ -118,7 +118,7 @@
             <limit effort="30" velocity="5" lower="-${PI/2}" upper="${PI/2}" />
         </joint>
-<!-- Plugin list -->
+    <!-- Plugin list -->
         <gazebo>
-            <!-- Gazebo plugin listens to the body-->
+        <!-- Gazebo plugin listens to the body-->
 		<!--<plugin name="LiftDragWW" filename="libLiftDragPlugin.so">-->
 		<plugin name="LiftDrag" filename="libliftdragww.so">
@@ -139,22 +139,21 @@
 <!--			<control_joint_name>rudder_joint</control_joint_name>-->
 <!--			<control_joint_rad_to_cl>4.0</control_joint_rad_to_cl>-->
-	      </plugin>
-<plugin name="freefloating_gazebo_control" filename="libfreefloating_gazebo_control.so">
-                <switchService>switch</switchService>
-                <updateRate>100</updateRate>
-                <link>base_link</link>
-                <!--    these two thrusters are actually orientable, so the map should not be hard-coded
-                        the thruster name is the name of the corresponding link -->
-                <thruster>
-                    <effort>30</effort>
-                    <name>fwd_left</name>
-                </thruster>
+      </plugin>
+        <plugin name="freefloating_gazebo_control" filename="libfreefloating_gazebo_control.so">
+            <switchService>switch</switchService>
+            <updateRate>100</updateRate>
+            <link>base_link</link>
+            <!--  these two thrusters are actually orientable, so the map should not be hard-coded the thruster name is the name of the corresponding link -->
+            <thruster>
+                <effort>30</effort>
+                <name>fwd_left</name>
+            </thruster>
 <thruster>
-                    <effort>30</effort>
-                    <name>fwd_right</name>
-                </thruster>
-                <!-- these thrusters are fixed and the map can be hard-coded
-                     they will be given a name (thr2 to thr4)  -->
-            </plugin>
+                <effort>30</effort>
+                <name>fwd_right</name>
+            </thruster>
+            <!-- these thrusters are fixed and the map can be hard-coded
+                 they will be given a name (thr2 to thr4)  -->
+        </plugin>
         </gazebo>
     <!-- Define two steering thrusters, with assumed force control in Z-direction -->
@@ -173,3 +172,3 @@
     <xacro:thruster_dummy_link name="thr3" xyz="-0.45 0.0 0.0" rpy="0.0 -0.0 0.0"/>
     <xacro:thruster_dummy_link name="thr4" xyz="0.45 0.0 0.0" rpy="0.0 -0.0 0.0"/>-->
-        </robot>
+</robot>
