Commit message: updates

File: src/usv_sim/urdf/boat_differential.xacro (robot description, xacro)
@@ -31,5 +31,5 @@
                 </geometry>
                 <material name="black">
-                    <color rgba="0 0 0 1"/>
+                    <color rgba="0 0 0 0"/>
                 </material>
             </visual>
@@ -40,5 +40,5 @@
                 </geometry>
                 <material name="black">
-                    <color rgba="0 0 0 1"/>
+                    <color rgba="0 0 0 0"/>
                 </material>
             </visual>

File: src/usv_sim/xacro/boat_common_subdivided.xacro (robot description, xacro)
@@ -22,5 +22,5 @@
             <mesh filename="package://usv_sim/meshes/simpleBoat-middle.stl"/>
           </geometry>
-          <material name="blue"/>
+          <material name="white"/>
         </visual>
         <collision>
@@ -48,5 +48,5 @@
             <mesh filename="package://usv_sim/meshes/simpleBoat-back.stl"/>
           </geometry>
-          <material name="blue"/>
+          <material name="white"/>
         </visual>
         <collision>
@@ -82,5 +82,5 @@
             <mesh filename="package://usv_sim/meshes/simpleBoat-front.stl"/>
           </geometry>
-          <material name="blue"/>
+          <material name="white"/>
         </visual>
         <collision>
@@ -127,5 +127,5 @@
                 </geometry>
                 <material name="black">
-                    <color rgba="0 0 0 1"/>
+                    <color rgba="255 255 255 1"/>
                 </material>
             </visual>
@@ -136,5 +136,5 @@
                 </geometry>
                 <material name="black">
-                    <color rgba="0 0 0 1"/>
+                    <color rgba="255 255 255 1"/>
                 </material>
             </visual>
