Commit message: starting to create divided scenarios for each usv

File: src/usv_sim/urdf/boat_rudder_dummy.urdf (robot description, URDF)
Before this commit: robot thrusters, 0 links, 1 joints
Joints:
- joint fwd: limit lower=-30 upper=30 -> lower=-100 upper=100

Commit message: Testing new plugin

File: src/usv_sim/urdf/boat_rudder_dummy.urdf (robot description, URDF)
Before this commit: robot thrusters, 0 links, 1 joints
Joints:
- joint fwd: limit lower=-30 upper=30 -> lower=-300 upper=300

File: src/usv_sim/xacro/boat_rudder.xacro (robot description, xacro)
@@ -6,12 +6,9 @@
     <gazebo>
     <!-- Gazebo plugin listens to the body-->
+	<!--
         <plugin name="rudder_plugin" filename="librudder_plugin.so">
             <a0>0</a0>
             <cla>0.752798721</cla>
             <cda>0.3417112299</cda>
-            <!--
-            <cma>-1.8</cma> momentum
-            <cma_stall>0</cma_stall>
-            -->
             <alpha_stall>0.785</alpha_stall>
             <cla_stall>-0.85</cla_stall>
@@ -24,4 +21,20 @@
             <link_name>rudder</link_name>
         </plugin>
+-->
+	<plugin name="usv_sail_plugin" filename="libusv_sailing_plugin.so">
+		<link_type>rudder</link_type>
+		<a0>0</a0>
+		<cla>0.752798721</cla>
+		<cda>0.3417112299</cda>
+		<alpha_stall>0.785</alpha_stall>
+		<cla_stall>-0.85</cla_stall>
+		<cda_stall>-0.3233984055</cda_stall>
+		<cp>-0.5 0 0</cp>
+		<area>0.06</area>
+		<air_density>1000</air_density>
+		<forward>1 0 0</forward>
+		<upward>0 1 0</upward>
+		<link_name>rudder</link_name>
+	</plugin>
         <plugin name="freefloating_gazebo_control" filename="libfreefloating_gazebo_control.so">
             <switchService>switch</switchService>

File: src/usv_sim/xacro/boat_subdivided4.xacro (robot description, xacro)
@@ -12,10 +12,6 @@
     <xacro:property name="front_water_displaced_mass" value="25"/>
     <xacro:property name="scale" value="0.3"/>
-    <!-- Thruster constants -->
-    <xacro:property name="tr1" value=".02" />
-    <xacro:property name="tl1" value=".1" />
-    <xacro:property name="tr2" value=".05" />
-    <xacro:property name="tl2" value=".03" />
-    <xacro:property name="eps" value="0.00000001"/>
+    <xacro:property name="bl1" value=".1" />
+    <xacro:property name="bl2" value=".1" />
     <link name="base_link">
         <visual>
@@ -232,5 +228,5 @@
           		<origin xyz="0 0 0" rpy="${-0.15*scale} 0 ${0.3*scale}"/>
           		<geometry>
-          		    <mesh filename="package://usv_sim/meshes/simpleHull/thruster.dae" scale="${scale} ${scale} ${scale}"/>
+          		    <mesh filename="package://usv_sim/meshes/simpleHull3/thruster.dae" scale="${scale} ${scale} ${scale}"/>
           		</geometry>
         	</collision>
@@ -238,5 +234,5 @@
                 <origin xyz="0 0 0" rpy="0 0 0" />
                 <geometry>
-                    <mesh filename="package://usv_sim/meshes/simpleHull/thruster.dae" scale="${scale} ${scale} ${scale}"/>
+                    <mesh filename="package://usv_sim/meshes/simpleHull3/thruster.dae" scale="${scale} ${scale} ${scale}"/>
                 </geometry>
                 <material name="black">
@@ -286,5 +282,5 @@
           		<origin xyz="0 0 0" rpy="0 0 0"/>
           		<geometry>
-          			<box size="${tl1} ${tl1} ${tl2}" />
+          			<box size="${bl1} ${bl1} ${bl2}" />
           		</geometry>
         	</collision>
@@ -292,5 +288,5 @@
                 <origin xyz="0 0 0" rpy="0 0 0" />
                 <geometry>
-                    <mesh filename="package://usv_sim/meshes/simpleHull/airPropeller.dae" scale="${scale} ${scale} ${scale}"/>
+                    	<mesh filename="package://usv_sim/meshes/simpleHull/airPropeller.dae" scale="${scale} ${scale} ${scale}"/>
                 </geometry>
             </visual>
@@ -339,8 +335,7 @@
             <visual name="visual">
                 <geometry>
-                  <mesh filename="package://usv_sim/meshes/simpleHull/box.dae" scale="${0.2*scale} ${0.02*scale} ${0.3*scale}"/>
+                  <mesh filename="package://usv_sim/meshes/simpleHull3/box.dae" scale="${0.2*scale} ${0.02*scale} ${0.3*scale}"/>
                 </geometry>
                 <origin rpy="0 0 0" xyz="${-0.1*scale} 0 0"/>
-                <material name="blue"/>
             </visual>
         </link>
@@ -372,7 +367,6 @@
         	<origin xyz="0 0 0" rpy="0 0 0"/>
         	<geometry>
-        		<mesh filename="package://usv_sim/meshes/simpleHull/box.dae" scale="0.1 0.1 0.1"/>
+        		<mesh filename="package://usv_sim/meshes/simpleHull3/box.dae" scale="0.1 0.1 0.1"/>
         	</geometry>
-        	<material name="blue"/>
         </visual>
         <inertial>

File: src/usv_sim/xacro/sailboat.xacro (robot description, xacro)
@@ -6,5 +6,5 @@
     <link name="sail">
 		<inertial>
-		    <origin rpy="0 0 0" xyz="-0.3 0 0.4"/>
+		    	<origin rpy="0 0 0" xyz="-0.3 0 0.4"/>
 			<mass value="0.1" />
 			<inertia
@@ -56,5 +56,5 @@
 	<visual name="visual">
 		<geometry>
-			<mesh filename="package://usv_sim/meshes/simpleHull/box.obj" scale="0.25 0.02 0.5"/>
+			<mesh filename="package://usv_sim/meshes/simpleHull3/box.dae" scale="0.25 0.02 0.5"/>
 		</geometry>
 		<origin rpy="0 0 0" xyz="0 0 0"/>
@@ -72,5 +72,5 @@
   <gazebo>
 	<plugin name="usv_sail_plugin" filename="libusv_sailing_plugin.so">
-		<linkType>sail</linkType>
+		<link_type>sail</link_type>
 		<a0>0</a0>
 		<cla>4.752798721</cla>
@@ -90,5 +90,5 @@
       </plugin>
       <plugin name="usv_sail_plugin" filename="libusv_sailing_plugin.so">
-		  <linkType>keel</linkType>
+		  <link_type>keel</link_type>
 		  <a0>0</a0>
 		  <cla>0.752798721</cla>
@@ -105,5 +105,5 @@
     </plugin>
     <plugin name="usv_sail_plugin" filename="libusv_sailing_plugin.so">
-		<linkType>rudder</linkType>
+		<link_type>rudder</link_type>
 		<a0>0</a0>
 		<cla>0.752798721</cla>
@@ -113,5 +113,5 @@
 		<cda_stall>-0.3233984055</cda_stall>
 		<cp>0 0 0</cp>
-		<area>0.1</area>
+		<area>0.5</area>
 		<air_density>1000</air_density>
 		<forward>1 0 0</forward>
