Commit message: Added usv_wind_current

File: src/usv_sim/urdf/sailboat_dummy.urdf (robot description, URDF)
Before this commit: robot thrusters, 0 links, 2 joints
Joints:
- removed joint fwd_left
- removed joint fwd_right

File: src/usv_sim/xacro/buoy.xacro (robot description, xacro)
@@ -3,5 +3,5 @@
   <link name="link">
     <visual>
-      <origin rpy="0 0 0" xyz="0 0 0"/>
+      <origin rpy="0 0 0" xyz="0 0 0.25"/>
       <geometry>
           <mesh filename="package://usv_sim/meshes/buoy.dae"/>
@@ -9,10 +9,10 @@
     </visual>
     <inertial>
-      <origin rpy="0 0 0" xyz="0 0 0"/>
-      <mass value="4.0"/>
+      <origin rpy="0 0 0" xyz="0 0 0.25"/>
+      <mass value="1.0"/>
       <inertia ixx="1" ixy="0.0" ixz="0.0" iyy="1" iyz="0" izz="1"/>
     </inertial>
     <collision>
-      <origin xyz="0 0 0" rpy="0 0 0"/>
+      <origin xyz="0 0 0" rpy="0 0 0.25"/>
      <geometry>
           <mesh filename="package://usv_sim/meshes/buoy.dae"/>
@@ -20,9 +20,9 @@
     </collision>
 		<buoyancy>
-        	<compensation>62</compensation>
-          	<origin xyz="0 0 0"/>
-          	<limit radius="0.5"/>
-          	<damping rpy="20 20 20" xyz="20 40 50"/>
-	  	  	<fluidVelocity>local</fluidVelocity>
+        	<compensation>10</compensation>
+          	<origin xyz="0 0 0.3"/>
+          	<limit radius="0.25"/>
+          	<damping rpy="20 20 20" xyz="100 100 50"/>
+	  	  	<fluidVelocity>none</fluidVelocity>
         </buoyancy>
   </link>

File: src/usv_sim/xacro/sailboat.xacro (robot description, xacro)
@@ -88,4 +88,5 @@
 		<upward>0 1 0</upward>
 		<link_name>sail</link_name>
+		<fluidVelocity>local</fluidVelocity>
       </plugin>
       <plugin name="usv_sail_plugin" filename="libusv_sailing_plugin.so">
@@ -103,4 +104,5 @@
 		  <upward>0 1 0</upward>
 		  <link_name>keel</link_name>
+		  <fluidVelocity>local</fluidVelocity>
     </plugin>
     <plugin name="usv_sail_plugin" filename="libusv_sailing_plugin.so">
@@ -118,4 +120,5 @@
 		<upward>0 1 0</upward>
 		<link_name>rudder</link_name>
+		<fluidVelocity>local</fluidVelocity>
       </plugin>
       <plugin name="freefloating_gazebo_control" filename="libfreefloating_gazebo_control.so">
