Commit message: Added a bridge at diluvio and changed boats center of mass

File: src/usv_sim/urdf/boat_diff_dummy.urdf (robot description, URDF)
Before this commit: robot thrusters, 0 links, 2 joints
Joints:
- joint fwd_left: limit lower=-30 upper=30 -> lower=-100 upper=100
- joint fwd_right: limit lower=-30.0 upper=30.0 -> lower=-100.0 upper=100.0

File: src/usv_sim/xacro/boat_diff.xacro (robot description, xacro)
@@ -9,9 +9,9 @@
             <link>fwd_left</link>
             <thruster>
-                <effort>30</effort>
+                <effort>100</effort>
                 <name>fwd_left</name>
             </thruster>
    	    <thruster>
-	        <effort>30</effort>
+	        <effort>100</effort>
 	        <name>fwd_right</name>
 	    </thruster>

File: src/usv_sim/xacro/boat_subdivided3.xacro (robot description, xacro)
@@ -3,5 +3,5 @@
     <xacro:property name="PI" value="3.1415926535897931"/>
     <!-- Body properties -->
-    <xacro:property name="front_body_mass" value="15"/>
+    <xacro:property name="front_body_mass" value="5"/>
     <xacro:property name="back_body_mass" value="15"/>
     <xacro:property name="middle_body_mass" value="10"/>
@@ -9,5 +9,5 @@
     <xacro:property name="front_body_mass" value="2"/>
     <xacro:property name="back_water_displaced_mass" value="40"/>
-    <xacro:property name="middle_water_displaced_mass" value="60"/>
+    <xacro:property name="middle_water_displaced_mass" value="40"/>
     <xacro:property name="front_water_displaced_mass" value="25"/>
     <xacro:property name="scale" value="0.3"/>
@@ -226,9 +226,9 @@
         <link name="${name}">
             <buoyancy>
-				<compensation>1.0</compensation>
+				<compensation>0.8</compensation>
 	        	<fluidVelocity>local</fluidVelocity>
 	    	</buoyancy>
 	    	<collision>
-          		<origin xyz="0 0 0" rpy="0 0 0"/>
+          		<origin xyz="0 0 0" rpy="{-0.15*scale} 0 ${0.3*scale}"/>
           		<geometry>
           		    <mesh filename="package://usv_sim/meshes/simpleHull/thruster.obj" scale="${scale} ${scale} ${scale}"/>
@@ -246,5 +246,5 @@
             <inertial>
                 <mass value="5"/>
-                <origin xyz="${0.2*scale} 0 ${0.2*scale}" rpy="0 0 0" />
+                <origin xyz="${-0.2*scale} 0 ${0.3*scale}" rpy="0 0 0" />
                 <inertia
                     ixx=".1"

Commit message: preparing for merge

File: src/usv_sim/urdf/boat_diff_dummy.urdf (robot description, URDF)
Before this commit: robot thrusters, 0 links, 2 joints
Joints:
- joint fwd_left: limit lower=-100 upper=100 -> lower=-300 upper=300
- joint fwd_right: limit lower=-100.0 upper=100.0 -> lower=-300.0 upper=300.0
