Commit message: reorganizing usv_sim launch and xacros

File: src/usv_sim/xacro/boat_common.xacro (robot description, xacro)
@@ -17,5 +17,5 @@
       <origin rpy="1.57079632679 0 1.57079632679"/>
       <geometry>
-        <mesh filename="file:///home/lsa/.uwsim/data/robot/barco/pt90.stl"/>
+        <mesh filename="package://usv_sim/meshes/pt90.stl"/>
       </geometry>
       <material name="blue"/>
@@ -85,4 +85,39 @@
     <link name="${name}"/>
 </xacro:macro>
+<!-- Rudder link -->
+<xacro:macro name="rudder_xacro">
+        <link name="rudder">
+            <inertial>
+                <mass value="0.05" />
+                <inertia
+                  ixx="0.05"
+                  ixy="0.0"
+                  iyy="0.05"
+                  ixz="0.0"
+                  iyz="0.0"
+                  izz="0.005"/>
+            </inertial>
+            <collision name="collision">
+                <geometry>
+                  <box size="0.1 0.02 0.3" />
+                </geometry>
+                <origin rpy="0 0 0" xyz="-0.1 0 0"/>
+            </collision>
+            <visual name="visual">
+                <geometry>
+                  <box size="0.1 0.02 0.3" />
+                </geometry>
+                <origin rpy="0 0 0" xyz="-0.1 0 0"/>
+            </visual>
+        </link>
+        <joint name="rudder_joint" type="revolute">
+            <parent link="base_link"/>
+            <child link="rudder"/>
+            <origin rpy="0 0 0" xyz="-0.53 0 -0.1"/>
+            <dynamics damping="1.0"/>
+            <axis xyz="0 0 1"/>
+            <limit effort="50" velocity="5" lower="-${PI/3}" upper="${PI/3}" />
+        </joint>
+</xacro:macro>
 <!-- Sensors -->
 <!-- Hokuyo Laser -->

File: src/usv_sim/xacro/boat_diff.xacro (robot description, xacro)
@@ -1,7 +1,6 @@
 <?xml version="1.0"?>
-<!-- STL-version of the URDF, used with gazebo for dynamic simulation  -->
 <robot name="boat_diff" xmlns:xacro="http://www.ros.org/wiki/xacro">
-    <xacro:include filename="$(find usv_sim)/urdf/boat_common.xacro" />
-    <!-- Plugin list -->
+<xacro:include filename="$(find usv_sim)/xacro/boat_common.xacro" />
+<!-- Plugin list -->
     <gazebo>
         <plugin name="freefloating_gazebo_control" filename="libfreefloating_gazebo_control.so">

Commit message: adding launch to initialize multiple robots

File: src/usv_sim/xacro/boat_common.xacro (robot description, xacro)
@@ -1,90 +1,90 @@
 <?xml version="1.0"?>
 <xacro xmlns:xacro="http://www.ros.org/wiki/xacro">
-<xacro:property name="PI" value="3.1415926535897931"/>
-<!-- Body properties -->
-<xacro:property name="body_mass" value="5"/>
-<xacro:property name="body_radius" value="0.13"/>
-<xacro:property name="body_length" value="1.0" />
-<xacro:property name="X_cog" value="${-0.5*body_radius}" />
-<!-- Thruster constants -->
-<xacro:property name="tr1" value=".02" />
-<xacro:property name="tl1" value=".1" />
-<xacro:property name="tr2" value=".05" />
-<xacro:property name="tl2" value=".03" />
-<xacro:property name="eps" value="0.00000001"/>
-<link name="base_link">
-    <visual>
-      <origin rpy="1.57079632679 0 1.57079632679"/>
-      <geometry>
-        <mesh filename="package://usv_sim/meshes/pt90.stl"/>
-      </geometry>
-      <material name="blue"/>
-    </visual>
-    <inertial>
-        <origin rpy="0 0 0" xyz="0 0 -0.05"/>
-      <mass value="10"/>
-      <inertia ixx="0.1" ixy="0.0" ixz="0.0" iyy="1.4" iyz="0.0" izz="1.4"/>
-    </inertial>
-    <buoyancy>
-      <compensation>1.2</compensation>
-      <origin xyz="-0.0005 0 0.05"/>
-      <limit radius="0.1"/>
-      <damping rpy="20 50 50" xyz="20 50 50"/>
-    </buoyancy>
-</link>
-<!-- Thruster link -->
-<xacro:macro name="thruster_link" params="name xyz rpy">
-    <joint name="${name}_link" type="revolute">
-        <parent link="base_link"/>
-        <child link="${name}"/>
-        <origin rpy="${rpy}" xyz="${xyz}"/>
-        <dynamics damping="10.0"/>
-        <axis xyz="0 1 0"/>
-        <limit effort="30" velocity="5.0" lower="-${PI/2}" upper="${PI/2}" />
-    </joint>
-    <link name="${name}">
-        <buoyancy><compensation>1.0</compensation></buoyancy>
-        <visual name="${name}_1">
-            <geometry>
-                <cylinder length="${tl1}" radius="${tr1}"/>
-            </geometry>
-            <material name="black">
-                <color rgba="0 0 0 1"/>
-            </material>
-        </visual>
-        <visual name="${name}_2">
-            <origin xyz="0 0 ${(tl1+tl2)/2}"/>
-            <geometry>
-                <cylinder length="${tl2}" radius="${tr2}"/>
-            </geometry>
-            <material name="black">
-                <color rgba="0 0 0 1"/>
-            </material>
+    <xacro:property name="PI" value="3.1415926535897931"/>
+    <!-- Body properties -->
+    <xacro:property name="body_mass" value="5"/>
+    <xacro:property name="body_radius" value="0.13"/>
+    <xacro:property name="body_length" value="1.0" />
+    <xacro:property name="X_cog" value="${-0.5*body_radius}" />
+    <!-- Thruster constants -->
+    <xacro:property name="tr1" value=".02" />
+    <xacro:property name="tl1" value=".1" />
+    <xacro:property name="tr2" value=".05" />
+    <xacro:property name="tl2" value=".03" />
+    <xacro:property name="eps" value="0.00000001"/>
+    <link name="base_link">
+        <visual>
+          <origin rpy="1.57079632679 0 1.57079632679"/>
+          <geometry>
+            <mesh filename="package://usv_sim/meshes/pt90.stl"/>
+          </geometry>
+          <material name="blue"/>
         </visual>
         <inertial>
-            <mass value=".1"/>
-            <inertia
-                ixx=".1"
-                ixy="0.0"
-                ixz="0.0"
-                iyy=".1"
-                iyz="0.0"
-                izz=".1"/>
+            <origin rpy="0 0 0" xyz="0 0 -0.05"/>
+          <mass value="10"/>
+          <inertia ixx="0.1" ixy="0.0" ixz="0.0" iyy="1.4" iyz="0.0" izz="1.4"/>
         </inertial>
+        <buoyancy>
+          <compensation>1.2</compensation>
+          <origin xyz="-0.0005 0 0.05"/>
+          <limit radius="0.1"/>
+          <damping rpy="20 50 50" xyz="20 50 50"/>
+        </buoyancy>
     </link>
-    <gazebo reference="${name}">
-        <material>Gazebo/Black</material>
-    </gazebo>
-</xacro:macro>
-<xacro:macro name="thruster_dummy_link" params="name xyz rpy">
-    <joint name="${name}" type="fixed">
-        <parent link="base_link"/>
-        <child link="${name}"/>
-        <origin rpy="${rpy}" xyz="${xyz}"/>
-    </joint>
-    <link name="${name}"/>
-</xacro:macro>
-<!-- Rudder link -->
-<xacro:macro name="rudder_xacro">
+    <!-- Thruster link -->
+    <xacro:macro name="thruster_link" params="name xyz rpy">
+        <joint name="${name}_link" type="revolute">
+            <parent link="base_link"/>
+            <child link="${name}"/>
+            <origin rpy="${rpy}" xyz="${xyz}"/>
+            <dynamics damping="10.0"/>
+            <axis xyz="0 1 0"/>
+            <limit effort="30" velocity="5.0" lower="-${PI/2}" upper="${PI/2}" />
+        </joint>
+        <link name="${name}">
+            <buoyancy><compensation>1.0</compensation></buoyancy>
+            <visual name="${name}_1">
+                <geometry>
+                    <cylinder length="${tl1}" radius="${tr1}"/>
+                </geometry>
+                <material name="black">
+                    <color rgba="0 0 0 1"/>
+                </material>
+            </visual>
+            <visual name="${name}_2">
+                <origin xyz="0 0 ${(tl1+tl2)/2}"/>
+                <geometry>
+                    <cylinder length="${tl2}" radius="${tr2}"/>
+                </geometry>
+                <material name="black">
+                    <color rgba="0 0 0 1"/>
+                </material>
+            </visual>
+            <inertial>
+                <mass value=".1"/>
+                <inertia
+                    ixx=".1"
+                    ixy="0.0"
+                    ixz="0.0"
+                    iyy=".1"
+                    iyz="0.0"
+                    izz=".1"/>
+            </inertial>
+        </link>
+        <gazebo reference="${name}">
+            <material>Gazebo/Black</material>
+        </gazebo>
+    </xacro:macro>
+    <xacro:macro name="thruster_dummy_link" params="name xyz rpy">
+        <joint name="${name}" type="fixed">
+            <parent link="base_link"/>
+            <child link="${name}"/>
+            <origin rpy="${rpy}" xyz="${xyz}"/>
+        </joint>
+        <link name="${name}"/>
+    </xacro:macro>
+    <!-- Rudder link -->
+    <xacro:macro name="rudder_xacro">
         <link name="rudder">
             <inertial>
@@ -119,66 +119,66 @@
             <limit effort="50" velocity="5" lower="-${PI/3}" upper="${PI/3}" />
         </joint>
-</xacro:macro>
-<!-- Sensors -->
-<!-- Hokuyo Laser -->
-<joint name="hokuyo_joint" type="fixed">
-    <axis xyz="0 1 0" />
-    <origin xyz="0.6 0 0.1" rpy="0 0 0"/>
-    <parent link="base_link"/>
-    <child link="hokuyo_link"/>
-</joint>
-<link name="hokuyo_link">
-    <collision>
-    <origin xyz="0 0 0" rpy="0 0 0"/>
-    <geometry>
-    <box size="0.1 0.1 0.1"/>
-    </geometry>
-    </collision>
-    <visual>
-    <origin xyz="0 0 0" rpy="0 0 0"/>
-    <geometry>
-    <mesh filename="package://usv_sim/meshes/hokuyo.dae"/>
-    </geometry>
-    </visual>
-    <inertial>
-    <mass value="1e-5" />
-    <origin xyz="0 0 0" rpy="0 0 0"/>
-    <inertia ixx="1e-6" ixy="0" ixz="0" iyy="1e-6" iyz="0" izz="1e-6" />
-    </inertial>
-</link>
-<gazebo reference="hokuyo_link">
-    <sensor type="gpu_ray" name="head_hokuyo_sensor">
-    <pose>0 0 0 0 0 0</pose>
-    <visualize>true</visualize>
-    <update_rate>40</update_rate>
-    <ray>
-    <scan>
-    <horizontal>
-    <samples>720</samples>
-    <resolution>1</resolution>
-    <min_angle>-1.570796</min_angle>
-    <max_angle>1.570796</max_angle>
-    </horizontal>
-    </scan>
-    <range>
-    <min>0.10</min>
-    <max>30.0</max>
-    <resolution>0.01</resolution>
-    </range>
-    <noise>
-    <type>gaussian</type>
-    <!-- Noise parameters based on published spec for Hokuyo laser
-    achieving "+-30mm" accuracy at range < 10m.  A mean of 0.0m and
-    stddev of 0.01m will put 99.7% of samples within 0.03m of the true
-    reading. -->
-    <mean>0.0</mean>
-    <stddev>0.01</stddev>
-    </noise>
-    </ray>
-    <plugin name="gazebo_ros_head_hokuyo_controller" filename="libgazebo_ros_gpu_laser.so">
-    <topicName>/scan</topicName>
-    <frameName>base_laser</frameName>
-    </plugin>
-    </sensor>
-</gazebo>
+    </xacro:macro>
+    <!-- Sensors -->
+    <!-- Hokuyo Laser -->
+    <joint name="hokuyo_joint" type="fixed">
+        <axis xyz="0 1 0" />
+        <origin xyz="0.6 0 0.1" rpy="0 0 0"/>
+        <parent link="base_link"/>
+        <child link="hokuyo_link"/>
+    </joint>
+    <link name="hokuyo_link">
+        <collision>
+        <origin xyz="0 0 0" rpy="0 0 0"/>
+        <geometry>
+        <box size="0.1 0.1 0.1"/>
+        </geometry>
+        </collision>
+        <visual>
+        <origin xyz="0 0 0" rpy="0 0 0"/>
+        <geometry>
+        <mesh filename="package://usv_sim/meshes/hokuyo.dae"/>
+        </geometry>
+        </visual>
+        <inertial>
+        <mass value="1e-5" />
+        <origin xyz="0 0 0" rpy="0 0 0"/>
+        <inertia ixx="1e-6" ixy="0" ixz="0" iyy="1e-6" iyz="0" izz="1e-6" />
+        </inertial>
+    </link>
+    <gazebo reference="hokuyo_link">
+        <sensor type="gpu_ray" name="head_hokuyo_sensor">
+        <pose>0 0 0 0 0 0</pose>
+        <visualize>true</visualize>
+        <update_rate>40</update_rate>
+        <ray>
+        <scan>
+        <horizontal>
+        <samples>720</samples>
+        <resolution>1</resolution>
+        <min_angle>-1.570796</min_angle>
+        <max_angle>1.570796</max_angle>
+        </horizontal>
+        </scan>
+        <range>
+        <min>0.10</min>
+        <max>30.0</max>
+        <resolution>0.01</resolution>
+        </range>
+        <noise>
+        <type>gaussian</type>
+        <!-- Noise parameters based on published spec for Hokuyo laser
+        achieving "+-30mm" accuracy at range < 10m.  A mean of 0.0m and
+        stddev of 0.01m will put 99.7% of samples within 0.03m of the true
+        reading. -->
+        <mean>0.0</mean>
+        <stddev>0.01</stddev>
+        </noise>
+        </ray>
+        <plugin name="gazebo_ros_head_hokuyo_controller" filename="libgazebo_ros_gpu_laser.so">
+        <topicName>/scan</topicName>
+        <frameName>base_laser</frameName>
+        </plugin>
+        </sensor>
+    </gazebo>
 </xacro>

File: src/usv_sim/xacro/boat_diff.xacro (robot description, xacro)
@@ -1,6 +1,6 @@
 <?xml version="1.0"?>
 <robot name="boat_diff" xmlns:xacro="http://www.ros.org/wiki/xacro">
-<xacro:include filename="$(find usv_sim)/xacro/boat_common.xacro" />
-<!-- Plugin list -->
+    <xacro:include filename="$(find usv_sim)/xacro/boat_common.xacro" />
+    <!-- Plugin list -->
     <gazebo>
         <plugin name="freefloating_gazebo_control" filename="libfreefloating_gazebo_control.so">

File: src/usv_sim/xacro/sailboat.xacro (robot description, xacro)
@@ -2,4 +2,6 @@
 <robot name="sailboat" xmlns:xacro="http://www.ros.org/wiki/xacro">
     <xacro:include filename="$(find usv_sim)/xacro/boat_common.xacro" />
+    <xacro:rudder_xacro/>
+    <!-- Defining sail model -->
     <link name="sail">
 		<inertial>
@@ -36,24 +38,22 @@
     <!-- Plugin list -->
     <gazebo>
-    <!-- Gazebo plugin listens to the body-->
-    <!--<plugin name="LiftDragWW" filename="libLiftDragPlugin.so">-->
-    <plugin name="LiftDrag" filename="libliftdragww.so">
-        <a0>0</a0>
-        <cla>2.752798721</cla>
-        <cda>2.6417112299</cda>
-        <cma>-1.8</cma>
-        <alpha_stall>0.785</alpha_stall>
-        <cla_stall>-3.85</cla_stall>
-        <cda_stall>-0.9233984055</cda_stall>
-        <cma_stall>0</cma_stall>
-        <cp>0 0 0</cp>
-        <area>0.4</area>
-        <air_density>1.2041</air_density>
-        <forward>1 0 0</forward>
-        <upward>0 1 0</upward>
-        <link_name>sail</link_name>
-        <!--<control_joint_name>rudder_joint</control_joint_name>-->
-        <!--<control_joint_rad_to_cl>4.0</control_joint_rad_to_cl>-->
-  </plugin>
+        <plugin name="LiftDrag" filename="libliftdragww.so">
+            <a0>0</a0>
+            <cla>2.752798721</cla>
+            <cda>2.6417112299</cda>
+            <cma>-1.8</cma>
+            <alpha_stall>0.785</alpha_stall>
+            <cla_stall>-3.85</cla_stall>
+            <cda_stall>-0.9233984055</cda_stall>
+            <cma_stall>0</cma_stall>
+            <cp>0 0 0</cp>
+            <area>0.4</area>
+            <air_density>1.2041</air_density>
+            <forward>1 0 0</forward>
+            <upward>0 1 0</upward>
+            <link_name>sail</link_name>
+            <!--<control_joint_name>rudder_joint</control_joint_name>-->
+            <!--<control_joint_rad_to_cl>4.0</control_joint_rad_to_cl>-->
+      </plugin>
   </gazebo>
 </robot>

Commit message: multiple differential boats working. launch is diff_start_world.launch

File: src/usv_sim/xacro/boat_common.xacro (robot description, xacro)
@@ -21,4 +21,10 @@
           <material name="blue"/>
         </visual>
+        <collision>
+          <origin rpy="1.57079632679 0 1.57079632679"/>
+          <geometry>
+            <mesh filename="package://usv_sim/meshes/pt90.stl"/>
+          </geometry>
+        </collision>
         <inertial>
             <origin rpy="0 0 0" xyz="0 0 -0.05"/>
@@ -177,5 +183,5 @@
         </ray>
         <plugin name="gazebo_ros_head_hokuyo_controller" filename="libgazebo_ros_gpu_laser.so">
-        <topicName>/scan</topicName>
+        <topicName>scan</topicName>
         <frameName>base_laser</frameName>
         </plugin>

Commit message: obstacle avoidance config improved

File: src/usv_sim/xacro/boat_common.xacro (robot description, xacro)
@@ -130,5 +130,5 @@
     <joint name="hokuyo_joint" type="fixed">
         <axis xyz="0 1 0" />
-        <origin xyz="0.6 0 0.1" rpy="0 0 0"/>
+        <origin xyz="0.7 0 0" rpy="0 0 0"/>
         <parent link="base_link"/>
         <child link="hokuyo_link"/>

Commit message: Sail plugin added

File: src/usv_sim/xacro/boat_common.xacro (robot description, xacro)
@@ -33,8 +33,8 @@
         </inertial>
         <buoyancy>
-          <compensation>1.2</compensation>
+          <compensation>5</compensation>
           <origin xyz="-0.0005 0 0.05"/>
           <limit radius="0.1"/>
-          <damping rpy="20 50 50" xyz="20 50 50"/>
+          <damping rpy="20 500 50" xyz="20 50 50"/>
         </buoyancy>
     </link>
@@ -144,5 +144,5 @@
         <origin xyz="0 0 0" rpy="0 0 0"/>
         <geometry>
-        <mesh filename="package://usv_sim/meshes/hokuyo.dae"/>
+        <mesh filename="package://usv_sim/meshes/hokuyo.stl"/>
         </geometry>
         </visual>

File: src/usv_sim/xacro/sailboat.xacro (robot description, xacro)
@@ -38,5 +38,5 @@
     <!-- Plugin list -->
     <gazebo>
-        <plugin name="LiftDrag" filename="libliftdragww.so">
+        <plugin name="sail_plugin" filename="libsail_plugin.so">
             <a0>0</a0>
             <cla>2.752798721</cla>
