Commit message: Added sail plugin and sailboat model

File: src/usv_sim/xacro/boat_common_subdivided.xacro (robot description, xacro)
@@ -3,8 +3,11 @@
     <xacro:property name="PI" value="3.1415926535897931"/>
     <!-- Body properties -->
-    <xacro:property name="body_mass" value="5"/>
-    <xacro:property name="body_radius" value="0.13"/>
-    <xacro:property name="body_length" value="1.0" />
-    <xacro:property name="X_cog" value="${-0.5*body_radius}" />
+    <xacro:property name="back_body_mass" value="5"/>
+    <xacro:property name="middle_body_mass" value="5"/>
+    <xacro:property name="rear_body_mass" value="5"/>
+    <xacro:property name="front_body_mass" value="2"/>
+    <xacro:property name="back_water_displaced_mass" value="60"/>
+    <xacro:property name="middle_water_displaced_mass" value="60"/>
+    <xacro:property name="front_water_displaced_mass" value="25"/>
     <!-- Thruster constants -->
     <xacro:property name="tr1" value=".02" />
@@ -15,23 +18,23 @@
     <link name="base_link">
         <visual>
-          <origin rpy="1.57079632679 0 1.57079632679"/>
-          <geometry>
-            <mesh filename="package://usv_sim/meshes/pt90.stl"/>
+          <origin rpy="0 0 0"/>
+          <geometry>
+            <mesh filename="package://usv_sim/meshes/simpleBoat-middle.stl"/>
           </geometry>
           <material name="blue"/>
         </visual>
         <collision>
-          <origin rpy="1.57079632679 0 1.57079632679"/>
-          <geometry>
-            <mesh filename="package://usv_sim/meshes/pt90.stl"/>
+          <origin rpy="0 0 0"/>
+          <geometry>
+            <mesh filename="package://usv_sim/meshes/simpleBoat-middle.stl"/>
           </geometry>
         </collision>
         <inertial>
             <origin rpy="0 0 0" xyz="0 0 -0.05"/>
-          <mass value="10"/>
+          <mass value="${middle_body_mass}"/>
           <inertia ixx="0.1" ixy="0.0" ixz="0.0" iyy="1.4" iyz="0.0" izz="1.4"/>
         </inertial>
         <buoyancy>
-          <compensation>5</compensation>
+          <compensation>${middle_water_displaced_mass/middle_body_mass}</compensation>
           <origin xyz="0 0 0.05"/>
           <limit radius="0.1"/>
@@ -39,4 +42,72 @@
         </buoyancy>
     </link>
+    <link name="back_link">
+        <visual>
+          <origin rpy="0 0 0" xyz="-0.25 0 0"/>
+          <geometry>
+            <mesh filename="package://usv_sim/meshes/simpleBoat-back.stl"/>
+          </geometry>
+          <material name="blue"/>
+        </visual>
+        <collision>
+          <origin rpy="0 0 0"  xyz="-0.25 0 0"/>
+          <geometry>
+            <mesh filename="package://usv_sim/meshes/simpleBoat-back.stl"/>
+          </geometry>
+        </collision>
+        <inertial>
+            <origin rpy="0 0 0" xyz="-0.25 0 -0.05"/>
+          <mass value="${back_body_mass}"/>
+          <inertia ixx="0.1" ixy="0.0" ixz="0.0" iyy="1.4" iyz="0.0" izz="1.4"/>
+        </inertial>
+        <buoyancy>
+          <compensation>${back_water_displaced_mass/back_body_mass}</compensation>
+          <origin xyz="0 0 0.05"/>
+          <limit radius="0.1"/>
+          <damping rpy="20 500 50" xyz="20 50 50"/>
+        </buoyancy>
+    </link>
+    <joint name="back_joint" type="revolute">
+        <parent link="base_link"/>
+        <child link="back_link"/>
+        <origin rpy="0 0 0" xyz="-0.25 0 0"/>
+	<limit effort="50" velocity="5" lower="0" upper="0" />
+            <dynamics damping="1.0"/>
+            <axis xyz="1 0 0"/>
+    </joint>
+    <link name="front_link">
+        <visual>
+          <origin rpy="0 0 0" xyz="0.25 0 0"/>
+          <geometry>
+            <mesh filename="package://usv_sim/meshes/simpleBoat-front.stl"/>
+          </geometry>
+          <material name="blue"/>
+        </visual>
+        <collision>
+          <origin rpy="0 0 0" xyz="0.25 0 0"/>
+          <geometry>
+            <mesh filename="package://usv_sim/meshes/simpleBoat-front.stl"/>
+          </geometry>
+        </collision>
+        <inertial>
+            <origin rpy="0 0 0" xyz="0.25 0 -0.05"/>
+          <mass value="${front_body_mass}"/>
+          <inertia ixx="0.1" ixy="0.0" ixz="0.0" iyy="1.4" iyz="0.0" izz="1.4"/>
+        </inertial>
+        <buoyancy>
+          <compensation>${front_water_displaced_mass/front_body_mass}</compensation>
+          <origin xyz="0 0 0.05"/>
+          <limit radius="0.1"/>
+          <damping rpy="20 500 50" xyz="20 50 50"/>
+        </buoyancy>
+    </link>
+    <joint name="front_joint" type="revolute">
+        <parent link="base_link"/>
+        <child link="front_link"/>
+        <origin rpy="0 0 0" xyz="0.25 0 0"/>
+	<limit effort="50" velocity="5" lower="0" upper="0" />
+            <dynamics damping="1.0"/>
+            <axis xyz="1 0 0"/>
+    </joint>
     <!-- Thruster link -->
     <xacro:macro name="thruster_link" params="name xyz rpy">

File: src/usv_sim/xacro/boat_rudder.xacro (robot description, xacro)
@@ -7,5 +7,4 @@
     <!-- Gazebo plugin listens to the body-->
         <plugin name="rudder_plugin" filename="librudder_plugin.so">
-    <!--<plugin name="liftdragww" filename="libliftdragww.so"> -->
             <a0>0</a0>
             <cla>0.752798721</cla>

File: src/usv_sim/xacro/sailboat.xacro (robot description, xacro)
@@ -1,5 +1,5 @@
 <?xml version="1.0"?>
 <robot name="sailboat" xmlns:xacro="http://www.ros.org/wiki/xacro">
-    <xacro:include filename="$(find usv_sim)/xacro/boat_common.xacro" />
+    <xacro:include filename="$(find usv_sim)/xacro/boat_common_subdivided.xacro" />
     <xacro:rudder_xacro/>
     <!-- Defining sail model -->
@@ -56,4 +56,27 @@
             <!--<control_joint_rad_to_cl>4.0</control_joint_rad_to_cl>-->
       </plugin>
+        <plugin name="rudder_plugin" filename="librudder_plugin.so">
+            <a0>0</a0>
+            <cla>0.752798721</cla>
+            <cda>0.3417112299</cda>
+            <!--
+            <cma>-1.8</cma> momentum
+            <cma_stall>0</cma_stall>
+            -->
+            <alpha_stall>0.785</alpha_stall>
+            <cla_stall>-0.85</cla_stall>
+            <cda_stall>-0.3233984055</cda_stall>
+            <cp>-0.5 0 0</cp>
+            <area>0.03</area>
+            <air_density>1000</air_density>
+            <forward>1 0 0</forward>
+            <upward>0 1 0</upward>
+            <link_name>rudder</link_name>
+        </plugin>
+        <plugin name="freefloating_gazebo_control" filename="libfreefloating_gazebo_control.so">
+            <switchService>switch</switchService>
+            <updateRate>100</updateRate>
+            <link>base_link</link>
+        </plugin>
   </gazebo>
 </robot>

Commit message: Changed configuration of sailboat.xacro

File: src/usv_sim/xacro/boat_common_subdivided.xacro (robot description, xacro)
@@ -111,5 +111,5 @@
     </joint>
     <!-- Thruster link -->
-    <xacro:macro name="thruster_link" params="name xyz rpy">
+    <xacro:macro name="thruster_link" params="name xyz rpy rotationAxis lowerLimit upperLimit">
         <joint name="${name}_link" type="revolute">
             <parent link="base_link"/>
@@ -117,6 +117,6 @@
             <origin rpy="${rpy}" xyz="${xyz}"/>
             <dynamics damping="10.0"/>
-            <axis xyz="0 1 0"/>
-            <limit effort="30" velocity="5.0" lower="-${PI/2}" upper="${PI/2}" />
+            <axis xyz="${rotationAxis}"/>
+            <limit effort="30" velocity="5.0" lower="${lowerLimit}" upper="${upperLimit}" />
         </joint>
         <link name="${name}">

File: src/usv_sim/xacro/boat_diff.xacro (robot description, xacro)
@@ -19,5 +19,5 @@
     </gazebo>
     <!-- Define two steering thrusters, with assumed force control in Z-direction -->
-    <xacro:thruster_link name="fwd_left" xyz="-0.52 0.1 0" rpy="0 ${-PI/2} 0"/>
-    <xacro:thruster_link name="fwd_right" xyz="-0.52 -0.1 0" rpy="0 ${-PI/2} 0"/>
+    <xacro:thruster_link name="fwd_left" xyz="-0.52 0.1 0" rpy="0 ${-PI/2} 0" rotationAxis="0 1 0" lowerLimit="-${PI/2}" upperLimit="${PI/2}"/>
+    <xacro:thruster_link name="fwd_right" xyz="-0.52 -0.1 0" rpy="0 ${-PI/2} 0" rotationAxis="0 1 0" lowerLimit="-${PI/2}" upperLimit="${PI/2}"/>
 </robot>

File: src/usv_sim/xacro/boat_rudder.xacro (robot description, xacro)
@@ -35,4 +35,4 @@
     </gazebo>
     <!-- Define two steering thrusters, with assumed force control in Z-direction -->
-    <xacro:thruster_link name="fwd" xyz="-0.52 0 -0.03" rpy="0 ${-PI/2} 0"/>
+    <xacro:thruster_link name="fwd" xyz="-0.52 0 -0.03" rpy="0 ${-PI/2} 0" rotationAxis="0 1 0" lowerLimit="-${PI/2}" upperLimit="${PI/2}"/>
 </robot>

File: src/usv_sim/xacro/sailboat.xacro (robot description, xacro)
@@ -19,5 +19,5 @@
               <box size="0.4 0.02 1" />
             </geometry>
-            <origin rpy="0 0 0" xyz="0 0 0"/>
+            <origin rpy="0 0 0" xyz="-0.2 0 0"/>
 	    </collision>
 	    <visual name="visual">
@@ -25,5 +25,5 @@
               <box size="0.4 0.02 1" />
             </geometry>
-            <origin rpy="0 0 0" xyz="0 0 0"/>
+            <origin rpy="0 0 0" xyz="-0.2 0 0"/>
 	    </visual>
     </link>
@@ -31,8 +31,40 @@
         <parent link="base_link"/>
         <child link="sail"/>
-        <origin rpy="0 0 ${PI/2}" xyz="0 0 +0.6"/>
+        <origin rpy="0 0 0" xyz="0 0 +0.6"/>
         <dynamics damping="1.0"/>
         <axis xyz="0 0 1"/>
         <limit effort="30" velocity="5" lower="-${PI/2}" upper="${PI/2}" />
+    </joint>
+    <link name="keel">
+	<inertial>
+		<mass value="20" />
+		<inertia
+		  ixx="0.4708"
+		  ixy="0.0"
+		  iyy="0.5208"
+		  ixz="0.0"
+		  iyz="0.0"
+		  izz="0.0508"/>
+	</inertial>
+	<collision name="collision">
+	<geometry>
+	<box size="0.25 0.02 0.5" />
+	</geometry>
+	<origin rpy="0 0 0" xyz="0 0 0"/>
+	</collision>
+	<visual name="visual">
+	<geometry>
+	<box size="0.25 0.02 0.5" />
+	</geometry>
+	<origin rpy="0 0 0" xyz="0 0 0"/>
+	</visual>
+    </link>
+    <joint name="keel_joint" type="revolute">
+        <parent link="base_link"/>
+        <child link="keel"/>
+        <origin rpy="0 0 0" xyz="0 0 -0.35"/>
+        <dynamics damping="1.0"/>
+        <axis xyz="0 0 1"/>
+        <limit effort="30" velocity="5" lower="0" upper="0" />
     </joint>
     <!-- Plugin list -->
@@ -40,6 +72,6 @@
         <plugin name="sail_plugin" filename="libsail_plugin.so">
             <a0>0</a0>
-            <cla>2.752798721</cla>
-            <cda>2.6417112299</cda>
+            <cla>4.752798721</cla>
+            <cda>0.6417112299</cda>
             <cma>-1.8</cma>
             <alpha_stall>0.785</alpha_stall>
@@ -47,5 +79,5 @@
             <cda_stall>-0.9233984055</cda_stall>
             <cma_stall>0</cma_stall>
-            <cp>0 0 0</cp>
+            <cp>-0.2 0 0</cp>
             <area>0.4</area>
             <air_density>1.2041</air_density>
@@ -74,4 +106,22 @@
             <link_name>rudder</link_name>
         </plugin>
+        <plugin name="rudder_plugin" filename="librudder_plugin.so">
+            <a0>0</a0>
+            <cla>4.752798721</cla>
+            <cda>2.3417112299</cda>
+            <!--
+            <cma>-1.8</cma> momentum
+            <cma_stall>0</cma_stall>
+            -->
+            <alpha_stall>0.785</alpha_stall>
+            <cla_stall>-3.85</cla_stall>
+            <cda_stall>-0.3233984055</cda_stall>
+            <cp>-0.25 0 0</cp>
+            <area>0.125</area>
+            <air_density>1000</air_density>
+            <forward>1 0 0</forward>
+            <upward>0 1 0</upward>
+            <link_name>keel</link_name>
+        </plugin>
         <plugin name="freefloating_gazebo_control" filename="libfreefloating_gazebo_control.so">
             <switchService>switch</switchService>

Commit message: Solved duplicated node and keel problem in sailboat.launch and sailboat.xacro

File: src/usv_sim/xacro/boat_common_subdivided.xacro (robot description, xacro)
@@ -201,5 +201,5 @@
     <joint name="hokuyo_joint" type="fixed">
         <axis xyz="0 1 0" />
-        <origin xyz="0.6 0 0.1" rpy="0 0 0"/>
+        <origin xyz="0.7 0 0.2" rpy="0 0 0"/>
         <parent link="base_link"/>
         <child link="hokuyo_link"/>
@@ -227,5 +227,5 @@
         <sensor type="gpu_ray" name="head_hokuyo_sensor">
         <pose>0 0 0 0 0 0</pose>
-        <visualize>false</visualize>
+        <visualize>true</visualize>
         <update_rate>40</update_rate>
         <ray>

File: src/usv_sim/xacro/sailboat.xacro (robot description, xacro)
@@ -92,5 +92,5 @@
 	<origin rpy="0 0 0" xyz="0 0 0"/>
 	</visual>
-    </link>
+</link>
     <joint name="keel_joint" type="revolute">
         <parent link="base_link"/>

File: src/usv_sim/xacro/sailboat_2.xacro (robot description, xacro)
@@ -28,4 +28,12 @@
 	    </visual>
     </link>
+    <joint name="sail_joint" type="revolute">
+        <parent link="base_link"/>
+        <child link="sail"/>
+        <origin rpy="0 0 0" xyz="0.2 0 0.6"/>
+        <dynamics damping="1.0"/>
+        <axis xyz="0 0 1"/>
+        <limit effort="0" velocity="5" lower="-${PI/2}" upper="${PI/2}" />
+    </joint>
     <link name="keel">
         <inertial>
@@ -60,13 +68,5 @@
         <limit effort="50" velocity="5" lower="0" upper="0" />
     </joint>
-    <joint name="sail_joint" type="revolute">
-        <parent link="base_link"/>
-        <child link="sail"/>
-        <origin rpy="0 0 0" xyz="0.2 0 0.6"/>
-        <dynamics damping="1.0"/>
-        <axis xyz="0 0 1"/>
-        <limit effort="0" velocity="5" lower="-${PI/2}" upper="${PI/2}" />
-    </joint>
-    <!-- Plugin list -->
+        <!-- Plugin list -->
   <gazebo>
         <plugin name="sail_plugin" filename="libsail_plugin.so">

Commit message: added pid heading control to diferential boat

File: src/usv_sim/xacro/boat_common_subdivided.xacro (robot description, xacro)
@@ -201,5 +201,5 @@
     <joint name="hokuyo_joint" type="fixed">
         <axis xyz="0 1 0" />
-        <origin xyz="0.7 0 0.2" rpy="0 0 0"/>
+        <origin xyz="0.7 0 0.1" rpy="0 0 0"/>
         <parent link="base_link"/>
         <child link="hokuyo_link"/>
