Commit message: Changed thruster configurations of boat_rudder and boat_diff

File: src/usv_sim/xacro/boat_diff.xacro (robot description, xacro)
@@ -7,17 +7,17 @@
             <switchService>switch</switchService>
             <updateRate>100</updateRate>
-            <link>base_link</link>
+            <link>fwd_left</link>
             <thruster>
                 <effort>30</effort>
                 <name>fwd_left</name>
             </thruster>
-        <thruster>
-            <effort>30</effort>
-            <name>fwd_right</name>
-        </thruster>
+   	    <thruster>
+	        <effort>30</effort>
+	        <name>fwd_right</name>
+	    </thruster>
         </plugin>
     </gazebo>
     <!-- Define two steering thrusters, with assumed force control in Z-direction -->
-    <xacro:thruster_link name="fwd_left" xyz="-0.52 0.1 0" rpy="0 ${-PI/2} 0" rotationAxis="0 1 0" lowerLimit="-${PI/2}" upperLimit="${PI/2}"/>
-    <xacro:thruster_link name="fwd_right" xyz="-0.52 -0.1 0" rpy="0 ${-PI/2} 0" rotationAxis="0 1 0" lowerLimit="-${PI/2}" upperLimit="${PI/2}"/>
+    <xacro:thruster_link name="fwd_left" xyz="-0.77 0.1 0" rpy="0 ${-PI/2} 0" rotationAxis="0 1 0" lowerLimit="-${PI/2}" upperLimit="${PI/2}"/>
+    <xacro:thruster_link name="fwd_right" xyz="-0.77 -0.1 0" rpy="0 ${-PI/2} 0" rotationAxis="0 1 0" lowerLimit="-${PI/2}" upperLimit="${PI/2}"/>
 </robot>

File: src/usv_sim/xacro/boat_rudder.xacro (robot description, xacro)
@@ -27,5 +27,5 @@
             <switchService>switch</switchService>
             <updateRate>100</updateRate>
-            <link>base_link</link>
+            <link>fwd</link>
             <thruster>
                 <effort>30</effort>
@@ -35,4 +35,4 @@
     </gazebo>
     <!-- Define two steering thrusters, with assumed force control in Z-direction -->
-    <xacro:thruster_link name="fwd" xyz="-0.52 0 -0.03" rpy="0 ${-PI/2} 0" rotationAxis="0 1 0" lowerLimit="-${PI/2}" upperLimit="${PI/2}"/>
+    <xacro:thruster_link name="fwd" xyz="-0.77 0 -0.03" rpy="0 ${-PI/2} 0" rotationAxis="0 1 0" lowerLimit="-${PI/2}" upperLimit="${PI/2}"/>
 </robot>

Commit message: Adding new hull to boat_rudder and boat_diff

File: src/usv_sim/xacro/boat_diff.xacro (robot description, xacro)
@@ -19,5 +19,5 @@
     </gazebo>
     <!-- Define two steering thrusters, with assumed force control in Z-direction -->
-    <xacro:thruster_link name="fwd_left"  xyz="-1.2 0 -0.5" rpy="0 ${-PI/2} 0" rotationAxis="1 0 0" lowerLimit="0" upperLimit="0" parentLink="back_l_link"/>
-    <xacro:thruster_link name="fwd_right" xyz="-1.2 0 -0.5" rpy="0 ${-PI/2} 0" rotationAxis="1 0 0" lowerLimit="0" upperLimit="0" parentLink="back_r_link"/>
+    <xacro:thruster_link name="fwd_left"  xyz="-0.4 0 -0.15" rpy="0 ${-PI/2} 0" rotationAxis="1 0 0" lowerLimit="0" upperLimit="0" parentLink="back_l_link"/>
+    <xacro:thruster_link name="fwd_right" xyz="-0.4 0 -0.15" rpy="0 ${-PI/2} 0" rotationAxis="1 0 0" lowerLimit="0" upperLimit="0" parentLink="back_r_link"/>
 </robot>

File: src/usv_sim/xacro/boat_rudder.xacro (robot description, xacro)
@@ -35,4 +35,4 @@
     </gazebo>
     <!-- Define two steering thrusters, with assumed force control in Z-direction -->
-    <xacro:thruster_link name="fwd" xyz="-0.8 0.22 -0.5" rpy="0 ${-PI/2} 0" rotationAxis="1 0 0" lowerLimit="0" upperLimit="0" />
+    <xacro:thruster_link name="fwd" xyz="-0.3 0.07 -0.15" rpy="0 ${-PI/2} 0" rotationAxis="1 0 0" lowerLimit="0" upperLimit="0" />
 </robot>

File: src/usv_sim/xacro/boat_sea_angler.xacro (robot description, xacro)
@@ -1,5 +1,5 @@
 <?xml version="1.0"?>
 <robot name="boat_diff" xmlns:xacro="http://www.ros.org/wiki/xacro">
-    <xacro:include filename="$(find usv_sim)/xacro/boat_sea_angler_subdivided2.xacro" />
+    <xacro:include filename="$(find usv_sim)/xacro/boat_subdivided.xacro" />
     <!-- Plugin list -->
     <gazebo>
@@ -15,4 +15,4 @@
     </gazebo>
     <!-- Define two steering thrusters, with assumed force control in Z-direction -->
-    <xacro:thruster_link name="fwd" xyz="-1.2 0.22 -0.50" rpy="0 ${-PI/2} 0" rotationAxis="1 0 0" lowerLimit="-${PI/4}" upperLimit="${PI/4}" effort="500"/>
+   <xacro:thruster_link name="fwd" xyz="-0.4 0.07 -0.15" rpy="0 ${-PI/2} 0" rotationAxis="1 0 0" lowerLimit="-${PI/4}" upperLimit="${PI/4}" effort="500"/>
 </robot>

File: src/usv_sim/xacro/boat_subdivided.xacro (robot description, xacro)
@@ -11,4 +11,5 @@
     <xacro:property name="middle_water_displaced_mass" value="60"/>
     <xacro:property name="front_water_displaced_mass" value="25"/>
+    <xacro:property name="scale" value="0.3"/>
     <!-- Thruster constants -->
     <xacro:property name="tr1" value=".02" />
@@ -21,16 +22,16 @@
           <origin rpy="0 0 0" xyz="0 0 0"/>
           <geometry>
-            <mesh filename="package://usv_sim/meshes/simpleHull/simpleHull.obj"/>
+            <mesh filename="package://usv_sim/meshes/simpleHull/simpleHull.obj" scale="${scale} ${scale} ${scale}"/>
           </geometry>
           <material name="white"/>
         </visual>
         <collision>
-          <origin rpy="0 0 1.57" xyz="0 0.44 0.1"/>
-          <geometry>
-            <mesh filename="package://usv_sim/meshes/simpleHull/centerLeft.stl"/>
-          </geometry>
-        </collision>
-        <inertial>
-            <origin rpy="0 0 0" xyz="0 0.44 0.1"/>
+          <origin rpy="0 0 1.57" xyz="0 ${0.44*scale} ${0.1*scale}"/>
+          <geometry>
+            <mesh filename="package://usv_sim/meshes/simpleHull/centerLeft.stl" scale="${scale} ${scale} ${scale}"/>
+          </geometry>
+        </collision>
+        <inertial>
+            <origin rpy="0 0 0" xyz="0 ${0.44*scale} ${0.1*scale}"/>
           <mass value="${middle_body_mass}"/>
           <inertia ixx="0.1" ixy="0.0" ixz="0.0" iyy="1.4" iyz="0.0" izz="1.4"/>
@@ -38,5 +39,5 @@
         <buoyancy>
           <compensation>${middle_water_displaced_mass/middle_body_mass}</compensation>
-          <origin xyz="0 0.44 0.15"/>
+          <origin xyz="0 ${0.44*scale} ${0.15*scale}"/>
           <limit radius="0.1"/>
           <damping rpy="20 20 20" xyz="20 20 50"/>
@@ -46,11 +47,11 @@
     <link name="center_r_link">
         <collision>
-          <origin rpy="0 0 1.57"  xyz="0 -0.22 0.05"/>
-          <geometry>
-           	<mesh filename="package://usv_sim/meshes/simpleHull/centerRight.stl"/>
-          </geometry>
-        </collision>
-        <inertial>
-            <origin rpy="0 0 0" xyz="0 -0.22 0.05"/>
+          <origin rpy="0 0 1.57"  xyz="0 ${-0.22*scale} ${0.05*scale}"/>
+          <geometry>
+           	<mesh filename="package://usv_sim/meshes/simpleHull/centerRight.stl" scale="${scale} ${scale} ${scale}"/>
+          </geometry>
+        </collision>
+        <inertial>
+            <origin rpy="0 0 0" xyz="0 ${-0.22*scale} ${0.05*scale}"/>
           <mass value="${middle_body_mass}"/>
           <inertia ixx="0.1" ixy="0.0" ixz="0.0" iyy="1.4" iyz="0.0" izz="1.4"/>
@@ -58,5 +59,5 @@
         <buoyancy>
           <compensation>${middle_water_displaced_mass/middle_body_mass}</compensation>
-          <origin xyz="0 -0.22 0.1"/>
+          <origin xyz="0 ${-0.22*scale} ${0.1*scale}"/>
           <limit radius="0.1"/>
           <damping rpy="20 20 20" xyz="20 20 50"/>
@@ -67,5 +68,5 @@
         <parent link="base_link"/>
         <child link="center_r_link"/>
-        <origin rpy="0 0 0" xyz="0 -0.22 0"/>
+        <origin rpy="0 0 0" xyz="0 ${-0.22*scale} 0"/>
 	<limit effort="50" velocity="5" lower="0" upper="0" />
             <dynamics damping="1.0"/>
@@ -74,11 +75,11 @@
     <link name="back_l_link">
         <collision>
-          <origin rpy="0 0 1.57"  xyz="-0.85 0.205 -0.2"/>
-          <geometry>
-           	<mesh filename="package://usv_sim/meshes/simpleHull/backLeft.stl"/>
-          </geometry>
-        </collision>
-        <inertial>
-            <origin rpy="0 0 0" xyz="-0.85 0.205 -0.2"/>
+          <origin rpy="0 0 1.57"  xyz="${-0.85*scale} ${0.205*scale} ${-0.2*scale}"/>
+          <geometry>
+           	<mesh filename="package://usv_sim/meshes/simpleHull/backLeft.stl" scale="${scale} ${scale} ${scale}"/>
+          </geometry>
+        </collision>
+        <inertial>
+            <origin rpy="0 0 0" xyz="${-0.85*scale} ${0.205*scale} ${-0.2*scale}"/>
           <mass value="${back_body_mass}"/>
           <inertia ixx="0.1" ixy="0.0" ixz="0.0" iyy="1.4" iyz="0.0" izz="1.4"/>
@@ -86,5 +87,5 @@
         <buoyancy>
           <compensation>${back_water_displaced_mass/back_body_mass}</compensation>
-          <origin xyz="-0.85 0.205 -0.15"/>
+          <origin xyz="${-0.85*scale} ${0.205*scale} ${-0.15*scale}"/>
           <limit radius="0.1"/>
           <damping rpy="20 20 20" xyz="20 20 50"/>
@@ -95,5 +96,5 @@
         <parent link="base_link"/>
         <child link="back_l_link"/>
-        <origin rpy="0 0 0" xyz="-0.85 0.205 0"/>
+        <origin rpy="0 0 0" xyz="${-0.85*scale} ${0.205*scale} 0"/>
 	<limit effort="50" velocity="5" lower="0" upper="0" />
             <dynamics damping="1.0"/>
@@ -102,11 +103,11 @@
     <link name="back_r_link">
         <collision>
-          <origin rpy="0 0 1.57"  xyz="-0.85 -0.205 -0.2"/>
-          <geometry>
-           	<mesh filename="package://usv_sim/meshes/simpleHull/backRight.stl"/>
-          </geometry>
-        </collision>
-        <inertial>
-            <origin rpy="0 0 0" xyz="-0.85 -0.205 -0.2"/>
+          <origin rpy="0 0 1.57"  xyz="${-0.85*scale} ${-0.205*scale} ${-0.2*scale}"/>
+          <geometry>
+           	<mesh filename="package://usv_sim/meshes/simpleHull/backRight.stl" scale="${scale} ${scale} ${scale}"/>
+          </geometry>
+        </collision>
+        <inertial>
+            <origin rpy="0 0 0" xyz="${-0.85*scale} ${-0.205*scale} ${-0.2*scale}"/>
           <mass value="${back_body_mass}"/>
           <inertia ixx="0.1" ixy="0.0" ixz="0.0" iyy="1.4" iyz="0.0" izz="1.4"/>
@@ -114,5 +115,5 @@
         <buoyancy>
           <compensation>${back_water_displaced_mass/back_body_mass}</compensation>
-          <origin xyz="-0.85 -0.205 -0.15"/>
+          <origin xyz="${-0.85*scale} ${-0.205*scale} ${-0.15*scale}"/>
           <limit radius="0.1"/>
           <damping rpy="20 20 20" xyz="20 20 50"/>
@@ -123,5 +124,5 @@
         <parent link="base_link"/>
         <child link="back_r_link"/>
-        <origin rpy="0 0 0" xyz="-0.85 -0.205 0"/>
+        <origin rpy="0 0 0" xyz="${-0.85*scale} ${-0.205*scale} 0"/>
 	<limit effort="50" velocity="5" lower="0" upper="0" />
             <dynamics damping="1.0"/>
@@ -130,11 +131,11 @@
     <link name="front_l_link">
         <collision>
-          <origin rpy="0 0 1.57"  xyz="0.85 0.17 0.2"/>
-          <geometry>
-           	<mesh filename="package://usv_sim/meshes/simpleHull/frontLeft.stl"/>
-          </geometry>
-        </collision>
-        <inertial>
-            <origin rpy="0 0 0" xyz="0.85 0.17 -0.1"/>
+          <origin rpy="0 0 1.57"  xyz="${0.85*scale} ${0.17*scale} ${0.2*scale}"/>
+          <geometry>
+           	<mesh filename="package://usv_sim/meshes/simpleHull/frontLeft.stl" scale="${scale} ${scale} ${scale}"/>
+          </geometry>
+        </collision>
+        <inertial>
+            <origin rpy="0 0 0" xyz="${0.85*scale} ${0.17*scale} ${-0.1*scale}"/>
           <mass value="${front_body_mass}"/>
           <inertia ixx="0.1" ixy="0.0" ixz="0.0" iyy="1.4" iyz="0.0" izz="1.4"/>
@@ -142,5 +143,5 @@
         <buoyancy>
           <compensation>${front_water_displaced_mass/front_body_mass}</compensation>
-          <origin xyz="0.85 0.17 -0.05"/>
+          <origin xyz="${0.85*scale} ${0.17*scale} ${-0.05*scale}"/>
           <limit radius="0.1"/>
           <damping rpy="20 20 20" xyz="20 20 50"/>
@@ -151,5 +152,5 @@
         <parent link="base_link"/>
         <child link="front_l_link"/>
-        <origin rpy="0 0 0" xyz="0.85 0.17 0"/>
+        <origin rpy="0 0 0" xyz="${0.85*scale} ${0.17*scale} 0"/>
 	<limit effort="50" velocity="5" lower="0" upper="0" />
             <dynamics damping="1.0"/>
@@ -158,11 +159,11 @@
     <link name="front_r_link">
         <collision>
-          <origin rpy="0 0 1.57"  xyz="0.85 -0.17 0.2"/>
-          <geometry>
-           	<mesh filename="package://usv_sim/meshes/simpleHull/frontRight.stl"/>
-          </geometry>
-        </collision>
-        <inertial>
-            <origin rpy="0 0 0" xyz="0.85 -0.17 -0.1"/>
+          <origin rpy="0 0 1.57"  xyz="${0.85*scale} ${-0.17*scale} ${0.2*scale}"/>
+          <geometry>
+           	<mesh filename="package://usv_sim/meshes/simpleHull/frontRight.stl" scale="${scale} ${scale} ${scale}"/>
+          </geometry>
+        </collision>
+        <inertial>
+            <origin rpy="0 0 0" xyz="${0.85*scale} ${-0.17*scale} ${-0.1*scale}"/>
           <mass value="${front_body_mass}"/>
           <inertia ixx="0.1" ixy="0.0" ixz="0.0" iyy="1.4" iyz="0.0" izz="1.4"/>
@@ -170,5 +171,5 @@
         <buoyancy>
           <compensation>${front_water_displaced_mass/front_body_mass}</compensation>
-          <origin xyz="0.85 -0.17 -0.05"/>
+          <origin xyz="${0.85*scale} ${-0.17*scale} ${-0.05*scale}"/>
           <limit radius="0.1"/>
           <damping rpy="20 20 20" xyz="20 20 50"/>
@@ -179,5 +180,5 @@
         <parent link="base_link"/>
         <child link="front_r_link"/>
-        <origin rpy="0 0 0" xyz="0.85 -0.17 0"/>
+        <origin rpy="0 0 0" xyz="${0.85*scale} ${-0.17*scale} 0"/>
 	<limit effort="50" velocity="5" lower="0" upper="0" />
             <dynamics damping="1.0"/>
@@ -202,5 +203,5 @@
           		<origin xyz="0 0 0" rpy="0 0 0"/>
           		<geometry>
-          			<box size="tl1 tl1 tl2" />
+          			<box size="${tl1} ${tl1} ${tl2}" />
           		</geometry>
         	</collision>
@@ -208,5 +209,5 @@
                 <origin xyz="0 0 0" rpy="0 0 0" />
                 <geometry>
-                    <mesh filename="package://usv_sim/meshes/simpleHull/thruster.obj"/>
+                    <mesh filename="package://usv_sim/meshes/simpleHull/thruster.obj" scale="${scale} ${scale} ${scale}"/>
                 </geometry>
                 <material name="black">
@@ -252,13 +253,13 @@
             <collision name="collision">
                 <geometry>
-                  <box size="0.2 0.02 0.3" />
+                  <box size="${0.2*scale} ${0.02*scale} ${0.3*scale}" />
                 </geometry>
-                <origin rpy="0 0 0" xyz="-0.1 0 0"/>
+                <origin rpy="0 0 0" xyz="${-0.1*scale} 0 0"/>
             </collision>
             <visual name="visual">
                 <geometry>
-                  <box size="0.1 0.02 0.3" />
+                  <box size="${0.2*scale} ${0.02*scale} ${0.3*scale}" />
                 </geometry>
-                <origin rpy="0 0 0" xyz="-0.1 0 0"/>
+                <origin rpy="0 0 0" xyz="${-0.1*scale} 0 0"/>
             </visual>
         </link>
@@ -266,5 +267,5 @@
             <parent link="back_r_link"/>
             <child link="rudder"/>
-            <origin rpy="0 0 0" xyz="-1.2 0.22 -0.5"/>
+            <origin rpy="0 0 0" xyz="${-1.4*scale} ${0.22*scale} ${-0.5*scale}"/>
             <dynamics damping="1.0"/>
             <axis xyz="0 0 1"/>
@@ -276,20 +277,20 @@
     <joint name="hokuyo_joint" type="fixed">
         <axis xyz="0 1 0" />
-        <origin xyz="0.7 0 0.1" rpy="0 0 0"/>
+        <origin xyz="0.7 0 0.2" rpy="0 0 0"/>
         <parent link="base_link"/>
         <child link="hokuyo_link"/>
     </joint>
     <link name="hokuyo_link">
-        <collision>
-        <origin xyz="0 0 0" rpy="0 0 0"/>
-        <geometry>
-        <box size="0.1 0.1 0.1"/>
-        </geometry>
-        </collision>
-        <visual>
-        <origin xyz="0 0 0" rpy="0 0 0"/>
-        <geometry>
-        <mesh filename="package://usv_sim/meshes/hokuyo.stl"/>
-        </geometry>
+        <collision name="collision">
+	        <origin xyz="0 0 0" rpy="0 0 0"/>
+	        <geometry>
+	        	<box size="0.1 0.1 0.1"/>
+	        </geometry>
+        </collision>
+        <visual name="visual">
+        	<origin xyz="0 0 0" rpy="0 0 0"/>
+        	<geometry>
+        		<mesh filename="package://usv_sim/meshes/hokuyo.stl"/>
+        	</geometry>
         </visual>
         <inertial>
