Commit message: Minor fixes

File: src/usv_sim/xacro/boat_subdivided3.xacro (robot description, xacro)
@@ -230,5 +230,5 @@
 	    	</buoyancy>
 	    	<collision>
-          		<origin xyz="0 0 0" rpy="{-0.15*scale} 0 ${0.3*scale}"/>
+          		<origin xyz="0 0 0" rpy="${-0.15*scale} 0 ${0.3*scale}"/>
           		<geometry>
           		    <mesh filename="package://usv_sim/meshes/simpleHull/thruster.obj" scale="${scale} ${scale} ${scale}"/>

Commit message: boat rudder  heading control working

File: src/usv_sim/xacro/boat_subdivided3.xacro (robot description, xacro)
@@ -351,5 +351,5 @@
             <dynamics damping="1.0"/>
             <axis xyz="0 0 1"/>
-            <limit effort="50" velocity="5" lower="-${PI/3}" upper="${PI/3}" />
+            <limit effort="100" velocity="5" lower="-${1.309}" upper="${1.309}" />
         </joint>
     </xacro:macro>
