Commit message: Changed some configurations of airboat

File: src/usv_sim/xacro/airboat.xacro (robot description, xacro)
@@ -16,4 +16,4 @@
     </gazebo>
     <!-- Define one steering thruster, with assumed force control in Z-direction -->
-    <xacro:thruster_link name="fwd" xyz="-0.5 0 0.2" rpy="0 ${-PI/2} 0" rotationAxis="1 0 0" lowerLimit="-${2*PI}" upperLimit="${2*PI}"/>
+    <xacro:thruster_link name="fwd" xyz="-0.5 0 0.2" rpy="0 ${-PI/2} 0" effort="50" velocity="20" rotationAxis="1 0 0" lowerLimit="-${PI}" upperLimit="${PI}"/>
 </robot>

File: src/usv_sim/xacro/boat_common_subdivided.xacro (robot description, xacro)
@@ -111,6 +111,6 @@
     </joint>
     <!-- Thruster link -->
-    <xacro:macro name="thruster_link" params="name xyz rpy rotationAxis lowerLimit upperLimit">
-        <joint name="${name}_link" type="revolute">
+    <xacro:macro name="thruster_link" params="name xyz rpy rotationAxis effort:=30 velocity:=5 lowerLimit upperLimit">
+        <joint name="${name}_joint" type="revolute">
             <parent link="base_link"/>
             <child link="${name}"/>
@@ -118,5 +118,5 @@
             <dynamics damping="10.0"/>
             <axis xyz="${rotationAxis}"/>
-            <limit effort="30" velocity="5.0" lower="${lowerLimit}" upper="${upperLimit}" />
+            <limit effort="${effort}" velocity="${velocity}" lower="${lowerLimit}" upper="${upperLimit}" />
         </joint>
         <link name="${name}">

Commit message: Added water surface to thruster max command

File: src/usv_sim/xacro/airboat.xacro (robot description, xacro)
@@ -8,7 +8,8 @@
             <switchService>switch</switchService>
             <updateRate>100</updateRate>
-            <link>base_link</link>
+            <link>fwd</link>
             <thruster>
-                <effort>20</effort>
+                <effortUnderWater>20</effortUnderWater>
+		<effortOverWater>30</effortOverWater>
                 <name>fwd</name>
             </thruster>

Commit message: Changed hull of sailboat

File: src/usv_sim/xacro/airboat.xacro (robot description, xacro)
@@ -1,5 +1,5 @@
 <?xml version="1.0"?>
 <robot name="boat_rudder" xmlns:xacro="http://www.ros.org/wiki/xacro">
-    <xacro:include filename="$(find usv_sim)/xacro/boat_common_subdivided.xacro" />
+    <xacro:include filename="$(find usv_sim)/xacro/boat_subdivided.xacro" />
     <!-- Plugin list -->
     <gazebo>
@@ -11,5 +11,5 @@
             <thruster>
                 <effortUnderWater>20</effortUnderWater>
-		<effortOverWater>30</effortOverWater>
+				<effortOverWater>30</effortOverWater>
                 <name>fwd</name>
             </thruster>
@@ -17,4 +17,6 @@
     </gazebo>
     <!-- Define one steering thruster, with assumed force control in Z-direction -->
-    <xacro:thruster_link name="fwd" xyz="-0.5 0 0.2" rpy="0 ${-PI/2} 0" effort="50" velocity="20" rotationAxis="1 0 0" lowerLimit="-${PI}" upperLimit="${PI}"/>
+    <!--<xacro:thruster_link name="fwd" xyz="0 0 0.2" rpy="0 ${-PI/2} 0" effort="50" velocity="20" rotationAxis="1 0 0" lowerLimit="-${PI/4}" upperLimit="${PI/4}"/>
+    -->
+    <xacro:airthruster_link name="fwd" xyz="0 0.05 0.3" rpy="0 ${-PI/2} 0" effort="50" velocity="20" rotationAxis="1 0 0" lowerLimit="-${PI/4}" upperLimit="${PI/4}"/>
 </robot>

File: src/usv_sim/xacro/boat_subdivided2.xacro (robot description, xacro)
@@ -22,5 +22,6 @@
           <origin rpy="0 0 0" xyz="0 0 0"/>
           <geometry>
-            <mesh filename="package://usv_sim/meshes/simpleHull/simpleHull.obj" scale="${scale} ${scale} ${scale}"/>
+            <!--<mesh filename="package://usv_sim/meshes/simpleHull/simpleHull.obj" scale="${scale} ${scale} ${scale}"/>-->
+            <box size="1.2 0.4 0.2" />
           </geometry>
           <material name="white"/>
@@ -29,5 +30,6 @@
           <origin rpy="0 0 1.57" xyz="0 ${0.44*scale} ${0.1*scale}"/>
           <geometry>
-            <mesh filename="package://usv_sim/meshes/simpleHull/centerLeft.stl" scale="${scale} ${scale} ${scale}"/>
+           <!-- <mesh filename="package://usv_sim/meshes/simpleHull/centerLeft.stl" scale="${scale} ${scale} ${scale}"/>-->
+           <box size="0.1 0.1 0.1" />
           </geometry>
         </collision>
@@ -49,5 +51,6 @@
           <origin rpy="0 0 1.57"  xyz="0 ${-0.22*scale} ${0.05*scale}"/>
           <geometry>
-           	<mesh filename="package://usv_sim/meshes/simpleHull/centerRight.stl" scale="${scale} ${scale} ${scale}"/>
+           <!--	<mesh filename="package://usv_sim/meshes/simpleHull/centerRight.stl" scale="${scale} ${scale} ${scale}"/>-->
+           <box size="0.1 0.1 0.1" />
           </geometry>
         </collision>
@@ -77,5 +80,6 @@
           <origin rpy="0 0 1.57"  xyz="${-0.85*scale} ${0.205*scale} ${-0.2*scale}"/>
           <geometry>
-           	<mesh filename="package://usv_sim/meshes/simpleHull/backLeft.stl" scale="${scale} ${scale} ${scale}"/>
+         <!--  	<mesh filename="package://usv_sim/meshes/simpleHull/backLeft.stl" scale="${scale} ${scale} ${scale}"/>-->
+         <box size="0.1 0.1 0.1" />
           </geometry>
         </collision>
@@ -105,5 +109,6 @@
           <origin rpy="0 0 1.57"  xyz="${-0.85*scale} ${-0.205*scale} ${-0.2*scale}"/>
           <geometry>
-           	<mesh filename="package://usv_sim/meshes/simpleHull/backRight.stl" scale="${scale} ${scale} ${scale}"/>
+           <!--	<mesh filename="package://usv_sim/meshes/simpleHull/backRight.stl" scale="${scale} ${scale} ${scale}"/>-->
+           <box size="0.1 0.1 0.1" />
           </geometry>
         </collision>
@@ -125,60 +130,4 @@
         <child link="back_r_link"/>
         <origin rpy="0 0 0" xyz="${-0.85*scale} ${-0.205*scale} 0"/>
-	<limit effort="50" velocity="5" lower="0" upper="0" />
-            <dynamics damping="1.0"/>
-            <axis xyz="1 0 0"/>
-    </joint>
-    <link name="front_l_link">
-        <collision>
-          <origin rpy="0 0 1.57"  xyz="${0.85*scale} ${0.17*scale} ${0.2*scale}"/>
-          <geometry>
-           	<mesh filename="package://usv_sim/meshes/simpleHull/frontLeft.stl" scale="${scale} ${scale} ${scale}"/>
-          </geometry>
-        </collision>
-        <inertial>
-            <origin rpy="0 0 0" xyz="${0.85*scale} ${0.17*scale} ${-0.1*scale}"/>
-          <mass value="${front_body_mass}"/>
-          <inertia ixx="0.1" ixy="0.0" ixz="0.0" iyy="1.4" iyz="0.0" izz="1.4"/>
-        </inertial>
-        <buoyancy>
-          <compensation>${front_water_displaced_mass/front_body_mass}</compensation>
-          <origin xyz="${0.85*scale} ${0.17*scale} ${-0.05*scale}"/>
-          <limit radius="0.1"/>
-          <damping rpy="20 20 20" xyz="20 20 50"/>
-	  <fluidVelocity>local</fluidVelocity>
-        </buoyancy>
-    </link>
-    <joint name="front_l_joint" type="revolute">
-        <parent link="base_link"/>
-        <child link="front_l_link"/>
-        <origin rpy="0 0 0" xyz="${0.85*scale} ${0.17*scale} 0"/>
-	<limit effort="50" velocity="5" lower="0" upper="0" />
-            <dynamics damping="1.0"/>
-            <axis xyz="1 0 0"/>
-    </joint>
-    <link name="front_r_link">
-        <collision>
-          <origin rpy="0 0 1.57"  xyz="${0.85*scale} ${-0.17*scale} ${0.2*scale}"/>
-          <geometry>
-           	<mesh filename="package://usv_sim/meshes/simpleHull/frontRight.stl" scale="${scale} ${scale} ${scale}"/>
-          </geometry>
-        </collision>
-        <inertial>
-            <origin rpy="0 0 0" xyz="${0.85*scale} ${-0.17*scale} ${-0.1*scale}"/>
-          <mass value="${front_body_mass}"/>
-          <inertia ixx="0.1" ixy="0.0" ixz="0.0" iyy="1.4" iyz="0.0" izz="1.4"/>
-        </inertial>
-        <buoyancy>
-          <compensation>${front_water_displaced_mass/front_body_mass}</compensation>
-          <origin xyz="${0.85*scale} ${-0.17*scale} ${-0.05*scale}"/>
-          <limit radius="0.1"/>
-          <damping rpy="20 20 20" xyz="20 20 50"/>
-	  <fluidVelocity>local</fluidVelocity>
-        </buoyancy>
-    </link>
-    <joint name="front_r_joint" type="revolute">
-        <parent link="base_link"/>
-        <child link="front_r_link"/>
-        <origin rpy="0 0 0" xyz="${0.85*scale} ${-0.17*scale} 0"/>
 	<limit effort="50" velocity="5" lower="0" upper="0" />
             <dynamics damping="1.0"/>
@@ -203,5 +152,5 @@
           		<origin xyz="0 0 0" rpy="0 0 0"/>
           		<geometry>
-          		    <box size="${tl1} ${tl1} ${tl2}" />
+          			<box size="${tl1} ${tl1} ${tl2}" />
           		</geometry>
         	</collision>
@@ -312,8 +261,7 @@
             <visual name="visual">
                 <geometry>
-                  <mesh filename="package://usv_sim/meshes/simpleHull/box.obj" scale="${0.2*scale} ${0.02*scale} ${0.3*scale}"/>
+                  <box size="${0.2*scale} ${0.02*scale} ${0.3*scale}" />
                 </geometry>
                 <origin rpy="0 0 0" xyz="${-0.1*scale} 0 0"/>
-                <material name="blue"/>
             </visual>
         </link>
@@ -339,5 +287,5 @@
 	        <origin xyz="0 0 0" rpy="0 0 0"/>
 	        <geometry>
-	        	<box size="0.1 0.1 0.1"/>
+	        	<box size="0.05 0.05 0.05"/>
 	        </geometry>
         </collision>
@@ -345,7 +293,7 @@
         	<origin xyz="0 0 0" rpy="0 0 0"/>
         	<geometry>
-        		<mesh filename="package://usv_sim/meshes/simpleHull/box.obj" scale="0.1 0.1 0.1"/>
+        		<!--<mesh filename="package://usv_sim/meshes/hokuyo.stl"/>-->
+        		<box size="0.05 0.05 0.05"/>
         	</geometry>
-        	<material name="blue"/>
         </visual>
         <inertial>

File: src/usv_sim/xacro/sailboat.xacro (robot description, xacro)
@@ -1,9 +1,10 @@
 <?xml version="1.0"?>
 <robot name="sailboat" xmlns:xacro="http://www.ros.org/wiki/xacro">
-    <xacro:include filename="$(find usv_sim)/xacro/boat_common_subdivided.xacro" />
+    <xacro:include filename="$(find usv_sim)/xacro/boat_subdivided.xacro" />
     <xacro:rudder_xacro/>
     <!-- Defining sail model -->
     <link name="sail">
 		<inertial>
+		    <origin rpy="0 0 0" xyz="-0.3 0 0.4"/>
 			<mass value="0.1" />
 			<inertia
@@ -17,14 +18,13 @@
 	    <collision name="collision">
             <geometry>
-              <box size="0.4 0.02 1" />
+              <mesh filename="package://usv_sim/meshes/simpleHull/sail.obj" scale="0.5 0.5 0.5"/>
             </geometry>
-            <origin rpy="0 0 0" xyz="-0.2 0 0"/>
+            <origin rpy="0 0 0" xyz="0 0 0"/>
 	    </collision>
 	    <visual name="visual">
-            <plugin name="some_visual_plugin" filename="some_visual_plugin.so"/>
             <geometry>
-              <box size="0.4 0.02 1" />
+              <mesh filename="package://usv_sim/meshes/simpleHull/sail.obj" scale="0.5 0.5 0.5"/>
             </geometry>
-            <origin rpy="0 0 0" xyz="-0.2 0 0"/>
+            <origin rpy="0 0 0" xyz="0 0 0"/>
 	    </visual>
     </link>
@@ -32,8 +32,8 @@
         <parent link="base_link"/>
         <child link="sail"/>
-        <origin rpy="0 0 0" xyz="0 0 +0.6"/>
+        <origin rpy="0 0 0" xyz="0.2 0 0.1"/>
         <dynamics damping="1.0"/>
         <axis xyz="0 0 1"/>
-        <limit effort="30" velocity="5" lower="-${PI/2}" upper="${PI/2}" />
+        <limit effort="50" velocity="5" lower="-1.5" upper="1.5" />
     </joint>
     <link name="keel">
@@ -49,14 +49,14 @@
 	</inertial>
 	<collision name="collision">
-	<geometry>
-	<box size="0.25 0.02 0.5" />
-	</geometry>
-	<origin rpy="0 0 0" xyz="0 0 0"/>
+		<geometry>
+			<box size="0.25 0.02 0.5" />
+		</geometry>
+		<origin rpy="0 0 0" xyz="0 0 0"/>
 	</collision>
 	<visual name="visual">
-	<geometry>
-	<box size="0.25 0.02 0.5" />
-	</geometry>
-	<origin rpy="0 0 0" xyz="0 0 0"/>
+		<geometry>
+			<mesh filename="package://usv_sim/meshes/simpleHull/box.obj" scale="0.25 0.02 0.5"/>
+		</geometry>
+		<origin rpy="0 0 0" xyz="0 0 0"/>
 	</visual>
 </link>
@@ -80,12 +80,11 @@
             <cda_stall>-0.9233984055</cda_stall>
             <cma_stall>0</cma_stall>
-            <cp>0 0 -0.4</cp>
-            <area>0.4</area>
+            <cp>0 0 0</cp>
+            <joint_name>sail_joint</joint_name>
+            <area>1.44</area>
             <air_density>1.2041</air_density>
             <forward>1 0 0</forward>
             <upward>0 1 0</upward>
             <link_name>sail</link_name>
-            <!--<control_joint_name>rudder_joint</control_joint_name>-->
-            <!--<control_joint_rad_to_cl>4.0</control_joint_rad_to_cl>-->
       </plugin>
       <plugin name="keel_plugin" filename="libkeel_plugin.so">
@@ -93,8 +92,4 @@
           <cla>0.752798721</cla>
           <cda>0.3417112299</cda>
-          <!--
-          <cma>-1.8</cma> momentum
-          <cma_stall>0</cma_stall>
-          -->
           <alpha_stall>0.785</alpha_stall>
           <cla_stall>-0.85</cla_stall>
@@ -111,8 +106,4 @@
           <cla>0.752798721</cla>
           <cda>0.3417112299</cda>
-          <!--
-          <cma>-1.8</cma> momentum
-          <cma_stall>0</cma_stall>
-          -->
           <alpha_stall>0.785</alpha_stall>
           <cla_stall>-0.85</cla_stall>

Commit message: Changed geometry of boats

File: src/usv_sim/xacro/airboat.xacro (robot description, xacro)
@@ -1,5 +1,5 @@
 <?xml version="1.0"?>
 <robot name="boat_rudder" xmlns:xacro="http://www.ros.org/wiki/xacro">
-    <xacro:include filename="$(find usv_sim)/xacro/boat_subdivided.xacro" />
+    <xacro:include filename="$(find usv_sim)/xacro/boat_subdivided3.xacro" />
     <!-- Plugin list -->
     <gazebo>

File: src/usv_sim/xacro/boat_diff.xacro (robot description, xacro)
@@ -1,5 +1,5 @@
 <?xml version="1.0"?>
 <robot name="boat_diff" xmlns:xacro="http://www.ros.org/wiki/xacro">
-    <xacro:include filename="$(find usv_sim)/xacro/boat_subdivided.xacro" />
+    <xacro:include filename="$(find usv_sim)/xacro/boat_subdivided3.xacro" />
     <!-- Plugin list -->
     <gazebo>

File: src/usv_sim/xacro/boat_rudder.xacro (robot description, xacro)
@@ -1,5 +1,5 @@
 <?xml version="1.0"?>
 <robot name="boat_rudder" xmlns:xacro="http://www.ros.org/wiki/xacro">
-    <xacro:include filename="$(find usv_sim)/xacro/boat_subdivided.xacro" />
+    <xacro:include filename="$(find usv_sim)/xacro/boat_subdivided3.xacro" />
     <xacro:rudder_xacro/>
     <!-- Plugin list -->

File: src/usv_sim/xacro/boat_sea_angler.xacro (robot description, xacro)
@@ -15,4 +15,4 @@
     </gazebo>
     <!-- Define two steering thrusters, with assumed force control in Z-direction -->
-   <xacro:thruster_link name="fwd" xyz="-0.45 0.07 -0.15" rpy="0 ${-PI/2} 0" rotationAxis="1 0 0" lowerLimit="-${PI/4}" upperLimit="${PI/4}" effort="500"/>
+   <xacro:thruster_link name="fwd" xyz="-0.45 0.12 -0.15" rpy="0 ${-PI/2} 0" rotationAxis="1 0 0" lowerLimit="-${PI/4}" upperLimit="${PI/4}" effort="500"/>
 </robot>

File: src/usv_sim/xacro/boat_subdivided.xacro (robot description, xacro)
@@ -22,5 +22,5 @@
           <origin rpy="0 0 0" xyz="0 0 0"/>
           <geometry>
-            <mesh filename="package://usv_sim/meshes/simpleHull/simpleHull.obj" scale="${scale} ${scale} ${scale}"/>
+            <mesh filename="package://usv_sim/meshes/simpleHull/simpleHull.dae" scale="${scale} ${scale} ${scale}"/>
           </geometry>
           <material name="white"/>

File: src/usv_sim/xacro/boat_subdivided3.xacro (robot description, xacro)
@@ -24,5 +24,4 @@
             <mesh filename="package://usv_sim/meshes/simpleHull2/base_link.obj" scale="${scale} ${scale} ${scale}"/>
           </geometry>
-          <material name="white"/>
         </visual>
         <collision>
@@ -81,5 +80,5 @@
     <link name="back_l_link">
         <visual>
-          <origin rpy="0 0 0"  xyz="${0.5*scale} ${-0.4*scale} 0"/>
+          <origin rpy="0 0 0"  xyz="0 0 0"/>
           <geometry>
            	<mesh filename="package://usv_sim/meshes/simpleHull2/backLeft.obj" scale="${scale} ${scale} ${scale}"/>
@@ -87,5 +86,5 @@
         </visual>
         <collision>
-          <origin rpy="0 0 0"  xyz="${0.5*scale} ${-0.4*scale} 0"/>
+          <origin rpy="0 0 0"  xyz="0 0 0"/>
           <geometry>
            	<mesh filename="package://usv_sim/meshes/simpleHull2/backLeft.obj" scale="${scale} ${scale} ${scale}"/>
@@ -108,5 +107,5 @@
         <parent link="base_link"/>
         <child link="back_l_link"/>
-        <origin rpy="0 0 0" xyz="${-0.5*scale} ${0.4*scale} 0"/>
+        <origin rpy="0 0 0" xyz="${-0.5*scale} ${0.39*scale} 0"/>
 	<limit effort="50" velocity="5" lower="0" upper="0" />
             <dynamics damping="1.0"/>
@@ -115,5 +114,5 @@
     <link name="back_r_link">
     	<visual>
-          <origin rpy="0 0 0"  xyz="${0.5*scale} ${0.4*scale} 0"/>
+          <origin rpy="0 0 0"  xyz="0 0 0"/>
           <geometry>
            	<mesh filename="package://usv_sim/meshes/simpleHull2/backRight.obj" scale="${scale} ${scale} ${scale}"/>
@@ -121,5 +120,5 @@
     	</visual>
         <collision>
-          <origin rpy="0 0 0"  xyz="${0.5*scale} ${0.4*scale} 0"/>
+          <origin rpy="0 0 0"  xyz="0 0 0"/>
           <geometry>
            	<mesh filename="package://usv_sim/meshes/simpleHull2/backRight.obj" scale="${scale} ${scale} ${scale}"/>
@@ -142,5 +141,5 @@
         <parent link="base_link"/>
         <child link="back_r_link"/>
-        <origin rpy="0 0 0" xyz="${-0.5*scale} ${-0.4*scale} 0"/>
+        <origin rpy="0 0 0" xyz="${-0.5*scale} ${-0.39*scale} 0"/>
 	<limit effort="50" velocity="5" lower="0" upper="0" />
             <dynamics damping="1.0"/>
@@ -149,5 +148,5 @@
     <link name="front_l_link">
     	<visual>
-    	<origin rpy="0 0 0"  xyz="${-1.3*scale} ${-0.4*scale} 0"/>
+    	<origin rpy="0 0 0"  xyz="0 0 0"/>
           <geometry>
            	<mesh filename="package://usv_sim/meshes/simpleHull2/frontLeft.obj" scale="${scale} ${scale} ${scale}"/>
@@ -155,5 +154,5 @@
     	</visual>
         <collision>
-          <origin rpy="0 0 0"  xyz="${-1.3*scale} ${-0.4*scale} 0"/>
+          <origin rpy="0 0 0"  xyz="0 0 0"/>
           <geometry>
            	<mesh filename="package://usv_sim/meshes/simpleHull2/frontLeft.obj" scale="${scale} ${scale} ${scale}"/>
@@ -176,5 +175,5 @@
         <parent link="base_link"/>
         <child link="front_l_link"/>
-        <origin rpy="0 0 0" xyz="${1.3*scale} ${0.4*scale} 0"/>
+        <origin rpy="0 0 0" xyz="${1.3*scale} ${0.2*scale} 0"/>
 	<limit effort="50" velocity="5" lower="0" upper="0" />
             <dynamics damping="1.0"/>
@@ -189,7 +188,7 @@
         </visual>
         <collision>
-          <origin rpy="0 0 0"  xyz="${-1.3*scale} ${0.4*scale} 0"/>
-          <geometry>
-           	<mesh filename="package://usv_sim/meshes/simpleHull2/frontRight.obj" scale="${scale} ${scale} ${scale}"/>
+          <origin rpy="0 0 0"  xyz="${0*scale} ${0*scale} 0"/>
+          <geometry>
+           	<mesh filename="package://usv_sim/meshes/simpleHull2/frontRight.obj" scale="${2*scale} ${2*scale} ${2*scale}"/>
           </geometry>
         </collision>
@@ -210,5 +209,5 @@
         <parent link="base_link"/>
         <child link="front_r_link"/>
-        <origin rpy="0 0 0" xyz="1 0 0"/>
+        <origin rpy="0 0 0" xyz="${1.3*scale} ${-0.2*scale} 0"/>
 	<limit effort="50" velocity="5" lower="0" upper="0" />
             <dynamics damping="1.0"/>
@@ -295,7 +294,4 @@
                     <mesh filename="package://usv_sim/meshes/simpleHull/airPropeller.obj" scale="${scale} ${scale} ${scale}"/>
                 </geometry>
-                <material name="black">
-                    <color rgba="255 255 255 1"/>
-                </material>
             </visual>
             <inertial>

File: src/usv_sim/xacro/sailboat.xacro (robot description, xacro)
@@ -1,5 +1,5 @@
 <?xml version="1.0"?>
 <robot name="sailboat" xmlns:xacro="http://www.ros.org/wiki/xacro">
-    <xacro:include filename="$(find usv_sim)/xacro/boat_subdivided.xacro" />
+    <xacro:include filename="$(find usv_sim)/xacro/boat_subdivided3.xacro" />
     <xacro:rudder_xacro/>
     <!-- Defining sail model -->
