Commit message: Started test unification of plugins- keel, rudder and sail

File: src/usv_sim/xacro/airboat.xacro (robot description, xacro)
@@ -1,5 +1,5 @@
 <?xml version="1.0"?>
 <robot name="boat_rudder" xmlns:xacro="http://www.ros.org/wiki/xacro">
-    <xacro:include filename="$(find usv_sim)/xacro/boat_subdivided3.xacro" />
+    <xacro:include filename="$(find usv_sim)/xacro/boat_subdivided4.xacro" />
     <!-- Plugin list -->
     <gazebo>

File: src/usv_sim/xacro/boat_rudder.xacro (robot description, xacro)
@@ -1,5 +1,5 @@
 <?xml version="1.0"?>
 <robot name="boat_rudder" xmlns:xacro="http://www.ros.org/wiki/xacro">
-    <xacro:include filename="$(find usv_sim)/xacro/boat_subdivided3.xacro" />
+    <xacro:include filename="$(find usv_sim)/xacro/boat_subdivided4.xacro" />
     <xacro:rudder_xacro/>
     <!-- Plugin list -->

File: src/usv_sim/xacro/sailboat.xacro (robot description, xacro)
@@ -1,5 +1,5 @@
 <?xml version="1.0"?>
 <robot name="sailboat" xmlns:xacro="http://www.ros.org/wiki/xacro">
-    <xacro:include filename="$(find usv_sim)/xacro/boat_subdivided3.xacro" />
+    <xacro:include filename="$(find usv_sim)/xacro/boat_subdivided4.xacro" />
     <xacro:rudder_xacro/>
     <!-- Defining sail model -->
@@ -18,5 +18,5 @@
 	    <collision name="collision">
             <geometry>
-              <mesh filename="package://usv_sim/meshes/simpleHull/sail.obj" scale="0.5 0.5 0.5"/>
+              <mesh filename="package://usv_sim/meshes/simpleHull/sail.dae" scale="0.5 0.5 0.5"/>
             </geometry>
             <origin rpy="0 0 0" xyz="0 0 0"/>
@@ -24,5 +24,5 @@
 	    <visual name="visual">
             <geometry>
-              <mesh filename="package://usv_sim/meshes/simpleHull/sail.obj" scale="0.5 0.5 0.5"/>
+              <mesh filename="package://usv_sim/meshes/simpleHull/sail.dae" scale="0.5 0.5 0.5"/>
             </geometry>
             <origin rpy="0 0 0" xyz="0 0 0"/>
@@ -71,4 +71,53 @@
     <!-- Plugin list -->
   <gazebo>
+	<plugin name="usv_sail_plugin" filename="libusv_sailing_plugin.so">
+		<linkType>sail</linkType>
+		<a0>0</a0>
+		<cla>4.752798721</cla>
+		<cda>0.6417112299</cda>
+		<cma>-1.8</cma>
+		<alpha_stall>0.785</alpha_stall>
+		<cla_stall>-3.85</cla_stall>
+		<cda_stall>-0.9233984055</cda_stall>
+		<cma_stall>0</cma_stall>
+		<cp>0 0 0</cp>
+		<joint_name>sail_joint</joint_name>
+		<area>1.44</area>
+		<air_density>1.2041</air_density>
+		<forward>1 0 0</forward>
+		<upward>0 1 0</upward>
+		<link_name>sail</link_name>
+      </plugin>
+      <plugin name="usv_sail_plugin" filename="libusv_sailing_plugin.so">
+		  <linkType>keel</linkType>
+		  <a0>0</a0>
+		  <cla>0.752798721</cla>
+		  <cda>0.3417112299</cda>
+		  <alpha_stall>0.785</alpha_stall>
+		  <cla_stall>-0.85</cla_stall>
+		  <cda_stall>-0.3233984055</cda_stall>
+		  <cp>0 0 0</cp>
+		  <area>0.1</area>
+		  <air_density>1000</air_density>
+		  <forward>1 0 0</forward>
+		  <upward>0 1 0</upward>
+		  <link_name>keel</link_name>
+    </plugin>
+    <plugin name="usv_sail_plugin" filename="libusv_sailing_plugin.so">
+		<linkType>rudder</linkType>
+		<a0>0</a0>
+		<cla>0.752798721</cla>
+		<cda>0.3417112299</cda>
+		<alpha_stall>0.785</alpha_stall>
+		<cla_stall>-0.85</cla_stall>
+		<cda_stall>-0.3233984055</cda_stall>
+		<cp>0 0 0</cp>
+		<area>0.1</area>
+		<air_density>1000</air_density>
+		<forward>1 0 0</forward>
+		<upward>0 1 0</upward>
+		<link_name>rudder</link_name>
+      </plugin>
+      <!--
         <plugin name="sail_plugin" filename="libsail_plugin.so">
             <a0>0</a0>
@@ -116,4 +165,5 @@
           <link_name>rudder</link_name>
       </plugin>
+-->
       <plugin name="freefloating_gazebo_control" filename="libfreefloating_gazebo_control.so">
           <switchService>switch</switchService>

Commit message: airboat working on scenario2

File: src/usv_sim/xacro/airboat.xacro (robot description, xacro)
@@ -1,4 +1,4 @@
 <?xml version="1.0"?>
-<robot name="boat_rudder" xmlns:xacro="http://www.ros.org/wiki/xacro">
+<robot name="airboat" xmlns:xacro="http://www.ros.org/wiki/xacro">
     <xacro:include filename="$(find usv_sim)/xacro/boat_subdivided4.xacro" />
     <!-- Plugin list -->
@@ -10,6 +10,6 @@
             <link>fwd</link>
             <thruster>
-                <effortUnderWater>20</effortUnderWater>
-				<effortOverWater>30</effortOverWater>
+                <effortUnderWater>100</effortUnderWater>
+				<effortOverWater>100</effortOverWater>
                 <name>fwd</name>
             </thruster>
@@ -17,4 +17,4 @@
     </gazebo>
     <!-- Define one steering thruster, with assumed force control in Z-direction -->
-    <xacro:airthruster_link name="fwd" xyz="0 0.05 0.3" rpy="0 ${-PI/2} 0" effort="50" velocity="20" rotationAxis="1 0 0" lowerLimit="-${PI/4}" upperLimit="${PI/4}"/>
+    <xacro:airthruster_link name="fwd" xyz="0 0.05 0.3" rpy="0 ${-PI/2} 0" effort="100" velocity="20" rotationAxis="1 0 0" lowerLimit="-${PI/4}" upperLimit="${PI/4}"/>
 </robot>

File: src/usv_sim/xacro/boat_subdivided4.xacro (robot description, xacro)
@@ -286,5 +286,5 @@
     </xacro:macro>
     <!-- Thruster link -->
-    <xacro:macro name="airthruster_link" params="name xyz rpy rotationAxis effort:=50 velocity:=5 lowerLimit upperLimit parentLink:=back_r_link">
+    <xacro:macro name="airthruster_link" params="name xyz rpy rotationAxis effort:=100 velocity:=20 lowerLimit upperLimit parentLink:=back_r_link">
         <joint name="${name}_joint" type="revolute">
             <parent link="${parentLink}"/>
