Commit message: sail lift/drag improved

File: src/usv_sim/xacro/sailboat.xacro (robot description, xacro)
@@ -28,14 +28,46 @@
 	    </visual>
     </link>
+    <link name="keel">
+        <inertial>
+            <mass value="0.5" />
+            <inertia
+              ixx="0.05"
+              ixy="0.0"
+              iyy="0.05"
+              ixz="0.0"
+              iyz="0.0"
+              izz="0.005"/>
+        </inertial>
+        <collision name="collision">
+            <geometry>
+              <box size="0.1 0.02 0.4" />
+            </geometry>
+            <origin rpy="0 0 0" xyz="0 0 0"/>
+        </collision>
+        <visual name="visual">
+            <geometry>
+              <box size="0.1 0.02 0.4" />
+            </geometry>
+            <origin rpy="0 0 0" xyz="0 0 0"/>
+        </visual>
+    </link>
+    <joint name="keel_joint" type="revolute">
+        <parent link="base_link"/>
+        <child link="keel"/>
+        <origin rpy="0 0 0" xyz="0 0 -0.2"/>
+        <dynamics damping="1.0"/>
+        <axis xyz="0 0 1"/>
+        <limit effort="50" velocity="5" lower="0" upper="0" />
+    </joint>
     <joint name="sail_joint" type="revolute">
         <parent link="base_link"/>
         <child link="sail"/>
-        <origin rpy="0 0 ${PI/2}" xyz="0 0 +0.6"/>
+        <origin rpy="0 0 ${PI}" xyz="0 0 0.6"/>
         <dynamics damping="1.0"/>
         <axis xyz="0 0 1"/>
-        <limit effort="30" velocity="5" lower="-${PI/2}" upper="${PI/2}" />
+        <limit effort="30" velocity="5" lower="-${PI}" upper="${PI}" />
     </joint>
     <!-- Plugin list -->
-    <gazebo>
+  <gazebo>
         <plugin name="sail_plugin" filename="libsail_plugin.so">
             <a0>0</a0>
@@ -67,5 +99,5 @@
             <cla_stall>-0.85</cla_stall>
             <cda_stall>-0.3233984055</cda_stall>
-            <cp>-0.5 0 0</cp>
+            <cp>0 0 0</cp>
             <area>0.03</area>
             <air_density>1000</air_density>

Commit message: teste

File: src/usv_sim/xacro/sailboat.xacro (robot description, xacro)
@@ -66,5 +66,5 @@
         <dynamics damping="1.0"/>
         <axis xyz="0 0 1"/>
-        <limit effort="30" velocity="5" lower="-${PI}" upper="${PI}" />
+        <limit effort="30" velocity="5" lower="-${PI/2}" upper="${PI/2}" />
     </joint>
     <!-- Plugin list -->
@@ -106,4 +106,22 @@
             <link_name>rudder</link_name>
         </plugin>
+        <plugin name="keel_plugin" filename="librudder_plugin.so">
+            <a0>0</a0>
+            <cla>0.752798721</cla>
+            <cda>0.3417112299</cda>
+            <!--
+            <cma>-1.8</cma> momentum
+            <cma_stall>0</cma_stall>
+            -->
+            <alpha_stall>0.785</alpha_stall>
+            <cla_stall>-0.85</cla_stall>
+            <cda_stall>-0.3233984055</cda_stall>
+            <cp>0 0 0</cp>
+            <area>0.1</area>
+            <air_density>1000</air_density>
+            <forward>1 0 0</forward>
+            <upward>0 1 0</upward>
+            <link_name>keel</link_name>
+        </plugin>
         <plugin name="freefloating_gazebo_control" filename="libfreefloating_gazebo_control.so">
             <switchService>switch</switchService>

Commit message: more realistic sailboat movement

File: src/usv_sim/xacro/sailboat.xacro (robot description, xacro)
@@ -22,4 +22,5 @@
 	    </collision>
 	    <visual name="visual">
+            <plugin name="some_visual_plugin" filename="some_visual_plugin.so"/>
             <geometry>
               <box size="0.4 0.02 1" />
@@ -30,5 +31,5 @@
     <link name="keel">
         <inertial>
-            <mass value="0.5" />
+            <mass value="50" />
             <inertia
               ixx="0.05"
@@ -63,5 +64,5 @@
         <parent link="base_link"/>
         <child link="sail"/>
-        <origin rpy="0 0 ${PI}" xyz="0 0 0.6"/>
+        <origin rpy="0 0 0" xyz="0 0 0.6"/>
         <dynamics damping="1.0"/>
         <axis xyz="0 0 1"/>
@@ -79,5 +80,5 @@
             <cda_stall>-0.9233984055</cda_stall>
             <cma_stall>0</cma_stall>
-            <cp>0 0 0</cp>
+            <cp>0 0 -0.4</cp>
             <area>0.4</area>
             <air_density>1.2041</air_density>
@@ -88,45 +89,45 @@
             <!--<control_joint_rad_to_cl>4.0</control_joint_rad_to_cl>-->
       </plugin>
-        <plugin name="rudder_plugin" filename="librudder_plugin.so">
-            <a0>0</a0>
-            <cla>0.752798721</cla>
-            <cda>0.3417112299</cda>
-            <!--
-            <cma>-1.8</cma> momentum
-            <cma_stall>0</cma_stall>
-            -->
-            <alpha_stall>0.785</alpha_stall>
-            <cla_stall>-0.85</cla_stall>
-            <cda_stall>-0.3233984055</cda_stall>
-            <cp>0 0 0</cp>
-            <area>0.03</area>
-            <air_density>1000</air_density>
-            <forward>1 0 0</forward>
-            <upward>0 1 0</upward>
-            <link_name>rudder</link_name>
-        </plugin>
-        <plugin name="keel_plugin" filename="librudder_plugin.so">
-            <a0>0</a0>
-            <cla>0.752798721</cla>
-            <cda>0.3417112299</cda>
-            <!--
-            <cma>-1.8</cma> momentum
-            <cma_stall>0</cma_stall>
-            -->
-            <alpha_stall>0.785</alpha_stall>
-            <cla_stall>-0.85</cla_stall>
-            <cda_stall>-0.3233984055</cda_stall>
-            <cp>0 0 0</cp>
-            <area>0.1</area>
-            <air_density>1000</air_density>
-            <forward>1 0 0</forward>
-            <upward>0 1 0</upward>
-            <link_name>keel</link_name>
-        </plugin>
-        <plugin name="freefloating_gazebo_control" filename="libfreefloating_gazebo_control.so">
-            <switchService>switch</switchService>
-            <updateRate>100</updateRate>
-            <link>base_link</link>
-        </plugin>
+      <plugin name="keel_plugin" filename="libkeel_plugin.so">
+          <a0>0</a0>
+          <cla>0.752798721</cla>
+          <cda>0.3417112299</cda>
+          <!--
+          <cma>-1.8</cma> momentum
+          <cma_stall>0</cma_stall>
+          -->
+          <alpha_stall>0.785</alpha_stall>
+          <cla_stall>-0.85</cla_stall>
+          <cda_stall>-0.3233984055</cda_stall>
+          <cp>0 0 0</cp>
+          <area>0.1</area>
+          <air_density>1000</air_density>
+          <forward>1 0 0</forward>
+          <upward>0 1 0</upward>
+          <link_name>keel</link_name>
+    </plugin>
+    <plugin name="rudder_plugin" filename="librudder_plugin.so">
+          <a0>0</a0>
+          <cla>0.752798721</cla>
+          <cda>0.3417112299</cda>
+          <!--
+          <cma>-1.8</cma> momentum
+          <cma_stall>0</cma_stall>
+          -->
+          <alpha_stall>0.785</alpha_stall>
+          <cla_stall>-0.85</cla_stall>
+          <cda_stall>-0.3233984055</cda_stall>
+          <cp>0 0 0</cp>
+          <area>0.1</area>
+          <air_density>1000</air_density>
+          <forward>1 0 0</forward>
+          <upward>0 1 0</upward>
+          <link_name>rudder</link_name>
+      </plugin>
+      <plugin name="freefloating_gazebo_control" filename="libfreefloating_gazebo_control.so">
+          <switchService>switch</switchService>
+          <updateRate>100</updateRate>
+          <link>base_link</link>
+      </plugin>
   </gazebo>
 </robot>

Commit message: expanded readme.me

File: src/usv_sim/xacro/sailboat.xacro (robot description, xacro)
@@ -29,36 +29,4 @@
 	    </visual>
     </link>
-    <link name="keel">
-        <inertial>
-            <mass value="50" />
-            <inertia
-              ixx="0.05"
-              ixy="0.0"
-              iyy="0.05"
-              ixz="0.0"
-              iyz="0.0"
-              izz="0.005"/>
-        </inertial>
-        <collision name="collision">
-            <geometry>
-              <box size="0.1 0.02 0.4" />
-            </geometry>
-            <origin rpy="0 0 0" xyz="0 0 0"/>
-        </collision>
-        <visual name="visual">
-            <geometry>
-              <box size="0.1 0.02 0.4" />
-            </geometry>
-            <origin rpy="0 0 0" xyz="0 0 0"/>
-        </visual>
-    </link>
-    <joint name="keel_joint" type="revolute">
-        <parent link="base_link"/>
-        <child link="keel"/>
-        <origin rpy="0 0 0" xyz="0 0 -0.2"/>
-        <dynamics damping="1.0"/>
-        <axis xyz="0 0 1"/>
-        <limit effort="50" velocity="5" lower="0" upper="0" />
-    </joint>
     <joint name="sail_joint" type="revolute">
         <parent link="base_link"/>

Commit message: Updated usv_wind_current

File: src/usv_sim/xacro/sailboat.xacro (robot description, xacro)
@@ -1,4 +1,5 @@
 <?xml version="1.0"?>
 <robot name="sailboat" xmlns:xacro="http://www.ros.org/wiki/xacro">
+    <xacro:property name="windType" value="global"/>
     <xacro:include filename="$(find usv_sim)/xacro/boat_subdivided4.xacro" />
     <xacro:rudder_xacro/>
@@ -88,5 +89,5 @@
 		<upward>0 1 0</upward>
 		<link_name>sail</link_name>
-		<fluidVelocity>local</fluidVelocity>
+		<fluidVelocity>${windType}</fluidVelocity>
       </plugin>
       <plugin name="usv_sail_plugin" filename="libusv_sailing_plugin.so">

Commit message: removed sailboat/angleLimits. now moving sail with sailboat/joint_setpoit

File: src/usv_sim/xacro/sailboat.xacro (robot description, xacro)
@@ -36,5 +36,5 @@
         <dynamics damping="1.0"/>
         <axis xyz="0 0 1"/>
-        <limit effort="50" velocity="5" lower="-1.5" upper="1.5" />
+        <limit effort="500000" velocity="5" lower="-${PI}" upper="${PI}" />
     </joint>
     <link name="keel">
