Commit message: Updated UML diagram

File: src/usv_sim/xacro/boat_subdivided4.xacro (robot description, xacro)
@@ -4,6 +4,6 @@
     <!-- Body properties -->
     <xacro:property name="front_body_mass" value="5"/>
-    <xacro:property name="back_body_mass" value="15"/>
-    <xacro:property name="middle_body_mass" value="10"/>
+    <xacro:property name="back_body_mass" value="5"/>
+    <xacro:property name="middle_body_mass" value="5"/>
     <xacro:property name="rear_body_mass" value="5"/>
     <xacro:property name="front_body_mass" value="2"/>
@@ -379,5 +379,5 @@
         <sensor type="gpu_ray" name="head_hokuyo_sensor">
         <pose>0 0 0 0 0 0</pose>
-        <visualize>true</visualize>
+        <visualize>false</visualize>
         <update_rate>40</update_rate>
         <ray>

File: src/usv_sim/xacro/sailboat.xacro (robot description, xacro)
@@ -7,5 +7,5 @@
 		<inertial>
 		    	<origin rpy="0 0 0" xyz="-0.3 0 0.4"/>
-			<mass value="0.1" />
+			<mass value="1" />
 			<inertia
 			  ixx="0.4708"

Commit message: Updated readme.

File: src/usv_sim/xacro/boat_subdivided4.xacro (robot description, xacro)
@@ -288,5 +288,5 @@
                 <origin xyz="0 0 0" rpy="0 0 0" />
                 <geometry>
-                    	<mesh filename="package://usv_sim/meshes/simpleHull/airPropeller.dae" scale="${scale} ${scale} ${scale}"/>
+                    	<mesh filename="package://usv_sim/meshes/simpleHull3/airPropeller.dae" scale="${scale} ${scale} ${scale}"/>
                 </geometry>
             </visual>

File: src/usv_sim/xacro/sailboat.xacro (robot description, xacro)
@@ -18,5 +18,5 @@
 	    <collision name="collision">
             <geometry>
-              <mesh filename="package://usv_sim/meshes/simpleHull/sail.dae" scale="0.5 0.5 0.5"/>
+              <mesh filename="package://usv_sim/meshes/simpleHull3/sail.dae" scale="0.5 0.5 0.5"/>
             </geometry>
             <origin rpy="0 0 0" xyz="0 0 0"/>
@@ -24,5 +24,5 @@
 	    <visual name="visual">
             <geometry>
-              <mesh filename="package://usv_sim/meshes/simpleHull/sail.dae" scale="0.5 0.5 0.5"/>
+              <mesh filename="package://usv_sim/meshes/simpleHull3/sail.dae" scale="0.5 0.5 0.5"/>
             </geometry>
             <origin rpy="0 0 0" xyz="0 0 0"/>

Commit message: Wind started to affect boat hulls

File: src/usv_sim/xacro/boat_subdivided4.xacro (robot description, xacro)
@@ -33,9 +33,13 @@
         </inertial>
         <buoyancy>
-          <compensation>${middle_water_displaced_mass/middle_body_mass}</compensation>
-          <origin xyz="${0.35*scale} ${0.44*scale} ${-0.15*scale}"/>
-          <limit radius="0.1"/>
-          <damping rpy="20 20 20" xyz="20 40 50"/>
-	  <fluidVelocity>local</fluidVelocity>
+			<compensation>${middle_water_displaced_mass/middle_body_mass}</compensation>
+			<origin xyz="${0.35*scale} ${0.44*scale} ${-0.15*scale}"/>
+			<limit radius="0.1"/>
+			<damping rpy="20 20 20" xyz="20 40 50"/>
+         	<windVelocity>global</windVelocity>
+			<frontal_area>0.0</frontal_area>
+			<lateral_area>0.06</lateral_area>
+			<lateral_length>1.2</lateral_length>
+	  		<fluidVelocity>local</fluidVelocity>
         </buoyancy>
     </link>
@@ -63,4 +67,8 @@
           <limit radius="0.1"/>
           <damping rpy="20 20 20" xyz="20 40 50"/>
+			<windVelocity>global</windVelocity>
+			<frontal_area>0.0</frontal_area>
+			<lateral_area>0.06</lateral_area>
+			<lateral_length>1.2</lateral_length>
 	  <fluidVelocity>local</fluidVelocity>
         </buoyancy>
@@ -93,9 +101,13 @@
         </inertial>
         <buoyancy>
-          <compensation>${back_water_displaced_mass/back_body_mass}</compensation>
-          <origin xyz="${-0.6*scale} 0 ${-0.15*scale}"/>
-          <limit radius="0.1"/>
-          <damping rpy="20 20 20" xyz="20 40 50"/>
-	  <fluidVelocity>local</fluidVelocity>
+			<compensation>${back_water_displaced_mass/back_body_mass}</compensation>
+			<origin xyz="${-0.6*scale} 0 ${-0.15*scale}"/>
+			<limit radius="0.1"/>
+			<damping rpy="20 20 20" xyz="20 40 50"/>
+			<windVelocity>global</windVelocity>
+			<frontal_area>0.04</frontal_area>
+			<lateral_area>0.06</lateral_area>
+			<lateral_length>1.2</lateral_length>
+	  		<fluidVelocity>local</fluidVelocity>
         </buoyancy>
     </link>
@@ -127,9 +139,13 @@
         </inertial>
         <buoyancy>
-          <compensation>${back_water_displaced_mass/back_body_mass}</compensation>
-          <origin xyz="${-0.6*scale} 0 ${-0.15*scale}"/>
-          <limit radius="0.1"/>
-          <damping rpy="20 20 20" xyz="20 40 50"/>
-	  <fluidVelocity>local</fluidVelocity>
+          	<compensation>${back_water_displaced_mass/back_body_mass}</compensation>
+          	<origin xyz="${-0.6*scale} 0 ${-0.15*scale}"/>
+          	<limit radius="0.1"/>
+          	<damping rpy="20 20 20" xyz="20 40 50"/>
+          	<windVelocity>global</windVelocity>
+			<frontal_area>0.04</frontal_area>
+			<lateral_area>0.06</lateral_area>
+			<lateral_length>1.2</lateral_length>
+	  		<fluidVelocity>local</fluidVelocity>
         </buoyancy>
     </link>
@@ -153,4 +169,42 @@
           <geometry>
            	<mesh filename="package://usv_sim/meshes/simpleHull3/frontLeft.dae" scale="${scale} ${scale} ${scale}"/>
+          </geometry>
+        </collision>
+        <inertial>
+            <origin rpy="0 0 0" xyz="${0.4*scale} 0 ${-0.1*scale}"/>
+          <mass value="${front_body_mass}"/>
+          <inertia ixx="0.1" ixy="0.0" ixz="0.0" iyy="1.4" iyz="0.0" izz="1.4"/>
+        </inertial>
+        <buoyancy>
+          	<compensation>${front_water_displaced_mass/front_body_mass}</compensation>
+          	<origin xyz="${0.4*scale} 0 ${-0.05*scale}"/>
+          	<limit radius="0.1"/>
+          	<damping rpy="20 20 20" xyz="20 40 50"/>
+          	<windVelocity>global</windVelocity>
+			<frontal_area>0.04</frontal_area>
+			<lateral_area>0.06</lateral_area>
+			<lateral_length>1.2</lateral_length>
+	  		<fluidVelocity>local</fluidVelocity>
+        </buoyancy>
+    </link>
+    <joint name="front_l_joint" type="revolute">
+        <parent link="base_link"/>
+        <child link="front_l_link"/>
+        <origin rpy="0 0 0" xyz="${1.3*scale} ${0.2*scale} 0"/>
+	<limit effort="50" velocity="5" lower="0" upper="0" />
+            <dynamics damping="1.0"/>
+            <axis xyz="1 0 0"/>
+    </joint>
+    <link name="front_r_link">
+    	<visual>
+    		<origin rpy="0 0 0"  xyz="0 0 0"/>
+          <geometry>
+           	<mesh filename="package://usv_sim/meshes/simpleHull3/frontRight.dae" scale="${scale} ${scale} ${scale}"/>
+          </geometry>
+        </visual>
+        <collision>
+          <origin rpy="0 0 0"  xyz="${0*scale} ${0*scale} 0"/>
+          <geometry>
+           	<mesh filename="package://usv_sim/meshes/simpleHull3/frontRight.dae" scale="${2*scale} ${2*scale} ${2*scale}"/>
           </geometry>
         </collision>
@@ -165,38 +219,5 @@
           <limit radius="0.1"/>
           <damping rpy="20 20 20" xyz="20 40 50"/>
-	  <fluidVelocity>local</fluidVelocity>
-        </buoyancy>
-    </link>
-    <joint name="front_l_joint" type="revolute">
-        <parent link="base_link"/>
-        <child link="front_l_link"/>
-        <origin rpy="0 0 0" xyz="${1.3*scale} ${0.2*scale} 0"/>
-	<limit effort="50" velocity="5" lower="0" upper="0" />
-            <dynamics damping="1.0"/>
-            <axis xyz="1 0 0"/>
-    </joint>
-    <link name="front_r_link">
-    	<visual>
-    		<origin rpy="0 0 0"  xyz="0 0 0"/>
-          <geometry>
-           	<mesh filename="package://usv_sim/meshes/simpleHull3/frontRight.dae" scale="${scale} ${scale} ${scale}"/>
-          </geometry>
-        </visual>
-        <collision>
-          <origin rpy="0 0 0"  xyz="${0*scale} ${0*scale} 0"/>
-          <geometry>
-           	<mesh filename="package://usv_sim/meshes/simpleHull3/frontRight.dae" scale="${2*scale} ${2*scale} ${2*scale}"/>
-          </geometry>
-        </collision>
-        <inertial>
-            <origin rpy="0 0 0" xyz="${0.4*scale} 0 ${-0.1*scale}"/>
-          <mass value="${front_body_mass}"/>
-          <inertia ixx="0.1" ixy="0.0" ixz="0.0" iyy="1.4" iyz="0.0" izz="1.4"/>
-        </inertial>
-        <buoyancy>
-          <compensation>${front_water_displaced_mass/front_body_mass}</compensation>
-          <origin xyz="${0.4*scale} 0 ${-0.05*scale}"/>
-          <limit radius="0.1"/>
-          <damping rpy="20 20 20" xyz="20 40 50"/>
+          <windVelocity>global</windVelocity>
 	  <fluidVelocity>local</fluidVelocity>
         </buoyancy>

Commit message: Added all scripts, launchs and xml to scenario 1, 2 and 3

File: src/usv_sim/xacro/boat_subdivided4.xacro (robot description, xacro)
@@ -206,5 +206,5 @@
           <origin rpy="0 0 0"  xyz="${0*scale} ${0*scale} 0"/>
           <geometry>
-           	<mesh filename="package://usv_sim/meshes/simpleHull3/frontRight.dae" scale="${2*scale} ${2*scale} ${2*scale}"/>
+           	<mesh filename="package://usv_sim/meshes/simpleHull3/frontRight.dae" scale="${scale} ${scale} ${scale}"/>
           </geometry>
         </collision>
@@ -247,5 +247,5 @@
 	    	</buoyancy>
 	    	<collision>
-          		<origin xyz="0 0 0" rpy="${-0.15*scale} 0 ${0.3*scale}"/>
+          		<origin xyz="${-0.15*scale} 0 ${0*scale}" rpy="0 0 0"/>
           		<geometry>
           		    <mesh filename="package://usv_sim/meshes/simpleHull3/thruster.dae" scale="${scale} ${scale} ${scale}"/>
@@ -253,5 +253,5 @@
         	</collision>
             <visual name="${name}">
-                <origin xyz="0 0 0" rpy="0 0 0" />
+                <origin xyz="${-0.15*scale} 0 ${0*scale}" rpy="0 0 0" />
                 <geometry>
                     <mesh filename="package://usv_sim/meshes/simpleHull3/thruster.dae" scale="${scale} ${scale} ${scale}"/>
@@ -364,5 +364,5 @@
             <parent link="back_r_link"/>
             <child link="rudder"/>
-            <origin rpy="0 0 0" xyz="${-1.4*scale} ${0.22*scale} ${-0.5*scale}"/>
+            <origin rpy="0 0 0" xyz="${-1.4*scale} ${0.35*scale} ${-0.5*scale}"/>
             <dynamics damping="1.0"/>
             <axis xyz="0 0 1"/>

File: src/usv_sim/xacro/rudderboat.xacro (robot description, xacro)
@@ -32,4 +32,4 @@
     </gazebo>
     <!-- Define two steering thrusters, with assumed force control in Z-direction -->
-    <xacro:thruster_link name="fwd" xyz="-0.3 0.07 -0.15" rpy="0 ${-PI/2} 0" rotationAxis="1 0 0" lowerLimit="0" upperLimit="0" />
+    <xacro:thruster_link name="fwd" xyz="-0.45 0.10 -0.15" rpy="0 ${-PI/2} 0" rotationAxis="1 0 0" lowerLimit="0" upperLimit="0" />
 </robot>

Commit message: Fixed topic publisher of freefloating_gazebo

File: src/usv_sim/xacro/boat_subdivided4.xacro (robot description, xacro)
@@ -367,5 +367,5 @@
             <dynamics damping="1.0"/>
             <axis xyz="0 0 1"/>
-            <limit effort="50" velocity="5" lower="-${PI/3}" upper="${PI/3}" />
+            <limit effort="100" velocity="5" lower="-${PI/2}" upper="${PI/2}" />
         </joint>
     </xacro:macro>

Commit message: Updated simulator

File: src/usv_sim/xacro/boat_subdivided4.xacro (robot description, xacro)
@@ -14,4 +14,6 @@
     <xacro:property name="bl1" value=".1" />
     <xacro:property name="bl2" value=".1" />
+    <xacro:property name="windType" value="none" />
+    <xacro:property name="waterType" value="none" />
     <link name="base_link">
         <visual>
@@ -37,9 +39,9 @@
 			<limit radius="0.1"/>
 			<damping rpy="20 20 20" xyz="20 40 50"/>
-         	<windVelocity>global</windVelocity>
+         	<windVelocity>${windType}</windVelocity>
 			<frontal_area>0.0</frontal_area>
 			<lateral_area>0.06</lateral_area>
 			<lateral_length>1.2</lateral_length>
-	  		<fluidVelocity>global</fluidVelocity>
+	  		<fluidVelocity>${waterType}</fluidVelocity>
         </buoyancy>
     </link>
@@ -67,9 +69,9 @@
           <limit radius="0.1"/>
           <damping rpy="20 20 20" xyz="20 40 50"/>
-			<windVelocity>global</windVelocity>
+			<windVelocity>${windType}</windVelocity>
 			<frontal_area>0.0</frontal_area>
 			<lateral_area>0.06</lateral_area>
 			<lateral_length>1.2</lateral_length>
-	  <fluidVelocity>global</fluidVelocity>
+	  <fluidVelocity>${waterType}</fluidVelocity>
         </buoyancy>
     </link>
@@ -105,9 +107,9 @@
 			<limit radius="0.1"/>
 			<damping rpy="20 20 20" xyz="20 40 50"/>
-			<windVelocity>global</windVelocity>
+			<windVelocity>${windType}</windVelocity>
 			<frontal_area>0.04</frontal_area>
 			<lateral_area>0.06</lateral_area>
 			<lateral_length>1.2</lateral_length>
-	  		<fluidVelocity>global</fluidVelocity>
+	  		<fluidVelocity>${waterType}</fluidVelocity>
         </buoyancy>
     </link>
@@ -143,9 +145,9 @@
           	<limit radius="0.1"/>
           	<damping rpy="20 20 20" xyz="20 40 50"/>
-          	<windVelocity>global</windVelocity>
+          	<windVelocity>${windType}</windVelocity>
 			<frontal_area>0.04</frontal_area>
 			<lateral_area>0.06</lateral_area>
 			<lateral_length>1.2</lateral_length>
-	  		<fluidVelocity>global</fluidVelocity>
+	  		<fluidVelocity>${waterType}</fluidVelocity>
         </buoyancy>
     </link>
@@ -181,9 +183,9 @@
           	<limit radius="0.1"/>
           	<damping rpy="20 20 20" xyz="20 40 50"/>
-          	<windVelocity>global</windVelocity>
+          	<windVelocity>${windType}</windVelocity>
 			<frontal_area>0.04</frontal_area>
 			<lateral_area>0.06</lateral_area>
 			<lateral_length>1.2</lateral_length>
-	  		<fluidVelocity>global</fluidVelocity>
+	  		<fluidVelocity>${waterType}</fluidVelocity>
         </buoyancy>
     </link>
@@ -219,6 +221,6 @@
           <limit radius="0.1"/>
           <damping rpy="20 20 20" xyz="20 40 50"/>
-          <windVelocity>global</windVelocity>
-	  <fluidVelocity>global</fluidVelocity>
+          <windVelocity>${windType}</windVelocity>
+	  <fluidVelocity>${waterType}</fluidVelocity>
         </buoyancy>
     </link>
@@ -244,5 +246,5 @@
             <buoyancy>
 				<compensation>0.8</compensation>
-	        	<fluidVelocity>global</fluidVelocity>
+	        	<fluidVelocity>${windType}</fluidVelocity>
 	    	</buoyancy>
 	    	<collision>
@@ -298,5 +300,5 @@
             <buoyancy>
 				<compensation>1.0</compensation>
-	        	<fluidVelocity>global</fluidVelocity>
+	        	<fluidVelocity>${waterType}</fluidVelocity>
 	    	</buoyancy>
 	    	<collision>

File: src/usv_sim/xacro/sailboat.xacro (robot description, xacro)
@@ -40,5 +40,5 @@
     <link name="keel">
 	<inertial>
-		<mass value="20" />
+		<mass value="5" />
 		<inertia
 		  ixx="0.4708"
@@ -75,6 +75,6 @@
 		<link_type>sail</link_type>
 		<a0>0</a0>
-		<cla>4.752798721</cla>
-		<cda>0.6417112299</cda>
+		<cla>3.0</cla>
+		<cda>3.0</cda>
 		<cma>-1.8</cma>
 		<alpha_stall>0.785</alpha_stall>
@@ -86,5 +86,5 @@
 		<area>1.44</area>
 		<air_density>1.2041</air_density>
-		<forward>1 0 0</forward>
+		<forward>-1 0 0</forward>
 		<upward>0 1 0</upward>
 		<link_name>sail</link_name>
@@ -94,11 +94,11 @@
 		  <link_type>keel</link_type>
 		  <a0>0</a0>
-		  <cla>0.752798721</cla>
-		  <cda>0.3417112299</cda>
+		  <cla>10.0</cla>
+		  <cda>8.0</cda>
 		  <alpha_stall>0.785</alpha_stall>
-		  <cla_stall>-0.85</cla_stall>
-		  <cda_stall>-0.3233984055</cda_stall>
+		  <cla_stall>-10.0</cla_stall>
+		  <cda_stall>-5.0</cda_stall>
 		  <cp>0 0 0</cp>
-		  <area>0.1</area>
+		  <area>1.0</area>
 		  <air_density>1000</air_density>
 		  <forward>1 0 0</forward>
@@ -110,6 +110,6 @@
 		<link_type>rudder</link_type>
 		<a0>0</a0>
-		<cla>0.752798721</cla>
-		<cda>0.3417112299</cda>
+		<cla>0.8</cla>
+		<cda>0.3</cda>
 		<alpha_stall>0.785</alpha_stall>
 		<cla_stall>-0.85</cla_stall>

Commit message: Update

File: src/usv_sim/xacro/boat_subdivided4.xacro (robot description, xacro)
@@ -14,6 +14,6 @@
     <xacro:property name="bl1" value=".1" />
     <xacro:property name="bl2" value=".1" />
-    <xacro:property name="windType" value="none" />
-    <xacro:property name="waterType" value="none" />
+    <xacro:property name="windType" value="global" />
+    <xacro:property name="waterType" value="global" />
     <link name="base_link">
         <visual>
@@ -341,5 +341,5 @@
         <link name="rudder">
             <inertial>
-                <mass value="0.05" />
+                <mass value="1" />
                 <inertia
                   ixx="0.05"
@@ -366,5 +366,5 @@
             <parent link="back_r_link"/>
             <child link="rudder"/>
-            <origin rpy="0 0 0" xyz="${-1.4*scale} ${0.35*scale} ${-0.5*scale}"/>
+            <origin rpy="0 0 0" xyz="${-1.4*scale} ${0.39*scale} ${-0.5*scale}"/>
             <dynamics damping="1.0"/>
             <axis xyz="0 0 1"/>

File: src/usv_sim/xacro/rudderboat.xacro (robot description, xacro)
@@ -8,13 +8,9 @@
 	<plugin name="usv_sail_plugin" filename="libusv_sailing_plugin.so">
 		<link_type>rudder</link_type>
-		<a0>0</a0>
-		<cla>0.752798721</cla>
-		<cda>0.3417112299</cda>
-		<alpha_stall>0.785</alpha_stall>
-		<cla_stall>-0.85</cla_stall>
-		<cda_stall>-0.3233984055</cda_stall>
-		<cp>-0.5 0 0</cp>
-		<area>0.06</area>
-		<air_density>1000</air_density>
+		<mult_lift>1.5</mult_lift>
+		<mult_drag>1</mult_drag>
+		<cp>-0.2 0 0</cp>
+		<area>0.02</area>
+		<fluid_density>1000</fluid_density>
 		<forward>1 0 0</forward>
 		<upward>0 1 0</upward>
@@ -32,4 +28,4 @@
     </gazebo>
     <!-- Define two steering thrusters, with assumed force control in Z-direction -->
-    <xacro:thruster_link name="fwd" xyz="-0.45 0.10 -0.15" rpy="0 ${-PI/2} 0" rotationAxis="1 0 0" lowerLimit="0" upperLimit="0" />
+    <xacro:thruster_link name="fwd" xyz="-0.45 0.117 -0.15" rpy="0 ${-PI/2} 0" rotationAxis="1 0 0" lowerLimit="0" upperLimit="0" />
 </robot>

Commit message: Updating some scenarios

File: src/usv_sim/xacro/boat_subdivided4.xacro (robot description, xacro)
@@ -14,6 +14,6 @@
     <xacro:property name="bl1" value=".1" />
     <xacro:property name="bl2" value=".1" />
-    <xacro:property name="windType" value="global" />
-    <xacro:property name="waterType" value="global" />
+    <xacro:property name="windType" value="local" />
+    <xacro:property name="waterType" value="local" />
     <link name="base_link">
         <visual>
@@ -38,5 +38,5 @@
 			<origin xyz="${0.35*scale} ${0.44*scale} ${-0.15*scale}"/>
 			<limit radius="0.1"/>
-			<damping rpy="20 20 20" xyz="20 40 50"/>
+			<damping rpy="20 20 20" xyz="20 40 25"/>
          	<windVelocity>${windType}</windVelocity>
 			<frontal_area>0.0</frontal_area>
@@ -68,5 +68,5 @@
           <origin xyz="${0.35*scale} ${-0.44*scale} ${-0.15*scale}"/>
           <limit radius="0.1"/>
-          <damping rpy="20 20 20" xyz="20 40 50"/>
+          <damping rpy="20 20 20" xyz="20 40 25"/>
 			<windVelocity>${windType}</windVelocity>
 			<frontal_area>0.0</frontal_area>
@@ -106,5 +106,5 @@
 			<origin xyz="${-0.6*scale} 0 ${-0.15*scale}"/>
 			<limit radius="0.1"/>
-			<damping rpy="20 20 20" xyz="20 40 50"/>
+			<damping rpy="20 20 20" xyz="20 40 25"/>
 			<windVelocity>${windType}</windVelocity>
 			<frontal_area>0.04</frontal_area>
@@ -144,5 +144,5 @@
           	<origin xyz="${-0.6*scale} 0 ${-0.15*scale}"/>
           	<limit radius="0.1"/>
-          	<damping rpy="20 20 20" xyz="20 40 50"/>
+          	<damping rpy="20 20 20" xyz="20 40 25"/>
           	<windVelocity>${windType}</windVelocity>
 			<frontal_area>0.04</frontal_area>
@@ -182,5 +182,5 @@
           	<origin xyz="${0.4*scale} 0 ${-0.05*scale}"/>
           	<limit radius="0.1"/>
-          	<damping rpy="20 20 20" xyz="20 40 50"/>
+          	<damping rpy="20 20 20" xyz="20 40 25"/>
           	<windVelocity>${windType}</windVelocity>
 			<frontal_area>0.04</frontal_area>
@@ -220,5 +220,5 @@
           <origin xyz="${0.4*scale} 0 ${-0.05*scale}"/>
           <limit radius="0.1"/>
-          <damping rpy="20 20 20" xyz="20 40 50"/>
+          <damping rpy="20 20 20" xyz="20 40 25"/>
           <windVelocity>${windType}</windVelocity>
 	  <fluidVelocity>${waterType}</fluidVelocity>

File: src/usv_sim/xacro/rudderboat.xacro (robot description, xacro)
@@ -11,5 +11,5 @@
 		<mult_drag>1</mult_drag>
 		<cp>-0.2 0 0</cp>
-		<area>0.02</area>
+		<area>0.025</area>
 		<fluid_density>1000</fluid_density>
 		<forward>1 0 0</forward>

Commit message: Changed parameters sailboat

File: src/usv_sim/xacro/boat_subdivided4.xacro (robot description, xacro)
@@ -14,5 +14,5 @@
     <xacro:property name="bl1" value=".1" />
     <xacro:property name="bl2" value=".1" />
-    <xacro:property name="windType" value="local" />
+    <xacro:property name="windType" value="global" />
     <xacro:property name="waterType" value="local" />
     <link name="base_link">

File: src/usv_sim/xacro/sailboat.xacro (robot description, xacro)
@@ -85,5 +85,5 @@
 		<joint_name>sail_joint</joint_name>
 		<area>1.44</area>
-		<air_density>1.2041</air_density>
+		<fluid_density>1.2041</fluid_density>
 		<forward>-1 0 0</forward>
 		<upward>0 1 0</upward>
@@ -101,5 +101,5 @@
 		  <cp>0 0 0</cp>
 		  <area>1.0</area>
-		  <air_density>1000</air_density>
+		  <fluid_density>1000</fluid_density>
 		  <forward>1 0 0</forward>
 		  <upward>0 1 0</upward>
@@ -117,5 +117,5 @@
 		<cp>0 0 0</cp>
 		<area>1</area>
-		<air_density>1000</air_density>
+		<fluid_density>1000</fluid_density>
 		<forward>1 0 0</forward>
 		<upward>0 1 0</upward>

Commit message: Changed parameters sailboat

File: src/usv_sim/xacro/boat_subdivided4.xacro (robot description, xacro)
@@ -14,5 +14,5 @@
     <xacro:property name="bl1" value=".1" />
     <xacro:property name="bl2" value=".1" />
-    <xacro:property name="windType" value="global" />
+    <xacro:property name="windType" value="local" />
     <xacro:property name="waterType" value="local" />
     <link name="base_link">

Commit message: Added scenario named flooding1

File: src/usv_sim/xacro/boat_subdivided4.xacro (robot description, xacro)
@@ -14,6 +14,6 @@
     <xacro:property name="bl1" value=".1" />
     <xacro:property name="bl2" value=".1" />
-    <xacro:property name="windType" value="local" />
-    <xacro:property name="waterType" value="local" />
+    <xacro:property name="windType" value="none" />
+    <xacro:property name="waterType" value="none" />
     <link name="base_link">
         <visual>

File: src/usv_sim/xacro/buoy.xacro (robot description, xacro)
@@ -25,4 +25,5 @@
           	<damping rpy="20 20 20" xyz="100 100 50"/>
 	  	  	<fluidVelocity>none</fluidVelocity>
+	  	  	<windVelocity>none</windVelocity>
         </buoyancy>
   </link>

Commit message: Updated flooding

File: src/usv_sim/xacro/boat_subdivided4.xacro (robot description, xacro)
@@ -15,5 +15,5 @@
     <xacro:property name="bl2" value=".1" />
     <xacro:property name="windType" value="none" />
-    <xacro:property name="waterType" value="none" />
+    <xacro:property name="waterType" value="local" />
     <link name="base_link">
         <visual>
