Commit message: Updated flooding scenario

File: src/usv_sim/xacro/boat_subdivided4.xacro (robot description, xacro)
@@ -14,5 +14,5 @@
     <xacro:property name="bl1" value=".1" />
     <xacro:property name="bl2" value=".1" />
-    <xacro:property name="windType" value="none" />
+    <xacro:property name="windType" value="local" />
     <xacro:property name="waterType" value="local" />
     <link name="base_link">

Commit message: Calibrated sailboat

File: src/usv_sim/xacro/boat_subdivided4.xacro (robot description, xacro)
@@ -14,5 +14,5 @@
     <xacro:property name="bl1" value=".1" />
     <xacro:property name="bl2" value=".1" />
-    <xacro:property name="windType" value="local" />
+    <xacro:property name="windType" value="global" />
     <xacro:property name="waterType" value="local" />
     <link name="base_link">
@@ -38,5 +38,5 @@
 			<origin xyz="${0.35*scale} ${0.44*scale} ${-0.15*scale}"/>
 			<limit radius="0.1"/>
-			<damping rpy="20 20 20" xyz="20 40 25"/>
+			<damping rpy="20 20 20" xyz="10 40 25"/>
          	<windVelocity>${windType}</windVelocity>
 			<frontal_area>0.0</frontal_area>
@@ -68,5 +68,5 @@
           <origin xyz="${0.35*scale} ${-0.44*scale} ${-0.15*scale}"/>
           <limit radius="0.1"/>
-          <damping rpy="20 20 20" xyz="20 40 25"/>
+          <damping rpy="20 20 20" xyz="10 40 25"/>
 			<windVelocity>${windType}</windVelocity>
 			<frontal_area>0.0</frontal_area>
@@ -106,5 +106,5 @@
 			<origin xyz="${-0.6*scale} 0 ${-0.15*scale}"/>
 			<limit radius="0.1"/>
-			<damping rpy="20 20 20" xyz="20 40 25"/>
+			<damping rpy="20 20 20" xyz="10 40 25"/>
 			<windVelocity>${windType}</windVelocity>
 			<frontal_area>0.04</frontal_area>
@@ -144,5 +144,5 @@
           	<origin xyz="${-0.6*scale} 0 ${-0.15*scale}"/>
           	<limit radius="0.1"/>
-          	<damping rpy="20 20 20" xyz="20 40 25"/>
+          	<damping rpy="20 20 20" xyz="10 40 25"/>
           	<windVelocity>${windType}</windVelocity>
 			<frontal_area>0.04</frontal_area>
@@ -182,5 +182,5 @@
           	<origin xyz="${0.4*scale} 0 ${-0.05*scale}"/>
           	<limit radius="0.1"/>
-          	<damping rpy="20 20 20" xyz="20 40 25"/>
+          	<damping rpy="20 20 20" xyz="10 40 25"/>
           	<windVelocity>${windType}</windVelocity>
 			<frontal_area>0.04</frontal_area>
@@ -220,5 +220,5 @@
           <origin xyz="${0.4*scale} 0 ${-0.05*scale}"/>
           <limit radius="0.1"/>
-          <damping rpy="20 20 20" xyz="20 40 25"/>
+          <damping rpy="20 20 20" xyz="10 40 25"/>
           <windVelocity>${windType}</windVelocity>
 	  <fluidVelocity>${waterType}</fluidVelocity>

File: src/usv_sim/xacro/sailboat.xacro (robot description, xacro)
@@ -40,5 +40,6 @@
     <link name="keel">
 	<inertial>
-		<mass value="5" />
+		<mass value="15" />
+		<origin rpy="0 0 0" xyz="0 0 -0.2"/>
 		<inertia
 		  ixx="0.4708"
@@ -84,5 +85,5 @@
 		<cp>0 0 0</cp>
 		<joint_name>sail_joint</joint_name>
-		<area>1.44</area>
+		<area>2</area>
 		<fluid_density>1.2041</fluid_density>
 		<forward>-1 0 0</forward>

Commit message: improved sailboat control and dynamics. changed secnario2 to add upwind points

File: src/usv_sim/xacro/boat_subdivided4.xacro (robot description, xacro)
@@ -369,5 +369,5 @@
             <dynamics damping="1.0"/>
             <axis xyz="0 0 1"/>
-            <limit effort="100" velocity="5" lower="-${PI/2}" upper="${PI/2}" />
+            <limit effort="100" velocity="5" lower="-${PI/3}" upper="${PI/3}" />
         </joint>
     </xacro:macro>

File: src/usv_sim/xacro/sailboat.xacro (robot description, xacro)
@@ -34,12 +34,12 @@
         <child link="sail"/>
         <origin rpy="0 0 0" xyz="0.2 0 0.1"/>
-        <dynamics damping="1.0"/>
+        <dynamics damping="7.0"/>
         <axis xyz="0 0 1"/>
-        <limit effort="500000" velocity="5" lower="-${PI}" upper="${PI}" />
+        <limit effort="5000999999900" velocity="7" lower="-${PI/2}" upper="${PI/2}" />
     </joint>
     <link name="keel">
 	<inertial>
-		<mass value="15" />
-		<origin rpy="0 0 0" xyz="0 0 -0.2"/>
+		<mass value="30" />
+		<origin rpy="0 0 0" xyz="0 0 -0.3"/>
 		<inertia
 		  ixx="0.4708"
@@ -111,6 +111,6 @@
 		<link_type>rudder</link_type>
 		<a0>0</a0>
-		<cla>0.8</cla>
-		<cda>0.3</cda>
+		<mult_lift>1.5</mult_lift>
+		<mult_drag>1.0</mult_drag>
 		<alpha_stall>0.785</alpha_stall>
 		<cla_stall>-0.85</cla_stall>
