Commit message: Added new buoy model

File: src/usv_sim/xacro/buoy.xacro (robot description, xacro)
@@ -5,21 +5,21 @@
       <origin rpy="0 0 0" xyz="0 0 0.25"/>
       <geometry>
-          <mesh filename="package://usv_sim/meshes/buoy.dae"/>
+          <mesh filename="package://usv_sim/meshes/buoy2.dae" scale="0.5 0.5 0.5"/>
       </geometry>
     </visual>
     <inertial>
-      <origin rpy="0 0 0" xyz="0 0 0.25"/>
-      <mass value="1.0"/>
+      <origin rpy="0 0 0" xyz="0 0 0"/>
+      <mass value="5.0"/>
       <inertia ixx="1" ixy="0.0" ixz="0.0" iyy="1" iyz="0" izz="1"/>
     </inertial>
     <collision>
-      <origin xyz="0 0 0" rpy="0 0 0.25"/>
+      <origin rpy="0 0 0" xyz="0 0 0.25"/>
      <geometry>
-          <mesh filename="package://usv_sim/meshes/buoy.dae"/>
+          <mesh filename="package://usv_sim/meshes/buoy2.dae" scale="0.5 0.5 0.5"/>
       </geometry>
     </collision>
 		<buoyancy>
         	<compensation>10</compensation>
-          	<origin xyz="0 0 0.3"/>
+          	<origin xyz="0 0 0.05"/>
           	<limit radius="0.25"/>
           	<damping rpy="20 20 20" xyz="100 100 50"/>

Commit message: Added hardcoded ground truth generation

File: src/usv_sim/xacro/buoy.xacro (robot description, xacro)
@@ -5,5 +5,5 @@
       <origin rpy="0 0 0" xyz="0 0 0.25"/>
       <geometry>
-          <mesh filename="package://usv_sim/meshes/buoy2.dae" scale="0.5 0.5 0.5"/>
+          <mesh filename="package://usv_sim/meshes/buoy2highPoly.dae" scale="0.5 0.5 0.5"/>
       </geometry>
     </visual>
@@ -16,5 +16,5 @@
       <origin rpy="0 0 0" xyz="0 0 0.25"/>
      <geometry>
-          <mesh filename="package://usv_sim/meshes/buoy2.dae" scale="0.5 0.5 0.5"/>
+          <mesh filename="package://usv_sim/meshes/buoy2highPoly.dae" scale="0.5 0.5 0.5"/>
       </geometry>
     </collision>
