Commit message: Added ground truth generation for ocean segmentation

File: usv_sim/xacro/boat_subdivided4.xacro (robot description, xacro)
@@ -15,5 +15,5 @@
     <xacro:property name="bl2" value=".1" />
     <xacro:property name="windType" value="global" />
-    <xacro:property name="waterType" value="global" />
+    <xacro:property name="waterType" value="local" />
     <link name="base_link">
         <visual>

Commit message: Reconfiguring wind and water current to global

File: usv_sim/xacro/boat_subdivided4.xacro (robot description, xacro)
@@ -15,5 +15,5 @@
     <xacro:property name="bl2" value=".1" />
     <xacro:property name="windType" value="global" />
-    <xacro:property name="waterType" value="local" />
+    <xacro:property name="waterType" value="global" />
     <link name="base_link">
         <visual>

Commit message: Updated submodules

File: usv_sim/xacro/boat_subdivided4.xacro (robot description, xacro)
@@ -14,6 +14,8 @@
     <xacro:property name="bl1" value=".1" />
     <xacro:property name="bl2" value=".1" />
-    <xacro:property name="windType" value="global" />
-    <xacro:property name="waterType" value="global" />
+    <xacro:arg name="windType" default="global" />
+    <xacro:arg name="waterType" default="global" />
+    <xacro:property name="windType" value="$(arg windType)" />
+    <xacro:property name="waterType" value="$(arg waterType)" />
     <link name="base_link">
         <visual>

File: usv_sim/xacro/buoy.xacro (robot description, xacro)
@@ -23,4 +23,5 @@
           	<origin xyz="0 0 0.05"/>
           	<limit radius="0.25"/>
+          	<windVelocity>none</windVelocity>
           	<damping rpy="20 20 20" xyz="100 100 50"/>
 	  	  	<fluidVelocity>none</fluidVelocity>
