Commit message: Updated scenarios

File: usv_sim/xacro/airboat_validation.xacro (robot description, xacro)
@@ -5,7 +5,8 @@
     <xacro:property name="windType" value="$(arg windType)" />
     <xacro:property name="waterType" value="$(arg waterType)" />
-    <xacro:property name="dampingXYZ" value="1.16 10 10" />
-    <xacro:property name="angularDampingXYZ" value="0.5 15 2" />
-    <xacro:include filename="$(find usv_sim)/xacro/boat_subdivided_validation.xacro" />
+    <xacro:property name="dampingXYZ" value="1.16 10 6.66" />
+    <xacro:property name="angularDampingXYZ" value="2 15 2" />
+    <xacro:property name="extraPayload" value="3" />
+    <xacro:include filename="$(find usv_sim)/xacro/boat_subdivided_validation2.xacro" />
     <!-- Plugin list -->
     <gazebo>
@@ -22,4 +23,4 @@
     </gazebo>
     <!-- Define one steering thruster, with assumed force control in Z-direction -->
-    <xacro:airthruster_link name="fwd" xyz="-0.3 0.12 0.2" rpy="0 ${-PI/2} 0" effort="100" velocity="20" rotationAxis="1 0 0" lowerLimit="${-PI/2}" upperLimit="0.5"/>
+    <xacro:airthruster_link name="fwd" xyz="-0.3 0 0.13" rpy="0 ${-PI/2} 0" effort="100" velocity="2" rotationAxis="1 0 0" lowerLimit="${-PI/2}" upperLimit="0.5" parentLink="base_link"/>
 </robot>

File: usv_sim/xacro/boat_subdivided_validation.xacro (robot description, xacro)
@@ -28,5 +28,5 @@
             <origin rpy="0 0 0" xyz="${0.35*scale} ${0.44*scale} ${-0.2*scale}"/>
           <mass value="${middle_body_mass}"/>
-          <inertia ixx="0.1" ixy="0.0" ixz="0.0" iyy="1.4" iyz="0.0" izz="1.4"/>
+          <inertia ixx="0.012" ixy="0.0" ixz="0.0" iyy="0.014" iyz="0.0" izz="0.018"/>
         </inertial>
         <buoyancy>
@@ -58,5 +58,5 @@
             <origin rpy="0 0 0" xyz="${0.35*scale} ${-0.44*scale} ${-0.2*scale}"/>
           <mass value="${middle_body_mass}"/>
-          <inertia ixx="0.1" ixy="0.0" ixz="0.0" iyy="1.4" iyz="0.0" izz="1.4"/>
+          <inertia ixx="0.012" ixy="0.0" ixz="0.0" iyy="0.014" iyz="0.0" izz="0.018"/>
         </inertial>
         <buoyancy>
@@ -94,11 +94,11 @@
         </collision>
         <inertial>
-            <origin rpy="0 0 0" xyz="${-0.6*scale} 0 ${-0.2*scale}"/>
+            <origin rpy="0 0 0" xyz="${-0.5*scale} 0 ${-0.2*scale}"/>
           <mass value="${back_body_mass}"/>
-          <inertia ixx="0.1" ixy="0.0" ixz="0.0" iyy="1.4" iyz="0.0" izz="1.4"/>
+          <inertia ixx="0.012" ixy="0.0" ixz="0.0" iyy="0.014" iyz="0.0" izz="0.018"/>
         </inertial>
         <buoyancy>
 			<compensation>${back_water_displaced_mass/back_body_mass}</compensation>
-			<origin xyz="${-0.6*scale} 0 ${-0.15*scale}"/>
+			<origin xyz="${-0.5*scale} 0 ${-0.15*scale}"/>
 			<limit radius="0.1"/>
 			<damping rpy="${angularDampingXYZ}" xyz="${dampingXYZ}"/>
@@ -132,11 +132,11 @@
         </collision>
         <inertial>
-            <origin rpy="0 0 0" xyz="${-0.6*scale} 0 ${-0.2*scale}"/>
+            <origin rpy="0 0 0" xyz="${-0.5*scale} 0 ${-0.2*scale}"/>
           <mass value="${back_body_mass}"/>
-          <inertia ixx="0.1" ixy="0.0" ixz="0.0" iyy="1.4" iyz="0.0" izz="1.4"/>
+          <inertia ixx="0.012" ixy="0.0" ixz="0.0" iyy="0.014" iyz="0.0" izz="0.018"/>
         </inertial>
         <buoyancy>
           	<compensation>${back_water_displaced_mass/back_body_mass}</compensation>
-          	<origin xyz="${-0.6*scale} 0 ${-0.15*scale}"/>
+          	<origin xyz="${-0.5*scale} 0 ${-0.15*scale}"/>
           	<limit radius="0.1"/>
           	<damping rpy="${angularDampingXYZ}" xyz="${dampingXYZ}"/>
@@ -172,5 +172,5 @@
             <origin rpy="0 0 0" xyz="${0.4*scale} 0 ${-0.1*scale}"/>
           <mass value="${front_body_mass}"/>
-          <inertia ixx="0.1" ixy="0.0" ixz="0.0" iyy="1.4" iyz="0.0" izz="1.4"/>
+          <inertia ixx="0.01" ixy="0.0" ixz="0.0" iyy="0.01" iyz="0.0" izz="0.014"/>
         </inertial>
         <buoyancy>
@@ -210,5 +210,5 @@
             <origin rpy="0 0 0" xyz="${0.4*scale} 0 ${-0.1*scale}"/>
           <mass value="${front_body_mass}"/>
-          <inertia ixx="0.1" ixy="0.0" ixz="0.0" iyy="1.4" iyz="0.0" izz="1.4"/>
+          <inertia ixx="0.01" ixy="0.0" ixz="0.0" iyy="0.01" iyz="0.0" izz="0.014"/>
         </inertial>
         <buoyancy>
@@ -299,16 +299,16 @@
                 <origin xyz="0 0 0" rpy="0 0 0" />
                 <geometry>
-                    	<mesh filename="package://usv_sim/meshes/simpleHull3/airPropeller.dae" scale="${scale} ${scale} ${scale}"/>
+                    	<mesh filename="package://usv_sim/meshes/simpleHull3/airPropeller.dae" scale="${0.5*scale} ${0.5*scale} ${0.5*scale}"/>
                 </geometry>
             </visual>
             <inertial>
-                <mass value=".1"/>
+                <mass value="0.01"/>
                 <inertia
-                    ixx=".1"
+                    ixx="0.1"
                     ixy="0.0"
                     ixz="0.0"
-                    iyy=".1"
+                    iyy="0.1"
                     iyz="0.0"
-                    izz=".1"/>
+                    izz="0.1"/>
             </inertial>
         </link>
@@ -362,4 +362,5 @@
     <!-- Sensors -->
     <!-- Hokuyo Laser -->
+    <!--
     <joint name="hokuyo_joint" type="revolute">
         <axis xyz="0 1 0" />
@@ -388,4 +389,5 @@
         </inertial>
     </link>
+    -->
     <gazebo reference="hokuyo_link">
         <sensor type="gpu_ray" name="head_hokuyo_sensor">

File: usv_sim/xacro/diffboat_validation.xacro (robot description, xacro)
@@ -5,7 +5,8 @@
     <xacro:property name="windType" value="$(arg windType)" />
     <xacro:property name="waterType" value="$(arg waterType)" />
-    <xacro:property name="dampingXYZ" value="1.88 10 10" />
-    <xacro:property name="angularDampingXYZ" value="0.5 15 2" />
-    <xacro:include filename="$(find usv_sim)/xacro/boat_subdivided_validation.xacro" />
+    <xacro:property name="dampingXYZ" value="1.88 10 6.66" />
+    <xacro:property name="angularDampingXYZ" value="2 15 2" />
+    <xacro:property name="extraPayload" value="3" />
+    <xacro:include filename="$(find usv_sim)/xacro/boat_subdivided_validation2.xacro" />
     <!-- Plugin list -->
     <gazebo>
@@ -20,5 +21,5 @@
             </thruster>
    	    <thruster>
-	        <effortUnderWater>12</effortUnderWater>
+	        <effortUnderWater>11.5</effortUnderWater>
 				<effortOverWater>0</effortOverWater>
 	        <name>fwd_right</name>
@@ -27,5 +28,5 @@
     </gazebo>
     <!-- Define two steering thrusters, with assumed force control in Z-direction -->
-    <xacro:thruster_link name="fwd_left"  xyz="-0.4 0 -0.1" rpy="0 ${-PI/2-0.26} 0" rotationAxis="1 0 0" lowerLimit="0" upperLimit="0" parentLink="back_l_link"/>
-    <xacro:thruster_link name="fwd_right" xyz="-0.4 0 -0.1" rpy="0 ${-PI/2-0.26} 0" rotationAxis="1 0 0" lowerLimit="0" upperLimit="0" parentLink="back_r_link"/>
+    <xacro:thruster_link name="fwd_left"  xyz="-0.3 0 -0.1" rpy="0 ${-PI/2-0.26} 0" rotationAxis="1 0 0" lowerLimit="0" upperLimit="0" parentLink="back_l_link"/>
+    <xacro:thruster_link name="fwd_right" xyz="-0.3 0 -0.1" rpy="0 ${-PI/2-0.26} 0" rotationAxis="1 0 0" lowerLimit="0" upperLimit="0" parentLink="back_r_link"/>
 </robot>

File: usv_sim/xacro/rudderboat.xacro (robot description, xacro)
@@ -5,5 +5,8 @@
     <xacro:property name="windType" value="$(arg windType)" />
     <xacro:property name="waterType" value="$(arg waterType)" />
-    <xacro:include filename="$(find usv_sim)/xacro/boat_subdivided4.xacro" />
+    <xacro:property name="dampingXYZ" value="1.88 10 6.66" />
+    <xacro:property name="angularDampingXYZ" value="2 15 2" />
+    <xacro:property name="extraPayload" value="3" />
+    <xacro:include filename="$(find usv_sim)/xacro/boat_subdivided_validation2.xacro" />
     <xacro:rudder_xacro/>
     <!-- Plugin list -->
@@ -27,5 +30,5 @@
             <link>fwd</link>
             <thruster>
-                <effort>300</effort>
+                <effort>11.5</effort>
                 <name>fwd</name>
             </thruster>
@@ -33,4 +36,4 @@
     </gazebo>
     <!-- Define two steering thrusters, with assumed force control in Z-direction -->
-    <xacro:thruster_link name="fwd" xyz="-0.45 0.117 -0.15" rpy="0 ${-PI/2} 0" rotationAxis="1 0 0" lowerLimit="0" upperLimit="0" />
+    <xacro:thruster_link name="fwd" xyz="-0.3 0.08 -0.15" rpy="0 ${-PI/2-0.26} 0" rotationAxis="1 0 0" lowerLimit="0" upperLimit="0" />
 </robot>

File: usv_sim/xacro/sailboat.xacro (robot description, xacro)
@@ -44,5 +44,5 @@
     <link name="keel">
 	<inertial>
-		<mass value="5" />
+		<mass value="30" />
 		<inertia
 		  ixx="0.4708"
