Commit message: error when launching gazebo

File: usv_sim/xacro/airboat.xacro (robot description, xacro)
@@ -1,5 +1,5 @@
 <?xml version="1.0"?>
 <robot name="airboat" xmlns:xacro="http://www.ros.org/wiki/xacro">
-    <xacro:include filename="$(find usv_sim)/xacro/boat_subdivided4.xacro" />
+    <xacro:include filename="$(find usv_sim)/xacro/boat_subdivided.xacro" />
     <!-- Plugin list -->
     <gazebo>

File: usv_sim/xacro/boat_subdivided.xacro (robot description, xacro)
@@ -11,4 +11,9 @@
     <xacro:property name="middle_water_displaced_mass" value="60"/>
     <xacro:property name="front_water_displaced_mass" value="25"/>
+    <xacro:property name="scale" value="0.3"/>
+    <xacro:property name="bl1" value=".1" />
+    <xacro:property name="bl2" value=".1" />
+    <xacro:property name="windType" value="global" />
+    <xacro:property name="waterType" value="global" />
     <!-- Thruster constants -->
     <xacro:property name="tr1" value=".02" />
@@ -44,6 +49,6 @@
         </buoyancy>
     </link>
-    <!-- Thruster link -->
-    <xacro:macro name="thruster_link" params="name xyz rpy rotationAxis effort:=50 velocity:=5 lowerLimit upperLimit parentLink:=back_r_link">
+<!-- Thruster link -->
+    <xacro:macro name="thruster_link" params="name xyz rpy rotationAxis effort:=50 velocity:=5 lowerLimit upperLimit parentLink:=base_link">
         <joint name="${name}_joint" type="revolute">
             <parent link="${parentLink}"/>
@@ -56,11 +61,65 @@
         <link name="${name}">
             <buoyancy>
+				<compensation>0.8</compensation>
+	        	<fluidVelocity>${windType}</fluidVelocity>
+	    	</buoyancy>
+	    	<collision>
+          		<origin xyz="${-0.15*scale} 0 ${0*scale}" rpy="0 0 0"/>
+          		<geometry>
+          		    <mesh filename="package://usv_sim/meshes/simpleHull3/thruster.dae" scale="${scale} ${scale} ${scale}"/>
+          		</geometry>
+        	</collision>
+            <visual name="${name}">
+                <origin xyz="${-0.15*scale} 0 ${0*scale}" rpy="0 0 0" />
+                <geometry>
+                    <mesh filename="package://usv_sim/meshes/simpleHull3/thruster.dae" scale="${scale} ${scale} ${scale}"/>
+                </geometry>
+                <material name="black">
+                    <color rgba="255 255 255 1"/>
+                </material>
+            </visual>
+            <inertial>
+                <mass value="5"/>
+                <origin xyz="${-0.2*scale} 0 ${0.3*scale}" rpy="0 0 0" />
+                <inertia
+                    ixx=".1"
+                    ixy="0.0"
+                    ixz="0.0"
+                    iyy=".1"
+                    iyz="0.0"
+                    izz=".1"/>
+            </inertial>
+        </link>
+        <gazebo reference="${name}">
+            <material>Gazebo/Black</material>
+        </gazebo>
+    </xacro:macro>
+    <xacro:macro name="thruster_dummy_link" params="name xyz rpy">
+        <joint name="${name}" type="fixed">
+            <parent link="base_link"/>
+            <child link="${name}"/>
+            <origin rpy="${rpy}" xyz="${xyz}"/>
+        </joint>
+        <link name="${name}"/>
+    </xacro:macro>
+    <!-- Thruster link -->
+    <xacro:macro name="airthruster_link" params="name xyz rpy rotationAxis effort:=100 velocity:=20 lowerLimit upperLimit parentLink:=base_link">
+        <joint name="${name}_joint" type="revolute">
+            <parent link="${parentLink}"/>
+            <child link="${name}"/>
+            <origin rpy="${rpy}" xyz="${xyz}"/>
+            <dynamics damping="10.0"/>
+            <axis xyz="${rotationAxis}"/>
+            <limit effort="${effort}" velocity="${velocity}" lower="${lowerLimit}" upper="${upperLimit}" />
+        </joint>
+        <link name="${name}">
+            <buoyancy>
 				<compensation>1.0</compensation>
-	        	<fluidVelocity>local</fluidVelocity>
+	        	<fluidVelocity>${waterType}</fluidVelocity>
 	    	</buoyancy>
 	    	<collision>
           		<origin xyz="0 0 0" rpy="0 0 0"/>
           		<geometry>
-          			<box size="tl1 tl1 tl2" />
+          			<box size="${bl1} ${bl1} ${bl2}" />
           		</geometry>
         	</collision>
@@ -68,9 +127,6 @@
                 <origin xyz="0 0 0" rpy="0 0 0" />
                 <geometry>
-                    <mesh filename="package://usv_sim/meshes/simpleHull/thruster.obj"/>
-                </geometry>
-                <material name="black">
-                    <color rgba="255 255 255 1"/>
-                </material>
+                    	<mesh filename="package://usv_sim/meshes/simpleHull3/airPropeller.dae" scale="${scale} ${scale} ${scale}"/>
+                </geometry>
             </visual>
             <inertial>
@@ -101,5 +157,5 @@
         <link name="rudder">
             <inertial>
-                <mass value="0.05" />
+                <mass value="1" />
                 <inertia
                   ixx="0.05"
@@ -112,22 +168,22 @@
             <collision name="collision">
                 <geometry>
-                  <box size="0.2 0.02 0.3" />
-                </geometry>
-                <origin rpy="0 0 0" xyz="-0.1 0 0"/>
+                  <box size="${0.2*scale} ${0.02*scale} ${0.3*scale}" />
+                </geometry>
+                <origin rpy="0 0 0" xyz="${-0.1*scale} 0 0"/>
             </collision>
             <visual name="visual">
                 <geometry>
-                  <box size="0.1 0.02 0.3" />
-                </geometry>
-                <origin rpy="0 0 0" xyz="-0.1 0 0"/>
+                  <mesh filename="package://usv_sim/meshes/simpleHull3/box.dae" scale="${0.2*scale} ${0.02*scale} ${0.3*scale}"/>
+                </geometry>
+                <origin rpy="0 0 0" xyz="${-0.1*scale} 0 0"/>
             </visual>
         </link>
         <joint name="rudder_joint" type="revolute">
-            <parent link="back_r_link"/>
+            <parent link="base_link"/>
             <child link="rudder"/>
-            <origin rpy="0 0 0" xyz="-1.2 0.22 -0.5"/>
+            <origin rpy="0 0 0" xyz="${-1.4*scale} ${0.39*scale} ${-0.5*scale}"/>
             <dynamics damping="1.0"/>
             <axis xyz="0 0 1"/>
-            <limit effort="50" velocity="5" lower="-${PI/3}" upper="${PI/3}" />
+            <limit effort="100" velocity="5" lower="-${PI/2}" upper="${PI/2}" />
         </joint>
     </xacro:macro>

Commit message: Updated package names, testes all usv_sim launchs

File: usv_sim/xacro/airboat.xacro (robot description, xacro)
@@ -1,8 +1,14 @@
 <?xml version="1.0"?>
 <robot name="airboat" xmlns:xacro="http://www.ros.org/wiki/xacro">
-    <xacro:include filename="$(find usv_sim)/xacro/boat_subdivided4.xacro" />
+    <xacro:arg name="windType" default="global" />
+    <xacro:arg name="waterType" default="global" />
+    <xacro:property name="windType" value="$(arg windType)" />
+    <xacro:property name="waterType" value="$(arg waterType)" />
+    <xacro:property name="dampingXYZ" value="1.16 10 6.66" />
+    <xacro:property name="angularDampingXYZ" value="2 15 2" />
+    <xacro:property name="extraPayload" value="3" />
+    <xacro:include filename="$(find usv_sim)/xacro/boat_subdivided_validated.xacro" />
     <!-- Plugin list -->
     <gazebo>
-    <!-- Gazebo plugin listens to the body-->
         <plugin name="freefloating_gazebo_control" filename="libfreefloating_gazebo_control.so">
             <switchService>switch</switchService>
@@ -10,6 +16,6 @@
             <link>fwd</link>
             <thruster>
-                <effortUnderWater>100</effortUnderWater>
-				<effortOverWater>100</effortOverWater>
+                <effortUnderWater>0</effortUnderWater>
+				<effortOverWater>4.12</effortOverWater>
                 <name>fwd</name>
             </thruster>
@@ -17,4 +23,4 @@
     </gazebo>
     <!-- Define one steering thruster, with assumed force control in Z-direction -->
-    <xacro:airthruster_link name="fwd" xyz="0 0.12 0.3" rpy="0 ${-PI/2} 0" effort="100" velocity="20" rotationAxis="1 0 0" lowerLimit="-${PI/4}" upperLimit="${PI/4}"/>
+    <xacro:airthruster_link name="fwd" xyz="-0.3 0 0.13" rpy="0 ${-PI/2} 0" effort="100" velocity="2" rotationAxis="1 0 0" lowerLimit="${-PI/2}" upperLimit="0.5" parentLink="base_link"/>
 </robot>

File: usv_sim/xacro/diffboat.xacro (robot description, xacro)
@@ -1,5 +1,12 @@
 <?xml version="1.0"?>
 <robot name="diffboat" xmlns:xacro="http://www.ros.org/wiki/xacro">
-    <xacro:include filename="$(find usv_sim)/xacro/boat_subdivided4.xacro" />
+    <xacro:arg name="windType" default="global" />
+    <xacro:arg name="waterType" default="global" />
+    <xacro:property name="windType" value="$(arg windType)" />
+    <xacro:property name="waterType" value="$(arg waterType)" />
+    <xacro:property name="dampingXYZ" value="1.88 10 6.66" />
+    <xacro:property name="angularDampingXYZ" value="2 15 2" />
+    <xacro:property name="extraPayload" value="3" />
+    <xacro:include filename="$(find usv_sim)/xacro/boat_subdivided_validated.xacro" />
     <!-- Plugin list -->
     <gazebo>
@@ -9,9 +16,11 @@
             <link>fwd_left</link>
             <thruster>
-                <effort>100</effort>
+				<effortUnderWater>11.5</effortUnderWater>
+				<effortOverWater>0</effortOverWater>
                 <name>fwd_left</name>
             </thruster>
    	    <thruster>
-	        <effort>100</effort>
+	        <effortUnderWater>11.5</effortUnderWater>
+				<effortOverWater>0</effortOverWater>
 	        <name>fwd_right</name>
 	    </thruster>
@@ -19,5 +28,5 @@
     </gazebo>
     <!-- Define two steering thrusters, with assumed force control in Z-direction -->
-    <xacro:thruster_link name="fwd_left"  xyz="-0.4 0 -0.15" rpy="0 ${-PI/2} 0" rotationAxis="1 0 0" lowerLimit="0" upperLimit="0" parentLink="back_l_link"/>
-    <xacro:thruster_link name="fwd_right" xyz="-0.4 0 -0.15" rpy="0 ${-PI/2} 0" rotationAxis="1 0 0" lowerLimit="0" upperLimit="0" parentLink="back_r_link"/>
+    <xacro:thruster_link name="fwd_left"  xyz="-0.3 0 -0.1" rpy="0 ${-PI/2-0.26} 0" rotationAxis="1 0 0" lowerLimit="0" upperLimit="0" parentLink="back_l_link"/>
+    <xacro:thruster_link name="fwd_right" xyz="-0.3 0 -0.1" rpy="0 ${-PI/2-0.26} 0" rotationAxis="1 0 0" lowerLimit="0" upperLimit="0" parentLink="back_r_link"/>
 </robot>

File: usv_sim/xacro/rudderboat.xacro (robot description, xacro)
@@ -8,5 +8,5 @@
     <xacro:property name="angularDampingXYZ" value="2 15 2" />
     <xacro:property name="extraPayload" value="3" />
-    <xacro:include filename="$(find usv_sim)/xacro/boat_subdivided_validation2.xacro" />
+    <xacro:include filename="$(find usv_sim)/xacro/boat_subdivided_validated.xacro" />
     <xacro:rudder_xacro/>
     <!-- Plugin list -->

Commit message: Added new scenario 3gt

File: usv_sim/xacro/airboat.xacro (robot description, xacro)
@@ -23,4 +23,4 @@
     </gazebo>
     <!-- Define one steering thruster, with assumed force control in Z-direction -->
-    <xacro:airthruster_link name="fwd" xyz="-0.3 0 0.13" rpy="0 ${-PI/2} 0" effort="100" velocity="2" rotationAxis="1 0 0" lowerLimit="${-PI/2}" upperLimit="0.5" parentLink="base_link"/>
+    <xacro:airthruster_link name="fwd" xyz="-0.3 0 0.18" rpy="0 ${-PI/2} 0" effort="100" velocity="2" rotationAxis="1 0 0" lowerLimit="-0.5" upperLimit="0.5" parentLink="base_link"/>
 </robot>

File: usv_sim/xacro/boat_subdivided_validated.xacro (robot description, xacro)
@@ -307,5 +307,5 @@
                 <origin xyz="0 0 0" rpy="0 0 0" />
                 <geometry>
-                    	<mesh filename="package://usv_sim/meshes/simpleHull3/airPropeller.dae" scale="${scale} ${scale} ${scale}"/>
+                    	<mesh filename="package://usv_sim/meshes/simpleHull3/airPropeller.dae" scale="${0.9*scale} ${0.9*scale} ${0.9*scale}"/>
                 </geometry>
             </visual>
