Commit message: Adding launch example of move_base

File: usv_sim/xacro/boat_subdivided_validated.xacro (robot description, xacro)
@@ -397,7 +397,8 @@
     </link>
     <gazebo reference="hokuyo_link">
-        <sensor type="gpu_ray" name="head_hokuyo_sensor">
+        <!--<sensor type="gpu_ray" name="head_hokuyo_sensor">-->
+        <sensor type="ray" name="head_hokuyo_sensor">
         <pose>0 0 0 0 0 0</pose>
-        <visualize>false</visualize>
+        <visualize>true</visualize>
         <update_rate>40</update_rate>
         <ray>
@@ -425,7 +426,8 @@
         </noise>
         </ray>
-        <plugin name="gazebo_ros_head_hokuyo_controller" filename="libgazebo_ros_gpu_laser.so">
-        <topicName>scan</topicName>
-        <frameName>base_laser</frameName>
+       <!-- <plugin name="gazebo_ros_head_hokuyo_controller" filename="libgazebo_ros_gpu_laser.so">-->
+        <plugin name="gazebo_ros_head_hokuyo_controller" filename="libgazebo_ros_laser.so">
+        <topicName>${namespace}/scan</topicName>
+        <frameName>${namespace}/base_laser</frameName>
         </plugin>
         </sensor>

File: usv_sim/xacro/diffboat.xacro (robot description, xacro)
@@ -3,6 +3,8 @@
     <xacro:arg name="windType" default="global" />
     <xacro:arg name="waterType" default="global" />
+    <xacro:arg name="namespace" default="diffboat" />
     <xacro:property name="windType" value="$(arg windType)" />
     <xacro:property name="waterType" value="$(arg waterType)" />
+    <xacro:property name="namespace" value="$(arg namespace)" />
     <xacro:property name="dampingXYZ" value="1.88 10 6.66" />
     <xacro:property name="angularDampingXYZ" value="2 15 2" />
