Commit message: Started to validate airboat and diffboat

File: usv_sim/urdf/airboat_dummy.urdf (robot description, URDF)
Before this commit: robot thrusters, 0 links, 1 joints
Joints:
- joint fwd: limit lower=-180 upper=180 -> lower=-4.12 upper=4.12

File: usv_sim/urdf/diffboat_dummy.urdf (robot description, URDF)
Before this commit: robot thrusters, 0 links, 2 joints
Joints:
- joint fwd_left: limit lower=-300 upper=300 -> lower=-11.5 upper=11.5
- joint fwd_right: limit lower=-300.0 upper=300.0 -> lower=-11.5 upper=11.5

File: usv_sim/xacro/boat_subdivided4.xacro (robot description, xacro)
@@ -45,5 +45,5 @@
 			<lateral_area>0.06</lateral_area>
 			<lateral_length>1.2</lateral_length>
-	  		<fluidVelocity>${waterType}</fluidVelocity>
+	  		<waterVelocity>${waterType}</waterVelocity>
         </buoyancy>
     </link>
@@ -75,5 +75,5 @@
 			<lateral_area>0.06</lateral_area>
 			<lateral_length>1.2</lateral_length>
-	  <fluidVelocity>${waterType}</fluidVelocity>
+	  <waterVelocity>${waterType}</waterVelocity>
         </buoyancy>
     </link>
@@ -113,5 +113,5 @@
 			<lateral_area>0.06</lateral_area>
 			<lateral_length>1.2</lateral_length>
-	  		<fluidVelocity>${waterType}</fluidVelocity>
+	  		<waterVelocity>${waterType}</waterVelocity>
         </buoyancy>
     </link>
@@ -151,5 +151,5 @@
 			<lateral_area>0.06</lateral_area>
 			<lateral_length>1.2</lateral_length>
-	  		<fluidVelocity>${waterType}</fluidVelocity>
+	  		<waterVelocity>${waterType}</waterVelocity>
         </buoyancy>
     </link>
@@ -189,5 +189,5 @@
 			<lateral_area>0.06</lateral_area>
 			<lateral_length>1.2</lateral_length>
-	  		<fluidVelocity>${waterType}</fluidVelocity>
+	  		<waterVelocity>${waterType}</waterVelocity>
         </buoyancy>
     </link>
@@ -224,5 +224,5 @@
           <damping rpy="20 20 20" xyz="20 40 50"/>
           <windVelocity>${windType}</windVelocity>
-	  <fluidVelocity>${waterType}</fluidVelocity>
+	  <waterVelocity>${waterType}</waterVelocity>
         </buoyancy>
     </link>
@@ -248,5 +248,5 @@
             <buoyancy>
 				<compensation>0.8</compensation>
-	        	<fluidVelocity>${windType}</fluidVelocity>
+	        	<waterVelocity>${waterType}</waterVelocity>
 	    	</buoyancy>
 	    	<collision>
@@ -302,5 +302,5 @@
             <buoyancy>
 				<compensation>1.0</compensation>
-	        	<fluidVelocity>${waterType}</fluidVelocity>
+	        	<waterVelocity>${waterType}</waterVelocity>
 	    	</buoyancy>
 	    	<collision>

File: usv_sim/xacro/buoy.xacro (robot description, xacro)
@@ -25,5 +25,5 @@
           	<windVelocity>none</windVelocity>
           	<damping rpy="20 20 20" xyz="100 100 50"/>
-	  	  	<fluidVelocity>none</fluidVelocity>
+	  	  	<waterVelocity>none</waterVelocity>
         </buoyancy>
   </link>

File: usv_sim/xacro/rudderboat.xacro (robot description, xacro)
@@ -1,4 +1,8 @@
 <?xml version="1.0"?>
 <robot name="rudderboat" xmlns:xacro="http://www.ros.org/wiki/xacro">
+    <xacro:arg name="windType" default="global" />
+    <xacro:arg name="waterType" default="global" />
+    <xacro:property name="windType" value="$(arg windType)" />
+    <xacro:property name="waterType" value="$(arg waterType)" />
     <xacro:include filename="$(find usv_sim)/xacro/boat_subdivided4.xacro" />
     <xacro:rudder_xacro/>
@@ -16,4 +20,5 @@
 		<upward>0 1 0</upward>
 		<link_name>rudder</link_name>
+		<fluidVelocity>${waterType}</fluidVelocity>
 	</plugin>
         <plugin name="freefloating_gazebo_control" filename="libfreefloating_gazebo_control.so">

File: usv_sim/xacro/sailboat.xacro (robot description, xacro)
@@ -1,4 +1,8 @@
 <?xml version="1.0"?>
 <robot name="sailboat" xmlns:xacro="http://www.ros.org/wiki/xacro">
+    <xacro:arg name="windType" default="global" />
+    <xacro:arg name="waterType" default="global" />
+    <xacro:property name="windType" value="$(arg windType)" />
+    <xacro:property name="waterType" value="$(arg waterType)" />
     <xacro:property name="windType" value="global"/>
     <xacro:include filename="$(find usv_sim)/xacro/boat_subdivided4.xacro" />
@@ -36,5 +40,5 @@
         <dynamics damping="1.0"/>
         <axis xyz="0 0 1"/>
-        <limit effort="50" velocity="5" lower="-1.5" upper="1.5" />
+        <limit effort="100" velocity="70" lower="-${PI}" upper="${PI}" />
     </joint>
     <link name="keel">
@@ -85,5 +89,5 @@
 		<joint_name>sail_joint</joint_name>
 		<area>1.44</area>
-		<air_density>1.2041</air_density>
+		<fluid_density>1.2041</fluid_density>
 		<forward>-1 0 0</forward>
 		<upward>0 1 0</upward>
@@ -101,9 +105,9 @@
 		  <cp>0 0 0</cp>
 		  <area>1.0</area>
-		  <air_density>1000</air_density>
+		  <fluid_density>1000</fluid_density>
 		  <forward>1 0 0</forward>
 		  <upward>0 1 0</upward>
 		  <link_name>keel</link_name>
-		  <fluidVelocity>local</fluidVelocity>
+		  <fluidVelocity>${waterType}</fluidVelocity>
     </plugin>
     <plugin name="usv_sail_plugin" filename="libusv_sailing_plugin.so">
@@ -117,9 +121,9 @@
 		<cp>0 0 0</cp>
 		<area>1</area>
-		<air_density>1000</air_density>
+		<fluid_density>1000</fluid_density>
 		<forward>1 0 0</forward>
 		<upward>0 1 0</upward>
 		<link_name>rudder</link_name>
-		<fluidVelocity>local</fluidVelocity>
+		<fluidVelocity>${waterType}</fluidVelocity>
       </plugin>
       <plugin name="freefloating_gazebo_control" filename="libfreefloating_gazebo_control.so">

Commit message: Changed validation values of airboat and diffboat

File: usv_sim/urdf/airboat_dummy.urdf (robot description, URDF)
Before this commit: robot thrusters, 0 links, 1 joints
Joints:
- joint fwd: limit lower=-4.12 upper=4.12 -> lower=-3.13 upper=3.13

File: usv_sim/xacro/airboat_validation.xacro (robot description, xacro)
@@ -5,5 +5,6 @@
     <xacro:property name="windType" value="$(arg windType)" />
     <xacro:property name="waterType" value="$(arg waterType)" />
-    <xacro:property name="dampingXYZ" value="2.7 18 60" />
+    <xacro:property name="dampingXYZ" value="1.16 10 10" />
+    <xacro:property name="angularDampingXYZ" value="0.5 15 2" />
     <xacro:include filename="$(find usv_sim)/xacro/boat_subdivided_validation.xacro" />
     <!-- Plugin list -->
@@ -21,4 +22,4 @@
     </gazebo>
     <!-- Define one steering thruster, with assumed force control in Z-direction -->
-    <xacro:airthruster_link name="fwd" xyz="0 0.12 0.3" rpy="0 ${-PI/2} 0" effort="100" velocity="20" rotationAxis="1 0 0" lowerLimit="-${PI/4}" upperLimit="${PI/4}"/>
+    <xacro:airthruster_link name="fwd" xyz="-0.3 0.12 0.2" rpy="0 ${-PI/2} 0" effort="100" velocity="20" rotationAxis="1 0 0" lowerLimit="${-PI/2}" upperLimit="0.5"/>
 </robot>

File: usv_sim/xacro/boat_subdivided_validation.xacro (robot description, xacro)
@@ -3,11 +3,11 @@
     <xacro:property name="PI" value="3.1415926535897931"/>
     <!-- Body properties -->
-    <xacro:property name="front_body_mass" value="1.5"/>
-    <xacro:property name="back_body_mass" value="1.5"/>
-    <xacro:property name="middle_body_mass" value="1.5"/>
-    <xacro:property name="back_water_displaced_mass" value="40"/>
-    <xacro:property name="middle_water_displaced_mass" value="40"/>
-    <xacro:property name="front_water_displaced_mass" value="25"/>
-    <xacro:property name="scale" value="0.3"/>
+    <xacro:property name="front_body_mass" value="0.5"/>
+    <xacro:property name="back_body_mass" value="2"/>
+    <xacro:property name="middle_body_mass" value="2"/>
+    <xacro:property name="back_water_displaced_mass" value="10"/>
+    <xacro:property name="middle_water_displaced_mass" value="10"/>
+    <xacro:property name="front_water_displaced_mass" value="2"/>
+    <xacro:property name="scale" value="0.24"/>
     <xacro:property name="bl1" value=".1" />
     <xacro:property name="bl2" value=".1" />
@@ -34,5 +34,5 @@
 			<origin xyz="${0.35*scale} ${0.44*scale} ${-0.15*scale}"/>
 			<limit radius="0.1"/>
-			<damping rpy="20 20 20" xyz="0 18 60"/>
+			<damping rpy="${angularDampingXYZ}" xyz="${dampingXYZ}"/>
          	<windVelocity>${windType}</windVelocity>
 			<frontal_area>0.0</frontal_area>
@@ -64,5 +64,5 @@
           <origin xyz="${0.35*scale} ${-0.44*scale} ${-0.15*scale}"/>
           <limit radius="0.1"/>
-          <damping rpy="20 20 20" xyz="0 18 60"/>
+          <damping rpy="${angularDampingXYZ}" xyz="${dampingXYZ}"/>
 			<windVelocity>${windType}</windVelocity>
 			<frontal_area>0.0</frontal_area>
@@ -102,5 +102,5 @@
 			<origin xyz="${-0.6*scale} 0 ${-0.15*scale}"/>
 			<limit radius="0.1"/>
-			<damping rpy="20 20 20" xyz="0 18 60"/>
+			<damping rpy="${angularDampingXYZ}" xyz="${dampingXYZ}"/>
 			<windVelocity>${windType}</windVelocity>
 			<frontal_area>0.04</frontal_area>
@@ -140,5 +140,5 @@
           	<origin xyz="${-0.6*scale} 0 ${-0.15*scale}"/>
           	<limit radius="0.1"/>
-          	<damping rpy="20 20 20" xyz="0 18 60"/>
+          	<damping rpy="${angularDampingXYZ}" xyz="${dampingXYZ}"/>
           	<windVelocity>${windType}</windVelocity>
 			<frontal_area>0.04</frontal_area>
@@ -178,5 +178,5 @@
           	<origin xyz="${0.4*scale} 0 ${-0.05*scale}"/>
           	<limit radius="0.1"/>
-          	<damping rpy="20 20 20" xyz="${dampingXYZ}"/>
+          	<damping rpy="${angularDampingXYZ}" xyz="${dampingXYZ}"/>
           	<windVelocity>${windType}</windVelocity>
 			<frontal_area>0.04</frontal_area>
@@ -216,5 +216,5 @@
           <origin xyz="${0.4*scale} 0 ${-0.05*scale}"/>
           <limit radius="0.1"/>
-          <damping rpy="20 20 20" xyz="${dampingXYZ}"/>
+          <damping rpy="${angularDampingXYZ}" xyz="${dampingXYZ}"/>
           <windVelocity>${windType}</windVelocity>
 	  <waterVelocity>${waterType}</waterVelocity>
@@ -235,5 +235,5 @@
             <child link="${name}"/>
             <origin rpy="${rpy}" xyz="${xyz}"/>
-            <dynamics damping="10.0"/>
+            <dynamics damping="1.0"/>
             <axis xyz="${rotationAxis}"/>
             <limit effort="${effort}" velocity="${velocity}" lower="${lowerLimit}" upper="${upperLimit}" />
@@ -364,5 +364,5 @@
     <joint name="hokuyo_joint" type="fixed">
         <axis xyz="0 1 0" />
-        <origin xyz="0.7 0 0.2" rpy="0 0 0"/>
+        <origin xyz="0.56 0 0.2" rpy="0 0 0"/>
         <parent link="base_link"/>
         <child link="hokuyo_link"/>

File: usv_sim/xacro/diffboat_validation.xacro (robot description, xacro)
@@ -5,5 +5,6 @@
     <xacro:property name="windType" value="$(arg windType)" />
     <xacro:property name="waterType" value="$(arg waterType)" />
-    <xacro:property name="dampingXYZ" value="5.7 18 60" />
+    <xacro:property name="dampingXYZ" value="1.88 10 10" />
+    <xacro:property name="angularDampingXYZ" value="0.5 15 2" />
     <xacro:include filename="$(find usv_sim)/xacro/boat_subdivided_validation.xacro" />
     <!-- Plugin list -->
@@ -26,5 +27,5 @@
     </gazebo>
     <!-- Define two steering thrusters, with assumed force control in Z-direction -->
-    <xacro:thruster_link name="fwd_left"  xyz="-0.4 0 -0.1" rpy="0 ${-PI/2} 0" rotationAxis="1 0 0" lowerLimit="0" upperLimit="0" parentLink="back_l_link"/>
-    <xacro:thruster_link name="fwd_right" xyz="-0.4 0 -0.1" rpy="0 ${-PI/2} 0" rotationAxis="1 0 0" lowerLimit="0" upperLimit="0" parentLink="back_r_link"/>
+    <xacro:thruster_link name="fwd_left"  xyz="-0.4 0 -0.1" rpy="0 ${-PI/2-0.26} 0" rotationAxis="1 0 0" lowerLimit="0" upperLimit="0" parentLink="back_l_link"/>
+    <xacro:thruster_link name="fwd_right" xyz="-0.4 0 -0.1" rpy="0 ${-PI/2-0.26} 0" rotationAxis="1 0 0" lowerLimit="0" upperLimit="0" parentLink="back_r_link"/>
 </robot>
